File: moonratII/moonratII/moonratII.kicad_sch (KiCad schematic)
At the start: 14 parts

Commit message: Add annotations to reference designators on schematic. Create initial PCB and place components.
Parts:
- gave numbers to parts that had none: 14
Changed lines of the file:
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@@
   (symbol (lib_id "Switch:SW_MEC_5G") (at 200.66 96.52 0) (unit 1)
     (in_bom yes) (on_board yes) (fields_autoplaced)
-    (property "Reference" "SW?" (id 0) (at 200.66 88.9 0))
+    (property "Reference" "SW101" (id 0) (at 200.66 88.9 0))
     (property "Value" "6mm 2 Pin Tact NO" (id 1) (at 200.66 91.44 0))
     (property "Footprint" "Button_Switch_THT:SW_PUSH_6mm" (id 2) (at 200.66 91.44 0)
@@
   (symbol (lib_id "Device:Battery") (at 121.92 120.65 90) (unit 1)
     (in_bom yes) (on_board yes) (fields_autoplaced)
-    (property "Reference" "BT?" (id 0) (at 121.539 113.03 90))
+    (property "Reference" "BT101" (id 0) (at 121.539 113.03 90))
     (property "Value" "Battery" (id 1) (at 121.539 115.57 90))
     (property "Footprint" "" (id 2) (at 120.396 120.65 90)
@@
   (symbol (lib_id "MCU_Module:Arduino_UNO_R3") (at 133.35 78.74 0) (mirror y) (unit 1)
     (in_bom yes) (on_board yes) (fields_autoplaced)
-    (property "Reference" "A?" (id 0) (at 138.6587 50.8 0)
+    (property "Reference" "A101" (id 0) (at 138.6587 50.8 0)
       (effects (font (size 1.27 1.27)) (justify right))
     )
@@
   (symbol (lib_id "Device:Heater") (at 121.92 156.21 90) (unit 1)
     (in_bom yes) (on_board yes) (fields_autoplaced)
-    (property "Reference" "R?" (id 0) (at 121.92 149.86 90))
+    (property "Reference" "R102" (id 0) (at 121.92 149.86 90))
     (property "Value" "Heater" (id 1) (at 121.92 152.4 90))
     (property "Footprint" "" (id 2) (at 121.92 157.988 90)
@@
   (symbol (lib_id "Connector:Conn_01x08_Male") (at 68.58 102.87 0) (unit 1)
     (in_bom yes) (on_board yes) (fields_autoplaced)
-    (property "Reference" "J?" (id 0) (at 69.215 90.17 0))
+    (property "Reference" "J101" (id 0) (at 69.215 90.17 0))
     (property "Value" " SSD1306 OLED" (id 1) (at 69.215 92.71 0))
     (property "Footprint" "" (id 2) (at 68.58 102.87 0)
@@
   (symbol (lib_id "Device:Buzzer") (at 163.83 115.57 0) (unit 1)
     (in_bom yes) (on_board yes) (fields_autoplaced)
-    (property "Reference" "BZ?" (id 0) (at 167.64 114.2999 0)
+    (property "Reference" "BZ101" (id 0) (at 167.64 114.2999 0)
       (effects (font (size 1.27 1.27)) (justify left))
     )
@@
   (symbol (lib_id "Device:R_US") (at 53.34 44.45 90) (unit 1)
     (in_bom yes) (on_board yes)
-    (property "Reference" "R?" (id 0) (at 49.53 41.91 90))
+    (property "Reference" "R101" (id 0) (at 49.53 41.91 90))
     (property "Value" "1R" (id 1) (at 57.15 41.91 90))
     (property "Footprint" "Resistor_SMD:R_0603_1608Metric_Pad0.98x0.95mm_HandSolder" (id 2) (at 53.594 43.434 90)
@@
   (symbol (lib_id "Device:R_US") (at 171.45 71.12 90) (unit 1)
     (in_bom yes) (on_board yes)
-    (property "Reference" "R?" (id 0) (at 167.64 68.58 90))
+    (property "Reference" "R103" (id 0) (at 167.64 68.58 90))
     (property "Value" "1K" (id 1) (at 175.26 68.58 90))
     (property "Footprint" "Resistor_SMD:R_0603_1608Metric_Pad0.98x0.95mm_HandSolder" (id 2) (at 171.704 70.104 90)
@@
   (symbol (lib_id "Sensor_Temperature:TMP36xS") (at 67.31 64.77 0) (unit 1)
     (in_bom yes) (on_board yes) (fields_autoplaced)
-    (property "Reference" "U?" (id 0) (at 82.55 60.4393 0))
+    (property "Reference" "U101" (id 0) (at 82.55 60.4393 0))
     (property "Value" "TMP36xS" (id 1) (at 82.55 62.9793 0))
     (property "Footprint" "Package_SO:SOIC-8_3.9x4.9mm_P1.27mm" (id 2) (at 67.31 76.2 0)
@@
   (symbol (lib_id "Switch:SW_MEC_5G") (at 201.93 83.82 0) (unit 1)
     (in_bom yes) (on_board yes) (fields_autoplaced)
-    (property "Reference" "SW?" (id 0) (at 201.93 76.2 0))
+    (property "Reference" "SW103" (id 0) (at 201.93 76.2 0))
     (property "Value" "6mm 2 Pin Tact NO" (id 1) (at 201.93 78.74 0))
     (property "Footprint" "Button_Switch_THT:SW_PUSH_6mm" (id 2) (at 201.93 78.74 0)
@@
   (symbol (lib_id "Device:R_US") (at 171.45 96.52 90) (unit 1)
     (in_bom yes) (on_board yes)
-    (property "Reference" "R?" (id 0) (at 167.64 93.98 90))
+    (property "Reference" "R105" (id 0) (at 167.64 93.98 90))
     (property "Value" "1K" (id 1) (at 175.26 93.98 90))
     (property "Footprint" "Resistor_SMD:R_0603_1608Metric_Pad0.98x0.95mm_HandSolder" (id 2) (at 171.704 95.504 90)
@@
   (symbol (lib_id "Switch:SW_MEC_5G") (at 201.93 71.12 0) (unit 1)
     (in_bom yes) (on_board yes) (fields_autoplaced)
-    (property "Reference" "SW?" (id 0) (at 201.93 63.5 0))
+    (property "Reference" "SW102" (id 0) (at 201.93 63.5 0))
     (property "Value" "6mm 2 Pin Tact NO" (id 1) (at 201.93 66.04 0))
     (property "Footprint" "Button_Switch_THT:SW_PUSH_6mm" (id 2) (at 201.93 66.04 0)
@@
   (symbol (lib_id "Device:R_US") (at 171.45 83.82 90) (unit 1)
     (in_bom yes) (on_board yes)
-    (property "Reference" "R?" (id 0) (at 167.64 81.28 90))
+    (property "Reference" "R104" (id 0) (at 167.64 81.28 90))
     (property "Value" "1K" (id 1) (at 175.26 81.28 90))
     (property "Footprint" "Resistor_SMD:R_0603_1608Metric_Pad0.98x0.95mm_HandSolder" (id 2) (at 171.704 82.804 90)
@@
   (symbol (lib_id "Transistor_FET:IRF540N") (at 123.19 134.62 0) (mirror y) (unit 1)
     (in_bom yes) (on_board yes) (fields_autoplaced)
-    (property "Reference" "Q?" (id 0) (at 116.84 133.3499 0)
+    (property "Reference" "Q101" (id 0) (at 116.84 133.3499 0)
       (effects (font (size 1.27 1.27)) (justify left))
     )
@@
   (symbol_instances
     (path "/0fc4f76a-705d-497c-9e91-55c81d276aff"
-      (reference "A?") (unit 1) (value "Arduino_UNO_R3") (footprint "Module:Arduino_UNO_R3")
+      (reference "A101") (unit 1) (value "Arduino_UNO_R3") (footprint "Module:Arduino_UNO_R3")
     )
     (path "/024c4a87-41bc-4832-b4d4-17f8e5d0ac5a"
-      (reference "BT?") (unit 1) (value "Battery") (footprint "")
+      (reference "BT101") (unit 1) (value "Battery") (footprint "")
     )
     (path "/48f275ed-f59b-4204-b788-8473d424ccde"
-      (reference "BZ?") (unit 1) (value "Buzzer") (footprint "")
+      (reference "BZ101") (unit 1) (value "Buzzer") (footprint "")
     )
     (path "/421cf19f-2598-44f1-b4b8-12029a54a8f1"
-      (reference "J?") (unit 1) (value " SSD1306 OLED") (footprint "")
+      (reference "J101") (unit 1) (value " SSD1306 OLED") (footprint "")
     )
     (path "/f2d94110-6a69-4b1b-b5c4-6ca4750b43c1"
-      (reference "Q?") (unit 1) (value "IRF540N") (footprint "Package_TO_SOT_THT:TO-220-3_Vertical")
+      (reference "Q101") (unit 1) (value "IRF540N") (footprint "Package_TO_SOT_THT:TO-220-3_Vertical")
+    )
+    (path "/55acff0f-d774-4d88-9979-3a80839147dc"
+      (reference "R101") (unit 1) (value "1R") (footprint "Resistor_SMD:R_0603_1608Metric_Pad0.98x0.95mm_HandSolder")
     )
     (path "/25ab3db7-8e68-48ea-a04a-d5591c3dee53"
-      (reference "R?") (unit 1) (value "Heater") (footprint "")
-    )
-    (path "/55acff0f-d774-4d88-9979-3a80839147dc"
-      (reference "R?") (unit 1) (value "1R") (footprint "Resistor_SMD:R_0603_1608Metric_Pad0.98x0.95mm_HandSolder")
+      (reference "R102") (unit 1) (value "Heater") (footprint "")
     )
     (path "/56a4b48a-0021-407f-a492-20363488553e"
-      (reference "R?") (unit 1) (value "1K") (footprint "Resistor_SMD:R_0603_1608Metric_Pad0.98x0.95mm_HandSolder")
+      (reference "R103") (unit 1) (value "1K") (footprint "Resistor_SMD:R_0603_1608Metric_Pad0.98x0.95mm_HandSolder")
+    )
+    (path "/f10a84a9-1785-4331-9ea1-4932a4ef7429"
+      (reference "R104") (unit 1) (value "1K") (footprint "Resistor_SMD:R_0603_1608Metric_Pad0.98x0.95mm_HandSolder")
     )
     (path "/a4ebb2b9-1ebc-4034-9363-910625a6cdcd"
-      (reference "R?") (unit 1) (value "1K") (footprint "Resistor_SMD:R_0603_1608Metric_Pad0.98x0.95mm_HandSolder")
-    )
-    (path "/f10a84a9-1785-4331-9ea1-4932a4ef7429"
-      (reference "R?") (unit 1) (value "1K") (footprint "Resistor_SMD:R_0603_1608Metric_Pad0.98x0.95mm_HandSolder")
+      (reference "R105") (unit 1) (value "1K") (footprint "Resistor_SMD:R_0603_1608Metric_Pad0.98x0.95mm_HandSolder")
     )
     (path "/0093c405-df54-4104-8221-98614aaf511c"
-      (reference "SW?") (unit 1) (value "6mm 2 Pin Tact NO") (footprint "Button_Switch_THT:SW_PUSH_6mm")
+      (reference "SW101") (unit 1) (value "6mm 2 Pin Tact NO") (footprint "Button_Switch_THT:SW_PUSH_6mm")
+    )
+    (path "/ba4f12ca-f950-490a-af85-08596793f3b6"
+      (reference "SW102") (unit 1) (value "6mm 2 Pin Tact NO") (footprint "Button_Switch_THT:SW_PUSH_6mm")
     )
     (path "/9ec8e748-fdd0-4ae9-9b83-5ef8dddf3f0a"
-      (reference "SW?") (unit 1) (value "6mm 2 Pin Tact NO") (footprint "Button_Switch_THT:SW_PUSH_6mm")
-    )
-    (path "/ba4f12ca-f950-490a-af85-08596793f3b6"
-      (reference "SW?") (unit 1) (value "6mm 2 Pin Tact NO") (footprint "Button_Switch_THT:SW_PUSH_6mm")
+      (reference "SW103") (unit 1) (value "6mm 2 Pin Tact NO") (footprint "Button_Switch_THT:SW_PUSH_6mm")
     )
     (path "/686b66f2-234f-432d-90a2-b7c59deab86b"
-      (reference "U?") (unit 1) (value "TMP36xS") (footprint "Package_SO:SOIC-8_3.9x4.9mm_P1.27mm")
-    )
-  )
+      (reference "U101") (unit 1) (value "TMP36xS") (footprint "Package_SO:SOIC-8_3.9x4.9mm_P1.27mm")
+    )
+  )

Commit message: Add connectors and add incubator components.
Parts:
- removed BT101: Battery, symbol Device:Battery
- removed R101: 1R, Resistor_SMD:R_0603_1608Metric_Pad0.98x0.95mm_HandSolder, symbol Device:R_US
- added J? (x2): Screw_Terminal_01x06, TerminalBlock_TE-Connectivity:TerminalBlock_TE_282834-6_1x06_P2.54mm_Horizontal, symbol Connector:Screw_Terminal_01x06
- added J?: Barrel_Jack_Switch_Pin3Ring 2.1mmx5mm, Connector_BarrelJack:BarrelJack_CLIFF_FC681465S_SMT_Horizontal, symbol Connector:Barrel_Jack_Switch_Pin3Ring
- added J? (x2): Conn_02x05_Odd_Even, Connector_PinHeader_2.54mm:PinHeader_2x05_P2.54mm_Vertical, symbol Connector_Generic:Conn_02x05_Odd_Even
- added R? (x2): 1R, Resistor_SMD:R_0603_1608Metric_Pad0.98x0.95mm_HandSolder, symbol Device:R_US
- Q101: value IRF540N -> IRF520N
- SW102: value 6mm 2 Pin Tact NO -> 6mm 2 Pin Tact NO Breadboard Friendly
Connections:
- net +5V: now reaches A101.5 (+5V), J101.2 (Pin_2), SW101.3 (B), SW101.4 (B), SW102.3 (B), SW102.4 (B), SW103.3 (B), SW103.4 (B), U101.8 (+Vs)
- net +5V: now also J?.3 (Pin_3), J?.4 (Pin_4), J?.4 (Pin_4), J?.8 (Pin_8), R?.2; no longer U101.4 (GND)
- net HeaterDrive: now reaches Q101.2 (D)
- net HeaterDrive: now also R102.1, J?.1 (Pin_1), J?.10 (Pin_10), J?.3 (Pin_3), J?.3 (Pin_3)
- net GND: now reaches A101.29 (GND), A101.6 (GND), A101.7 (GND), BZ101.2 (+), J101.1 (Pin_1), J101.5 (Pin_5), J101.6 (Pin_6), J101.7 (Pin_7), J101.8 (Pin_8), R103.1, R104.1, R105.1
- net GND: now also Q101.3 (S), U101.4 (GND), J?.1 (Pin_1), J?.1 (Pin_1), J?.2, J?.2 (Pin_2), J?.3, J?.9 (Pin_9); no longer R102.2
- net VCC: now reaches A101.8 (VIN)
- net VCC: now also R102.2, J?.2 (Pin_2), J?.2 (Pin_2), J?.5 (Pin_5), J?.6 (Pin_6), R?.2
- net TempOut: now reaches A101.9 (A0), U101.1 (Vout)
- net TempOut: now also J?.4 (Pin_4), J?.5 (Pin_5), J?.5 (Pin_5), J?.7 (Pin_7)
- net at U101.5 (~{SHUTDOWN}): now also R?.1
- new net: J?.1, R?.1
Other:
- note added: "OLED Display 1-GND 2-+5V 3-SCL 4-SDA 5-MH1 6-MH2 7-MH3 8-MH4"
- note added: "VCC is the raw power coming in from a batter or wall supply."
- note removed: "OLED Display 1-GND 2-VCC 3-SCL 4-SDA 5-MH1 6-MH2 7-MH3 8-MH4"
- moved on the sheet: A101, BZ101, J101, Q101, R102, R103, R104, R105, SW101, SW102, SW103, U101

Commit message: Finished wiring connectors.
Parts:
- removed J?: Conn_02x05_Odd_Even, Connector_PinHeader_2.54mm:PinHeader_2x05_P2.54mm_Vertical, symbol Connector_Generic:Conn_02x05_Odd_Even
- added J?: Conn_02x05_Odd_Even, Connector_PinHeader_2.54mm:PinHeader_2x05_P2.54mm_Vertical, symbol Connector_Generic:Conn_02x05_Odd_Even
Connections:
- net +5V: now also J?.3 (Pin_3), J?.8 (Pin_8); no longer SW101.3 (B), SW101.4 (B), SW102.3 (B), SW102.4 (B), SW103.3 (B), SW103.4 (B)
- net GND: now also J?.2 (Pin_2), J?.9 (Pin_9)
- net HeaterDrive: now also J?.1 (Pin_1), J?.10 (Pin_10)
- net TempOut: now also J?.4 (Pin_4), J?.7 (Pin_7)
- net VCC: now also J?.5 (Pin_5), J?.6 (Pin_6)
- new net: SW101.3 (B), SW101.4 (B)
- new net: SW103.3 (B), SW103.4 (B)
- new net: SW102.3 (B), SW102.4 (B)
Other:
- moved on the sheet: A101, BZ101, J101, J?, Q101, R103, R104, R105, R?, SW101, SW102, SW103

Commit message: Named more nets, Add reverse voltage protection.
Parts:
- removed BZ101: Buzzer, symbol Device:Buzzer
- removed SW101, SW103: 6mm 2 Pin Tact NO, Button_Switch_THT:SW_PUSH_6mm, symbol Switch:SW_MEC_5G
- added BZ1: Buzzer_Adafruit_P1536A, GeneralPurposeAlarmDevicePCB:Buzzer_12.2mm_9.7mm_7.62mm, symbol GPAD_SCH_LIB:Buzzer_Adafruit_P1536A
- added D1: Schottky 2A, Diode_SMD:D_SMB, symbol Device:D_Schottky
- added Q2: BSS138, Package_TO_SOT_SMD:SOT-23, symbol Transistor_FET:BSS138
- added R2: 1R, Resistor_SMD:R_0603_1608Metric_Pad0.98x0.95mm_HandSolder, symbol Device:R_US
- added R3: 1K, Resistor_SMD:R_0603_1608Metric_Pad0.98x0.95mm_HandSolder, symbol Device:R_US
- added SW1, SW3: 6mm 2 Pin Tact NO Breadboard Friendly, Button_Switch_THT:SW_PUSH_6mm, symbol Switch:SW_MEC_5G
- gave numbers to parts that had none: 7
- renumbered A101 to A1, J101 to J2, Q101 to Q1, R103 to R4, R104 to R5, R105 to R6, R102 to R8, SW102 to SW2, U101 to U1
Connections:
- net +5V: now also SW2.3 (B), SW2.4 (B), BZ1.1 (-), SW1.3 (B), SW1.4 (B), SW3.3 (B), SW3.4 (B)
- net GND: now also J4.6 (Pin_6), J5.6 (Pin_6), Q2.2 (S)
- net HeaterDrive: now also D1.1 (K); no longer R8.1
- net TempOut: now also R2.2; no longer A1.9 (A0)
- net BTN_DOWN: now reaches A1.22 (D7), R6.2
- net BTN_DOWN: now also SW1.1 (A), SW1.2 (A)
- net SCL: now reaches A1.13 (SDA/A4), J2.4 (Pin_4)
- net BTN_SELECT: now reaches A1.20 (D5), R4.2, SW2.1 (A), SW2.2 (A)
- net BTN_UP: now reaches A1.21 (D6), R5.2
- net BTN_UP: now also SW3.1 (A), SW3.2 (A)
- net HEATER_ON: now reaches A1.23 (D8), Q1.1 (G)
- net BUZZER_ON: now reaches A1.24 (D9)
- net BUZZER_ON: now also R3.1
- new net: D1.2 (A), R8.1
- new net: Q2.1 (G), R3.2
- new net: BZ1.2 (+), Q2.3 (D)
- new net TEMP_IN: A1.9 (A0), R2.1
Other:
- note added: "Controller Board"
- note added: "Incubator Board"
- note added: "VCC is the raw power coming in from a battery or wall supply."
- note removed: "VCC is the raw power coming in from a batter or wall supply."
- moved on the sheet: J1, R1

Commit message: Add many JLCPCB and other vendor part numbers. Add cables.
Parts:
- removed J1: Barrel_Jack_Switch_Pin3Ring 2.1mmx5mm, Connector_BarrelJack:BarrelJack_CLIFF_FC681465S_SMT_Horizontal, symbol Connector:Barrel_Jack_Switch_Pin3Ring
- added Cable_MoldedFemale1: Cable_02x06_Female, symbol Connector_Generic:Conn_02x05_Odd_Even
- added Cable_MoldedMale1: Cable_02x06_Male, symbol Connector_Generic:Conn_02x05_Odd_Even
- added Cable_Ribbon1: Cable_02x05, symbol Connector_Generic:Conn_02x05_Odd_Even
- added D?: Schottky 2A, Diode_SMD:D_SMB, symbol Device:D_Schottky
- added J1: Barrel_Jack_Switch_SMT, GeneralPurposeAlarmDevicePCB:BarrelJack_CLIFF_FC681465S_SMT_Horizontal, symbol GPAD_SCH_LIB:Barrel_Jack_Switch_SMT
- added TP1: TP_GND, TestPoint:TestPoint_Loop_D2.54mm_Drill1.5mm_Beaded, symbol Connector:TestPoint
- A1: AssemblyType (none) -> HAND
- J3, J6: AssemblyType (none) -> HAND; Cost (none) -> 0.0655; Distributor 1 (none) -> JLCPCB; Distributor 1 PN (none) -> C5665; MPN (none) -> C5665; Manufacturer (none) -> BOOMELE(Boom Precision Elec)
- J4, J5: AssemblyType (none) -> HAND; Cost (none) -> 0.4614; Distributor 1 (none) -> JLCPCB; Distributor 1 PN (none) -> C2915642; MPN (none) -> DB128V-5.08-6P-GN-S; Manufacturer (none) -> DIBO
- Q1: AssemblyType (none) -> HAND; Cost (none) -> 0.6995; Distributor 1 (none) -> JLCPCB; Distributor 1 PN (none) -> C2598; MPN (none) -> IRF520NPBF; Manufacturer (none) -> Infineon Technologies
- R1, R2, R7: AssemblyType (none) -> SMT; Cost (none) -> 0.0015; Distributor 1 (none) -> JLCPCB; Distributor 1 PN (none) -> C269434; MPN (none) -> RMC060315%N; Manufacturer (none) -> TyoHM
- R3: renamed from R4; AssemblyType (none) -> SMT; Cost (none) -> 0.0015; Distributor 1 (none) -> JLCPCB; Distributor 1 PN (none) -> C269704; MPN (none) -> RMC06031K1%N; Manufacturer (none) -> TyoHM
- R4: renamed from R5; AssemblyType (none) -> SMT; Cost (none) -> 0.0015; Distributor 1 (none) -> JLCPCB; Distributor 1 PN (none) -> C269704; MPN (none) -> RMC06031K1%N; Manufacturer (none) -> TyoHM
- R5: renamed from R6; AssemblyType (none) -> SMT; Cost (none) -> 0.0015; Distributor 1 (none) -> JLCPCB; Distributor 1 PN (none) -> C269704; MPN (none) -> RMC06031K1%N; Manufacturer (none) -> TyoHM
- R6: renamed from R3; AssemblyType (none) -> SMT; Cost (none) -> 0.0015; Distributor 1 (none) -> JLCPCB; Distributor 1 PN (none) -> C269704; MPN (none) -> RMC06031K1%N; Manufacturer (none) -> TyoHM
- R8: AssemblyType (none) -> OTHER; Cost (none) -> 4.50; Distributor 1 (none) -> Sparkfun; Distributor 1 PN (none) -> COM-11288
- U1: AssemblyType (none) -> SMT; Cost (none) -> 1.297; Distributor 1 (none) -> JLCPCB; Distributor 1 PN (none) -> C129489; MPN (none) -> TMP36GRTZ; Manufacturer (none) -> Analog Devices
Connections:
- net GND: now also J1.2, J1.3, TP1.1
- net SCL: now also A1.14 (SCL/A5), J2.3 (Pin_3); no longer A1.13 (SDA/A4), J2.4 (Pin_4)
- net at R1.1: now also J1.1, J1.4
- new net SDA: A1.13 (SDA/A4), J2.4 (Pin_4)
- no-connect marks 0 -> 18
Other:
- note added: "Molded Cable from Controller to Incubator."
- note added: "Ribbon Cable from Controller to Incubator."

Commit message: Pull in parts to PCB. Make some initial placement.
Parts:
- removed D?: Schottky 2A, Diode_SMD:D_SMB, symbol Device:D_Schottky
- added J7: Screw_Terminal_01x02, TerminalBlock_4Ucon:TerminalBlock_4Ucon_1x02_P3.50mm_Horizontal, symbol Connector:Screw_Terminal_01x02
- added R9: 1K, Resistor_SMD:R_0603_1608Metric_Pad0.98x0.95mm_HandSolder, symbol Device:R_US
- renumbered D1 to D2, SW2 to SW1, SW3 to SW2, SW1 to SW3
Connections:
- net HEATER_ON: now also R9.1; no longer A1.23 (D8)
- net VCC: now also J7.1 (Pin_1)
- net at D2.2 (A), R8.1: now also J7.2 (Pin_2)
- new net: A1.23 (D8), R9.2
Other:
- moved on the sheet: R8

Commit message: Add remaning new footprint files, add parts files.
Parts:
- A1: Cost (none) -> 1000000
- SW1, SW2, SW3: Cost (none) -> 0.50000; Distributor 1 (none) -> Digikey; Distributor 1 PN (none) -> SW798TB-ND
- TP1: AssemblyType NA -> DNI; Cost (none) -> 0.38000; Distributor 1 NA -> Digikey; Distributor 1 PN NA -> 36-5117-ND; MPN NA -> 5117; Manufacturer NA -> Keystone Electronics; now left out of the parts list
Changed lines of the file:
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@@
+      (effects (font (size 1.27 1.27)) hide)
+    )
+    (property "Cost" "1000000" (id 5) (at 86.36 77.47 0)
       (effects (font (size 1.27 1.27)) hide)
     )
@@
       (effects (font (size 1.27 1.27)) hide)
     )
+    (property "Cost" "0.50000" (id 4) (at 153.67 95.25 0)
+      (effects (font (size 1.27 1.27)) hide)
+    )
+    (property "Distributor 1" "Digikey" (id 5) (at 153.67 95.25 0)
+      (effects (font (size 1.27 1.27)) hide)
+    )
+    (property "Distributor 1 PN" "SW798TB-ND" (id 6) (at 153.67 95.25 0)
+      (effects (font (size 1.27 1.27)) hide)
+    )
     (pin "1")
     (pin "3")
@@
     )
     (property "Datasheet" "https://www.amazon.com/Momentary-Tactile-Through-Breadboard-Friendly/dp/B07WF76VHT/" (id 3) (at 154.94 77.47 0)
+      (effects (font (size 1.27 1.27)) hide)
+    )
+    (property "Cost" "0.50000" (id 4) (at 154.94 82.55 0)
+      (effects (font (size 1.27 1.27)) hide)
+    )
+    (property "Distributor 1" "Digikey" (id 5) (at 154.94 82.55 0)
+      (effects (font (size 1.27 1.27)) hide)
+    )
+    (property "Distributor 1 PN" "SW798TB-ND" (id 6) (at 154.94 82.55 0)
       (effects (font (size 1.27 1.27)) hide)
     )
@@
       (effects (font (size 1.27 1.27)) hide)
     )
+    (property "Cost" "0.50000" (id 4) (at 154.94 69.85 0)
+      (effects (font (size 1.27 1.27)) hide)
+    )
+    (property "Distributor 1" "Digikey" (id 5) (at 154.94 69.85 0)
+      (effects (font (size 1.27 1.27)) hide)
+    )
+    (property "Distributor 1 PN" "SW798TB-ND" (id 6) (at 154.94 69.85 0)
+      (effects (font (size 1.27 1.27)) hide)
+    )
     (pin "1")
     (pin "3")
@@
   )
   (symbol (lib_id "Connector:TestPoint") (at 27.305 46.99 0) (unit 1)
-    (in_bom yes) (on_board yes)
+    (in_bom no) (on_board yes)
     (property "Reference" "TP1" (id 0) (at 18.415 44.45 0)
       (effects (font (size 1.27 1.27)) (justify left))
@@
       (effects (font (size 1.27 1.27)) hide)
     )
-    (property "Datasheet" "NA" (id 3) (at 32.385 46.99 0)
-      (effects (font (size 1.27 1.27)) hide)
-    )
-    (property "AssemblyType" "NA" (id 4) (at 27.305 46.99 0)
-      (effects (font (size 1.27 1.27)) hide)
-    )
-    (property "Description" "NA" (id 5) (at 27.305 46.99 0)
-      (effects (font (size 1.27 1.27)) hide)
-    )
-    (property "Distributor 1" "NA" (id 6) (at 27.305 46.99 0)
-      (effects (font (size 1.27 1.27)) hide)
-    )
-    (property "Distributor 1 PN" "NA" (id 7) (at 27.305 46.99 0)
-      (effects (font (size 1.27 1.27)) hide)
-    )
-    (property "MPN" "NA" (id 8) (at 27.305 46.99 0)
-      (effects (font (size 1.27 1.27)) hide)
-    )
-    (property "Manufacturer" "NA" (id 9) (at 27.305 46.99 0)
-      (effects (font (size 1.27 1.27)) hide)
-    )
+    (property "Datasheet" "https://www.keyelco.com/userAssets/file/M65p56.pdf" (id 3) (at 32.385 46.99 0)
+      (effects (font (size 1.27 1.27)) hide)
+    )
+    (property "AssemblyType" "DNI" (id 4) (at 27.305 46.99 0)
+      (effects (font (size 1.27 1.27)) hide)
+    )
+    (property "Description" "Blue PC Test Point, Miniature Phosphor Bronze Silver Plating Through Hole Mounting Type" (id 5) (at 27.305 46.99 0)
+      (effects (font (size 1.27 1.27)) hide)
+    )
+    (property "Distributor 1" "Digikey" (id 6) (at 27.305 46.99 0)
+      (effects (font (size 1.27 1.27)) hide)
+    )
+    (property "Distributor 1 PN" "36-5117-ND" (id 7) (at 27.305 46.99 0)
+      (effects (font (size 1.27 1.27)) hide)
+    )
+    (property "MPN" "5117" (id 8) (at 27.305 46.99 0)
+      (effects (font (size 1.27 1.27)) hide)
+    )
+    (property "Manufacturer" "Keystone Electronics" (id 9) (at 27.305 46.99 0)
+      (effects (font (size 1.27 1.27)) hide)
+    )
+    (property "Cost" "0.38000" (id 10) (at 27.305 46.99 0)
+      (effects (font (size 1.27 1.27)) hide)
+    )
