File: moonratII/moonratII/moonratII.kicad_sch (KiCad schematic)
At the start: 29 parts, among them J1 Barrel_Jack_Switch_SMT, J2 SSD1306 OLED, J3 Conn_02x05_Odd_Even, J4 Screw_Terminal_01x06, J5 Screw_Terminal_01x06, J6 Conn_02x05_Odd_Even, J7 Screw_Terminal_01x02, Q1 IRF520N, Q2 BSS138, SW1 6mm 2 Pin Tact NO Breadboard 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, SW2 6mm 2 Pin Tact NO Breadboard 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, SW3 6mm 2 Pin Tact NO Breadboard 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, U1 TMP36xS

Commit message: Add more PCB 3D models. Place and lock down mounting holes.
Parts:
- removed R1: 1R, Resistor_SMD:R_0603_1608Metric_Pad0.98x0.95mm_HandSolder, symbol Device:R_US
- added F1: Polyfuse 6A, GeneralPurposeAlarmDevicePCB:PlaceHolderOpossum, symbol Device:Polyfuse
- added H1, H2, H3, H4, H5, H6: MountingHole_Pad_3.5mm, GeneralPurposeAlarmDevicePCB:MountingHole_3.5mm_Pad_Via, symbol GPAD_SCH_LIB:MountingHole_Pad_3.5mm
- added J3: Conn_01x06_Male, Connector_PinHeader_2.54mm:PinHeader_1x06_P2.54mm_Vertical, symbol Connector:Conn_01x06_Male
- added J4, J7: Conn_01x08_Male, Connector_PinHeader_2.54mm:PinHeader_1x08_P2.54mm_Vertical, symbol Connector:Conn_01x08_Male
- added J8: Conn_01x10_Male, Connector_PinHeader_2.54mm:PinHeader_1x10_P2.54mm_Vertical, symbol Connector:Conn_01x10_Male
- added TP2: TP_GND, TestPoint:TestPoint_Loop_D2.54mm_Drill1.5mm_Beaded, symbol Connector:TestPoint
- A1: footprint Module:Arduino_UNO_R3 -> GeneralPurposeAlarmDevicePCB:Arduino_UNO_R3_NoMountingHoles3D
- J11: renamed from J7; footprint TerminalBlock_4Ucon:TerminalBlock_4Ucon_1x02_P3.50mm_Horizontal -> TerminalBlock_TE-Connectivity:TerminalBlock_TE_282834-2_1x02_P2.54mm_Horizontal; AssemblyType (none) -> HAND; Cost (none) -> 0.1537; Distributor 1 (none) -> JLCPCB; Distributor 1 PN (none) -> C2915639
- J2: AssemblyType (none) -> HAND; Cost (none) -> 1.64; Distributor 1 (none) -> JLCPCB; Distributor 1 PN (none) -> C5248080; Distributor 2 (none) -> Amazon; Distributor 2 PN (none) -> https://www.amazon.com/gp/product/B08R8X2WWL/ref=ox_sc_act_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; MPN (none) -> HS96L03W2C03; Manufacturer (none) -> HS
- renumbered D2 to D1, J6 to J10, J3 to J5, J4 to J6, J5 to J9, R2 to R1, R9 to R2, SW3 to SW1, SW1 to SW2, SW2 to SW3
Connections:
- net GND: now also H1.1, H2.1, H3.1, H4.1, H5.1, H6.1, TP2.1
- net VCC: now also F1.1
- net at J1.1, J1.4: now also F1.2
Other:
- note added: "Board to UNO Headers"
- moved on the sheet: BZ1
