File: moonratII/moonratII/moonratII.kicad_sch (KiCad schematic)
At the start: 40 parts, among them J1 Barrel_Jack_Switch_SMT, J10 Conn_02x05_Odd_Even, J11 Screw_Terminal_01x02, J2 HS96L03W2C03_0.96_Oled, J3 Conn_01x06_Male, J4 Conn_01x08_Male, J5 Conn_02x05_Odd_Even, J6 Screw_Terminal_01x06, J7 Conn_01x08_Male, J8 Conn_01x10_Male, J9 Screw_Terminal_01x06, Q1 IRF520N, Q2 BSS138, SW1 6mm 2 Pin Tact NO Breadboard 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, SW2 6mm 2 Pin Tact NO Breadboard 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, SW3 6mm 2 Pin Tact NO Breadboard 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, U1 TMP36xS

Commit message: Deleted board to board headers. Placed components before getting to route
Parts:
- removed J3: Conn_01x06_Male, Connector_PinHeader_2.54mm:PinHeader_1x06_P2.54mm_Vertical, symbol Connector:Conn_01x06_Male
- removed J4, J7: Conn_01x08_Male, Connector_PinHeader_2.54mm:PinHeader_1x08_P2.54mm_Vertical, symbol Connector:Conn_01x08_Male
- removed J8: Conn_01x10_Male, Connector_PinHeader_2.54mm:PinHeader_1x10_P2.54mm_Vertical, symbol Connector:Conn_01x10_Male
- Q1: footprint Package_TO_SOT_THT:TO-220-3_Vertical -> Package_TO_SOT_THT:TO-220-3_Horizontal_TabDown

Commit message: Fixed footprint for SW 1, 2, 3. Significant update on bottom copper ground
Parts:
- SW1, SW2, SW3: footprint Button_Switch_THT:SW_PUSH_6mm -> GeneralPurposeAlarmDevicePCB:Switch_Tactile_THT_6x6mm
Changed lines of the file:
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@@
       (effects (font (size 1.27 1.27)))
     )
-    (property "Footprint" "Button_Switch_THT:SW_PUSH_6mm" (at 153.67 87.63 0)
+    (property "Footprint" "GeneralPurposeAlarmDevicePCB:Switch_Tactile_THT_6x6mm" (at 153.67 87.63 0)
       (effects (font (size 1.27 1.27)) hide)
     )
@@
       (effects (font (size 1.27 1.27)))
     )
-    (property "Footprint" "Button_Switch_THT:SW_PUSH_6mm" (at 154.94 74.93 0)
+    (property "Footprint" "GeneralPurposeAlarmDevicePCB:Switch_Tactile_THT_6x6mm" (at 154.94 74.93 0)
       (effects (font (size 1.27 1.27)) hide)
     )
@@
       (effects (font (size 1.27 1.27)))
     )
-    (property "Footprint" "Button_Switch_THT:SW_PUSH_6mm" (at 154.94 62.23 0)
-      (effects (font (size 1.27 1.27)) hide)
-    )
+    (property "Footprint" "GeneralPurposeAlarmDevicePCB:Switch_Tactile_THT_6x6mm" (at 154.94 62.23 0)
+      (effects (font (size 1.27 1.27)) hide)
+    )

Commit message: Performing design rule checks. Added ground between SCL & SDA traces to reduce the opportunity for cross talk.
Connections:
- no-connect marks 20 -> 19
Changed lines of the file:
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@@
   (junction (at 161.29 82.55) (diameter 0) (color 0 0 0 0)
   )
-  (no_connect (at 68.58 100.33))
   (no_connect (at 73.66 80.01))
   (no_connect (at 73.66 82.55))

Commit message: Update to fix schematic errors and warnings.
Parts:
- J2: symbol Connector:Conn_01x08_Male -> Connector:Conn_01x08_Pin
Connections:
- no-connect marks 19 -> 48
Changed lines of the file:
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@@
   (junction (at 162.56 69.85) (diameter 0) (color 0 0 0 0)
   )
+  (junction (at 243.84 116.84) (diameter 0) (color 0 0 0 0)
+  )
   (junction (at 222.25 151.13) (diameter 0) (color 0 0 0 0)
   )
@@
   (junction (at 163.83 69.85) (diameter 0) (color 0 0 0 0)
   )
+  (junction (at 215.9 123.19) (diameter 0) (color 0 0 0 0)
+  )
   (junction (at 81.28 45.72) (diameter 0) (color 0 0 0 0)
   )
@@
   (junction (at 241.3 148.59) (diameter 0) (color 0 0 0 0)
   )
+  (junction (at 190.5 110.49) (diameter 0) (color 0 0 0 0)
+  )
   (junction (at 134.62 151.13) (diameter 0) (color 0 0 0 0)
   )
@@
   (junction (at 161.29 82.55) (diameter 0) (color 0 0 0 0)
   )
+  (no_connect (at 212.09 27.94))
+  (no_connect (at 248.92 64.77))
+  (no_connect (at 196.85 66.04))
+  (no_connect (at 209.55 58.42))
   (no_connect (at 73.66 80.01))
   (no_connect (at 73.66 82.55))
@@
   (no_connect (at 99.06 72.39))
   (no_connect (at 99.06 62.23))
-  (no_connect (at 255.27 157.48))
+  (no_connect (at 248.92 57.15))
+  (no_connect (at 248.92 62.23))
+  (no_connect (at 261.62 64.77))
+  (no_connect (at 261.62 67.31))
+  (no_connect (at 199.39 25.4))
+  (no_connect (at 199.39 27.94))
+  (no_connect (at 196.85 55.88))
+  (no_connect (at 212.09 25.4))
+  (no_connect (at 199.39 33.02))
+  (no_connect (at 196.85 60.96))
+  (no_connect (at 209.55 63.5))
+  (no_connect (at 248.92 67.31))
+  (no_connect (at 261.62 62.23))
+  (no_connect (at 196.85 58.42))
+  (no_connect (at 261.62 59.69))
+  (no_connect (at 248.92 59.69))
+  (no_connect (at 212.09 33.02))
+  (no_connect (at 261.62 57.15))
+  (no_connect (at 212.09 30.48))
+  (no_connect (at 212.09 35.56))
+  (no_connect (at 209.55 60.96))
+  (no_connect (at 199.39 30.48))
+  (no_connect (at 209.55 66.04))
+  (no_connect (at 209.55 55.88))
+  (no_connect (at 196.85 63.5))
+  (no_connect (at 199.39 35.56))
   (wire (pts (xy 146.05 138.43) (xy 143.51 138.43))
     (stroke (width 0) (type default))
@@
     (stroke (width 0) (type default))
   )
+  (wire (pts (xy 219.075 123.19) (xy 215.9 123.19))
+    (stroke (width 0) (type default))
+  )
   (wire (pts (xy 135.89 156.21) (xy 133.35 156.21))
     (stroke (width 0) (type default))
@@
     (stroke (width 0) (type default))
   )
+  (wire (pts (xy 215.9 123.19) (xy 215.9 125.73))
+    (stroke (width 0) (type default))
+  )
   (wire (pts (xy 99.06 82.55) (xy 106.68 82.55))
     (stroke (width 0) (type default))
@@
     (stroke (width 0) (type default))
   )
+  (wire (pts (xy 219.075 118.11) (xy 219.075 123.19))
+    (stroke (width 0) (type default))
+  )
   (wire (pts (xy 208.28 123.19) (xy 208.28 113.03))
     (stroke (width 0) (type default))
@@
     (stroke (width 0) (type default))
   )
+  (wire (pts (xy 190.5 110.49) (xy 184.785 110.49))
+    (stroke (width 0) (type default))
+  )
   (wire (pts (xy 41.91 111.76) (xy 41.91 109.22))
     (stroke (width 0) (type default))
@@
     (stroke (width 0) (type default))
   )
+  (wire (pts (xy 190.5 110.49) (xy 190.5 113.03))
+    (stroke (width 0) (type default))
+  )
   (wire (pts (xy 62.23 90.17) (xy 62.23 99.06))
     (stroke (width 0) (type default))
@@
     (stroke (width 0) (type default))
   )
+  (wire (pts (xy 243.84 116.84) (xy 248.285 116.84))
+    (stroke (width 0) (type default))
+  )
   (wire (pts (xy 161.29 80.01) (xy 161.29 82.55))
     (stroke (width 0) (type default))
@@
     (stroke (width 0) (type default))
   )
+  (wire (pts (xy 248.285 116.84) (xy 248.285 106.68))
+    (stroke (width 0) (type default))
+  )
   (wire (pts (xy 241.3 158.75) (xy 241.3 152.4))
     (stroke (width 0) (type default))
@@
     (stroke (width 0) (type default))
   )
-  (wire (pts (xy 243.84 114.3) (xy 243.84 119.38))
+  (wire (pts (xy 243.84 114.3) (xy 243.84 116.84))
     (stroke (width 0) (type default))
   )
@@
     (stroke (width 0) (type default))
   )
+  (wire (pts (xy 215.9 118.745) (xy 215.9 123.19))
+    (stroke (width 0) (type default))
+  )
   (wire (pts (xy 215.9 140.97) (xy 215.9 153.67))
     (stroke (width 0) (type default))
@@
     (stroke (width 0) (type default))
   )
+  (wire (pts (xy 184.785 110.49) (xy 184.785 108.585))
+    (stroke (width 0) (type default))
+  )
   (wire (pts (xy 163.83 105.41) (xy 166.37 105.41))
     (stroke (width 0) (type default))
@@
     (stroke (width 0) (type default))
   )
-  (wire (pts (xy 190.5 105.41) (xy 190.5 113.03))
+  (wire (pts (xy 190.5 105.41) (xy 190.5 110.49))
     (stroke (width 0) (type default))
   )
@@
     (stroke (width 0) (type default))
   )
+  (wire (pts (xy 243.84 116.84) (xy 243.84 119.38))
+    (stroke (width 0) (type default))
+  )
   (wire (pts (xy 208.28 128.27) (xy 226.06 128.27))
     (stroke (width 0) (type default))
@@
     )
   )
+  (symbol (lib_id "power:PWR_FLAG") (at 219.075 118.11 0) (unit 1)
+    (in_bom yes) (on_board yes) (dnp no)
+    (property "Reference" "#FLG04" (at 219.075 116.205 0)
+      (effects (font (size 1.27 1.27)) hide)
+    )
+    (property "Value" "PWR_FLAG" (at 225.425 116.84 0)
+      (effects (font (size 1.27 1.27)))
+    )
+    (property "Footprint" "" (at 219.075 118.11 0)
+      (effects (font (size 1.27 1.27)) hide)
+    )
+    (property "Datasheet" "~" (at 219.075 118.11 0)
+      (effects (font (size 1.27 1.27)) hide)
+    )
+    (pin "1")
+    (instances
+      (project "moonratII"
+        (path "/9ef5effe-cb46-4a9a-bbbe-a65ab44b9e67"
+          (reference "#FLG04") (unit 1)
+        )
+      )
+    )
+  )
   (symbol (lib_id "Connector_Generic:Conn_02x05_Odd_Even") (at 204.47 30.48 0) (unit 1)
     (in_bom yes) (on_board no) (dnp no) (fields_autoplaced)
@@
     )
   )
-  (symbol (lib_id "Connector:Conn_01x08_Male") (at 30.48 101.6 0) (unit 1)
+  (symbol (lib_id "Connector:Conn_01x08_Pin") (at 30.48 101.6 0) (unit 1)
     (in_bom yes) (on_board yes) (dnp no)
     (property "Reference" "J2" (at 31.115 88.9 0)
@@
       (effects (font (size 1.27 1.27)))
     )
-    (property "Footprint" "GeneralPurposeAlarmDevicePCB:HS96L03W2C03_0.96_Oled" (at 34.29 68.58 0)
-      (effects (font (size 1.27 1.27)))
+    (property "Footprint" "GeneralPurposeAlarmDevicePCB:HS96L03W2C03_0.96_Oled" (at 30.48 101.6 0)
+      (effects (font (size 1.27 1.27)) hide)
     )
-    (property "Datasheet" "2305050946_HS-HS96L03W2C03_C5248080.pdf" (at 30.48 101.6 0)
+    (property "Datasheet" "~" (at 30.48 101.6 0)
       (effects (font (size 1.27 1.27)) hide)
     )
@@
     )
   )
+  (symbol (lib_id "power:PWR_FLAG") (at 184.785 108.585 0) (unit 1)
+    (in_bom yes) (on_board yes) (dnp no)
+    (property "Reference" "#FLG05" (at 184.785 106.68 0)
+      (effects (font (size 1.27 1.27)) hide)
+    )
+    (property "Value" "PWR_FLAG" (at 191.135 107.95 0)
+      (effects (font (size 1.27 1.27)))
+    )
+    (property "Footprint" "" (at 184.785 108.585 0)
+      (effects (font (size 1.27 1.27)) hide)
+    )
+    (property "Datasheet" "~" (at 184.785 108.585 0)
+      (effects (font (size 1.27 1.27)) hide)
+    )
+    (pin "1")
+    (instances
+      (project "moonratII"
+        (path "/9ef5effe-cb46-4a9a-bbbe-a65ab44b9e67"
+          (reference "#FLG05") (unit 1)
+        )
+      )
+    )
+  )
   (symbol (lib_id "Switch:SW_MEC_5E") (at 153.67 95.25 0) (unit 1)
     (in_bom yes) (on_board yes) (dnp no)
@@
     )
   )
+  (symbol (lib_id "power:PWR_FLAG") (at 248.285 106.68 0) (unit 1)
+    (in_bom yes) (on_board yes) (dnp no)
+    (property "Reference" "#FLG06" (at 248.285 104.775 0)
+      (effects (font (size 1.27 1.27)) hide)
+    )
+    (property "Value" "PWR_FLAG" (at 254.635 106.045 0)
+      (effects (font (size 1.27 1.27)))
+    )
+    (property "Footprint" "" (at 248.285 106.68 0)
+      (effects (font (size 1.27 1.27)) hide)
+    )
+    (property "Datasheet" "~" (at 248.285 106.68 0)
+      (effects (font (size 1.27 1.27)) hide)
+    )
+    (pin "1")
+    (instances
+      (project "moonratII"
+        (path "/9ef5effe-cb46-4a9a-bbbe-a65ab44b9e67"
+          (reference "#FLG06") (unit 1)
+        )
+      )
+    )
+  )
   (symbol (lib_id "power:GND1") (at 243.84 144.78 0) (unit 1)
     (in_bom yes) (on_board yes) (dnp no) (fields_autoplaced)
@@
     )
   )
-  (symbol (lib_id "power:VCCQ") (at 215.9 125.73 0) (unit 1)
+  (symbol (lib_id "power:VCCQ") (at 215.9 118.745 0) (unit 1)
     (in_bom yes) (on_board yes) (dnp no) (fields_autoplaced)
-    (property "Reference" "#PWR016" (at 215.9 129.54 0)
+    (property "Reference" "#PWR016" (at 215.9 122.555 0)
       (effects (font (size 1.27 1.27)) hide)
     )
-    (property "Value" "VCCQ" (at 215.9 120.65 0)
+    (property "Value" "VCCQ" (at 215.9 113.665 0)
       (effects (font (size 1.27 1.27)))
     )
-    (property "Footprint" "" (at 215.9 125.73 0)
+    (property "Footprint" "" (at 215.9 118.745 0)
       (effects (font (size 1.27 1.27)) hide)
     )
-    (property "Datasheet" "" (at 215.9 125.73 0)
+    (property "Datasheet" "" (at 215.9 118.745 0)
       (effects (font (size 1.27 1.27)) hide)
     )

Commit message: Cleared all DRC errors and warnings. Added 3 footprints
Parts:
- A1: footprint GeneralPurposeAlarmDevicePCB:Arduino_UNO_R3_NoMountingHoles3D -> GeneralPurposeAlarmDevicePCB:Arduino_UNO_R3_NoMountingHoles3D_Text_Top_&_Bottom
- J6, J9: footprint TerminalBlock_TE-Connectivity:TerminalBlock_TE_282834-6_1x06_P2.54mm_Horizontal -> GeneralPurposeAlarmDevicePCB:1x6P 20A -40℃~+105℃ 300V Green 12~30 Straight pin 5.08mm 2.5 1 6 Plugin,P=5.08mm Screw ter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
Changed lines of the file:
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@@
       (effects (font (size 1.27 1.27)) (justify left))
     )
-    (property "Footprint" "TerminalBlock_TE-Connectivity:TerminalBlock_TE_282834-6_1x06_P2.54mm_Horizontal" (at 203.2 128.27 0)
+    (property "Footprint" "GeneralPurposeAlarmDevicePCB:1x6P 20A -40℃~+105℃ 300V Green 12~30 Straight pin 5.08mm 2.5 1 6 Plugin,P=5.08mm Screw terminal ROHS" (at 203.2 128.27 0)
       (effects (font (size 1.27 1.27)) hide)
     )
@@
       (effects (font (size 1.27 1.27)) (justify right))
     )
-    (property "Footprint" "GeneralPurposeAlarmDevicePCB:Arduino_UNO_R3_NoMountingHoles3D" (at 86.36 77.47 0)
+    (property "Footprint" "GeneralPurposeAlarmDevicePCB:Arduino_UNO_R3_NoMountingHoles3D_Text_Top_&_Bottom" (at 86.36 77.47 0)
       (effects (font (size 1.27 1.27) italic) hide)
     )
@@
       (effects (font (size 1.27 1.27)) (justify left))
     )
-    (property "Footprint" "TerminalBlock_TE-Connectivity:TerminalBlock_TE_282834-6_1x06_P2.54mm_Horizontal" (at 151.13 130.81 0)
-      (effects (font (size 1.27 1.27)) hide)
-    )
+    (property "Footprint" "GeneralPurposeAlarmDevicePCB:1x6P 20A -40℃~+105℃ 300V Green 12~30 Straight pin 5.08mm 2.5 1 6 Plugin,P=5.08mm Screw terminal ROHS" (at 151.13 130.81 0)
+      (effects (font (size 1.27 1.27)) hide)
+    )

Commit message: Issue 70 completed: Add license info & open hardware & PI logo/symbols and related to schematic and PCB (Kicad)
Parts:
- added SM1: Logo_Open_Hardware_Small, GeneralPurposeAlarmDevicePCB:Logo_PI_BandW_70percent_10x10, symbol Graphic:Logo_Open_Hardware_Small
Other:
- note added: "MoonratII Controller Board"
- note added: "MoonratII Heater Board"
- note removed: "Controller Board"
- note removed: "Incubator Board"
- company: (none) -> PublicInvention

Commit message: Issue 53: Added key caps to switches in schematic
Parts:
- added MF102 (x3): CAP TACTILE ROUND IVORY, symbol GPAD_SCH_LIB:ENCLOSURE_GPAD_VER1
Changed lines of the file:
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@@
+    )
+  )
+  (symbol (lib_id "GPAD_SCH_LIB:ENCLOSURE_GPAD_VER1") (at 106.68 186.69 0) (unit 1)
+    (in_bom yes) (on_board no) (dnp no)
+    (property "Reference" "MF102" (at 102.87 175.26 0)
+      (effects (font (size 1.27 1.27)) (justify left))
+    )
+    (property "Value" "CAP TACTILE ROUND IVORY" (at 92.71 186.69 0)
+      (effects (font (size 1.27 1.27)) (justify left))
+    )
+    (property "Footprint" "" (at 106.68 186.69 0)
+      (effects (font (size 1.27 1.27)) hide)
+    )
+    (property "Datasheet" "https://omronfs.omron.com/en_US/ecb/products/pdf/en-b32.pdf" (at 106.68 186.69 0)
+      (effects (font (size 1.27 1.27)) hide)
+    )
+    (property "Distributor 1" "JCLPCB" (at 106.68 186.69 0)
+      (effects (font (size 1.27 1.27)) hide)
+    )
+    (property "Distributor 1 PN" "C231316" (at 106.68 186.69 0)
+      (effects (font (size 1.27 1.27)) hide)
+    )
+    (property "Cost" "1000000" (at 106.68 186.69 0)
+      (effects (font (size 1.27 1.27)) hide)
+    )
+    (instances
+      (project "GeneralPurposeAlarmDevicePCB"
+        (path "/412a327d-1ee3-473e-bc00-1545004b7edf"
+          (reference "MF102") (unit 1)
+        )
+      )
+      (project "moonratII"
+        (path "/9ef5effe-cb46-4a9a-bbbe-a65ab44b9e67"
+          (reference "MF2") (unit 1)
+        )
+      )
     )
   )
@@
     )
   )
+  (symbol (lib_id "GPAD_SCH_LIB:ENCLOSURE_GPAD_VER1") (at 140.97 186.69 0) (unit 1)
+    (in_bom yes) (on_board no) (dnp no)
+    (property "Reference" "MF102" (at 137.16 175.26 0)
+      (effects (font (size 1.27 1.27)) (justify left))
+    )
+    (property "Value" "CAP TACTILE ROUND IVORY" (at 127 186.69 0)
+      (effects (font (size 1.27 1.27)) (justify left))
+    )
+    (property "Footprint" "" (at 140.97 186.69 0)
+      (effects (font (size 1.27 1.27)) hide)
+    )
+    (property "Datasheet" "https://omronfs.omron.com/en_US/ecb/products/pdf/en-b32.pdf" (at 140.97 186.69 0)
+      (effects (font (size 1.27 1.27)) hide)
+    )
+    (property "Distributor 1" "JCLPCB" (at 140.97 186.69 0)
+      (effects (font (size 1.27 1.27)) hide)
+    )
+    (property "Distributor 1 PN" "C231316" (at 140.97 186.69 0)
+      (effects (font (size 1.27 1.27)) hide)
+    )
+    (property "Cost" "1000000" (at 140.97 186.69 0)
+      (effects (font (size 1.27 1.27)) hide)
+    )
+    (instances
+      (project "GeneralPurposeAlarmDevicePCB"
+        (path "/412a327d-1ee3-473e-bc00-1545004b7edf"
+          (reference "MF102") (unit 1)
+        )
+      )
+      (project "moonratII"
+        (path "/9ef5effe-cb46-4a9a-bbbe-a65ab44b9e67"
+          (reference "MF3") (unit 1)
+        )
+      )
+    )
+  )
   (symbol (lib_id "GPAD_SCH_LIB:MountingHole_Pad_3.5mm") (at 27.94 181.61 0) (unit 1)
     (in_bom yes) (on_board yes) (dnp no)
@@
         )
       )
+    )
+  )
+  (symbol (lib_id "GPAD_SCH_LIB:ENCLOSURE_GPAD_VER1") (at 72.39 186.69 0) (unit 1)
+    (in_bom yes) (on_board no) (dnp no)
+    (property "Reference" "MF102" (at 68.58 175.26 0)
+      (effects (font (size 1.27 1.27)) (justify left))
+    )
+    (property "Value" "CAP TACTILE ROUND IVORY" (at 58.42 186.69 0)
+      (effects (font (size 1.27 1.27)) (justify left))
+    )
+    (property "Footprint" "" (at 72.39 186.69 0)
+      (effects (font (size 1.27 1.27)) hide)
+    )
+    (property "Datasheet" "https://omronfs.omron.com/en_US/ecb/products/pdf/en-b32.pdf" (at 72.39 186.69 0)
+      (effects (font (size 1.27 1.27)) hide)
+    )
+    (property "Distributor 1" "JCLPCB" (at 72.39 186.69 0)
+      (effects (font (size 1.27 1.27)) hide)
+    )
+    (property "Distributor 1 PN" "C231316" (at 72.39 186.69 0)
+      (effects (font (size 1.27 1.27)) hide)
+    )
+    (property "Cost" "1000000" (at 72.39 186.69 0)
+      (effects (font (size 1.27 1.27)) hide)
+    )
+    (instances
+      (project "GeneralPurposeAlarmDevicePCB"
+        (path "/412a327d-1ee3-473e-bc00-1545004b7edf"
+          (reference "MF102") (unit 1)
+        )
+      )
+      (project "moonratII"
+        (path "/9ef5effe-cb46-4a9a-bbbe-a65ab44b9e67"
+          (reference "MF1") (unit 1)
+        )
+      )
