File: moonratII/moonratII/moonratII.kicad_sch (KiCad schematic)
At the start: 40 parts, among them J1 Barrel_Jack_Switch_SMT, J10 Conn_02x05_Odd_Even, J11 Screw_Terminal_01x02, J2 HS96L03W2C03_0.96_Oled, J5 Conn_02x05_Odd_Even, J6 Screw_Terminal_01x06, J9 Screw_Terminal_01x06, Q1 IRF520N, Q2 BSS138, SW1 6mm 2 Pin Tact NO Breadboard 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, SW2 6mm 2 Pin Tact NO Breadboard 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, SW3 6mm 2 Pin Tact NO Breadboard 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, U1 TMP36xS

Commit message: Issue 114: Corrected U1 footprint. Changed from SOIC-8 to SOT-23-5.
Parts:
- removed U1: TMP36xS, Package_SO:SOIC-8_3.9x4.9mm_P1.27mm, symbol Sensor_Temperature:TMP36xS
- added U1: TMP36GRTZ-REEL7, Package_TO_SOT_SMD:SOT-23-5, symbol GPAD_SCH_LIB:TMP36GRTZ-REEL7
- BZ1: value Buzzer_Adafruit_P1536A -> Buzzer_D12mm_H9.6mm_LS7.6mm; Cost .98 -> .16; Distributor 1 Adafruit -> JCLPCB; Distributor 1 PN P1536A -> C360615; Distributor 2 JCLPCB -> Adafruit; Distributor 2 PN PS1240P02BT -> P1536A; MPN PS1240P02BT -> P1536A; Manufacturer https://jlcpcb.com/partdetail/Tdk-PS1420P02CT/C91080 -> Adafruit
Connections:
- net +5P: now also U1.2 (+Vs)
- net GND1: now also U1.5 (V_{SS})
- net TempOut_IB: now also U1.1 (Vout)
- net at R7.1: now also U1.4 (/SHUTDOWN)
- no-connect marks 48 -> 49
Changed lines of the file:
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@@
   (title_block
     (title "MoonratII")
-    (date "2023-06-21")
-    (rev "0.1")
+    (date "2023-11-15")
+    (rev "1.0")
     (company "PublicInvention")
     (comment 1 "GNU Affero General Public License v3.0")
@@
   (no_connect (at 248.92 67.31))
   (no_connect (at 261.62 62.23))
+  (no_connect (at 233.68 133.35))
   (no_connect (at 196.85 58.42))
   (no_connect (at 261.62 59.69))
@@
     (stroke (width 0) (type default))
   )
-  (wire (pts (xy 243.84 121.92) (xy 243.84 119.38))
+  (wire (pts (xy 243.84 119.38) (xy 243.84 123.19))
     (stroke (width 0) (type default))
   )
@@
     (stroke (width 0) (type default))
   )
-  (wire (pts (xy 228.6 132.08) (xy 228.6 119.38))
+  (wire (pts (xy 228.6 130.81) (xy 228.6 119.38))
     (stroke (width 0) (type default))
   )
@@
     (stroke (width 0) (type default))
   )
-  (wire (pts (xy 256.54 132.08) (xy 257.81 132.08))
+  (wire (pts (xy 257.81 128.27) (xy 254 128.27))
     (stroke (width 0) (type default))
   )
@@
     (stroke (width 0) (type default))
   )
-  (wire (pts (xy 243.84 142.24) (xy 243.84 144.78))
+  (wire (pts (xy 243.84 138.43) (xy 243.84 144.78))
     (stroke (width 0) (type default))
   )
@@
     (stroke (width 0) (type default))
   )
-  (wire (pts (xy 231.14 132.08) (xy 228.6 132.08))
+  (wire (pts (xy 228.6 130.81) (xy 233.68 130.81))
     (stroke (width 0) (type default))
   )
@@
     (stroke (width 0) (type default))
   )
-  (wire (pts (xy 257.81 132.08) (xy 257.81 148.59))
+  (wire (pts (xy 257.81 128.27) (xy 257.81 148.59))
     (stroke (width 0) (type default))
   )
@@
     )
   )
-  (symbol (lib_id "Sensor_Temperature:TMP36xS") (at 243.84 132.08 0) (unit 1)
-    (in_bom yes) (on_board yes) (dnp no) (fields_autoplaced)
-    (property "Reference" "U1" (at 259.08 127.7493 0)
-      (effects (font (size 1.27 1.27)))
-    )
-    (property "Value" "TMP36xS" (at 259.08 130.2893 0)
-      (effects (font (size 1.27 1.27)))
-    )
-    (property "Footprint" "Package_SO:SOIC-8_3.9x4.9mm_P1.27mm" (at 243.84 143.51 0)
-      (effects (font (size 1.27 1.27)) hide)
-    )
-    (property "Datasheet" "https://www.analog.com/media/en/technical-documentation/data-sheets/TMP35_36_37.pdf" (at 243.84 132.08 0)
-      (effects (font (size 1.27 1.27)) hide)
-    )
-    (property "AssemblyType" "SMT" (at 243.84 132.08 0)
-      (effects (font (size 1.27 1.27)) hide)
-    )
-    (property "Distributor 1" "JLCPCB" (at 243.84 132.08 0)
-      (effects (font (size 1.27 1.27)) hide)
-    )
-    (property "Distributor 1 PN" "C129489" (at 243.84 132.08 0)
-      (effects (font (size 1.27 1.27)) hide)
-    )
-    (property "MPN" "TMP36GRTZ" (at 243.84 132.08 0)
-      (effects (font (size 1.27 1.27)) hide)
-    )
-    (property "Manufacturer" "Analog Devices" (at 243.84 132.08 0)
-      (effects (font (size 1.27 1.27)) hide)
-    )
-    (property "Cost" "1.297" (at 243.84 132.08 0)
-      (effects (font (size 1.27 1.27)) hide)
-    )
-    (property "Description" "TMP36GRTZ SOT-23-5 Temperature Sensors ROHS" (at 243.84 132.08 0)
-      (effects (font (size 1.27 1.27)) hide)
-    )
-    (pin "1")
-    (pin "4")
-    (pin "5")
-    (pin "8")
-    (instances
-      (project "moonratII"
-        (path "/9ef5effe-cb46-4a9a-bbbe-a65ab44b9e67"
-          (reference "U1") (unit 1)
-        )
-      )
-    )
-  )
   (symbol (lib_id "Graphic:Logo_Open_Hardware_Small") (at 240.03 179.07 0) (unit 1)
     (in_bom no) (on_board no) (dnp no) (fields_autoplaced)
@@
       (effects (font (size 1.27 1.27)) (justify left))
     )
-    (property "Value" "Buzzer_Adafruit_P1536A" (at 144.78 102.87 0)
+    (property "Value" "Buzzer_D12mm_H9.6mm_LS7.6mm" (at 144.78 102.87 0)
       (effects (font (size 1.27 1.27)) (justify left))
     )
@@
       (effects (font (size 1.27 1.27)) hide)
     )
-    (property "Datasheet" "https://www.adafruit.com/product/1536" (at 168.275 100.33 90)
+    (property "Datasheet" "https://jlcpcb.com/partdetail/ss-SUN_12095_5VPA76/C360615" (at 168.275 100.33 90)
       (effects (font (size 1.27 1.27)) hide)
     )
-    (property "Distributor 2" "JCLPCB" (at 168.91 102.87 0)
+    (property "Distributor 2" "Adafruit" (at 168.91 102.87 0)
       (effects (font (size 1.27 1.27)) hide)
     )
-    (property "Distributor 2 PN" "PS1240P02BT" (at 168.91 102.87 0)
+    (property "Distributor 2 PN" "P1536A" (at 168.91 102.87 0)
       (effects (font (size 1.27 1.27)) hide)
     )
-    (property "Manufacturer" "https://jlcpcb.com/partdetail/Tdk-PS1420P02CT/C91080" (at 168.91 102.87 0)
+    (property "Manufacturer" "Adafruit" (at 168.91 102.87 0)
       (effects (font (size 1.27 1.27)) hide)
     )
-    (property "MPN" "PS1240P02BT" (at 168.91 102.87 0)
+    (property "MPN" "P1536A" (at 168.91 102.87 0)
       (effects (font (size 1.27 1.27)) hide)
     )
-    (property "Distributor 1" "Adafruit" (at 168.91 102.87 0)
+    (property "Distributor 1" "JCLPCB" (at 168.91 102.87 0)
       (effects (font (size 1.27 1.27)) hide)
     )
-    (property "Distributor 1 PN" "P1536A" (at 168.91 102.87 0)
+    (property "Distributor 1 PN" "C360615" (at 168.91 102.87 0)
       (effects (font (size 1.27 1.27)) hide)
     )
-    (property "Cost" ".98" (at 168.91 102.87 0)
+    (property "Cost" ".16" (at 168.91 102.87 0)
       (effects (font (size 1.27 1.27)) hide)
     )
@@
         )
       )
+    )
+  )
+  (symbol (lib_id "GPAD_SCH_LIB:TMP36GRTZ-REEL7") (at 243.84 130.81 0) (unit 1)
+    (in_bom yes) (on_board yes) (dnp no) (fields_autoplaced)
+    (property "Reference" "U1" (at 261.62 124.6221 0)
+      (effects (font (size 1.27 1.27)))
+    )
+    (property "Value" "TMP36GRTZ-REEL7" (at 261.62 127.1621 0)
+      (effects (font (size 1.27 1.27)))
+    )
+    (property "Footprint" "Package_TO_SOT_SMD:SOT-23-5" (at 245.11 137.16 0)
+      (effects (font (size 1.27 1.27)) (justify left) hide)
+    )
+    (property "Datasheet" "https://www.analog.com/media/en/technical-documentation/data-sheets/TMP35_36_37.pdf" (at 245.11 130.81 0)
+      (effects (font (size 1.27 1.27)) hide)
+    )
+    (pin "1")
+    (pin "2")
+    (pin "3")
+    (pin "4")
+    (pin "5")
+    (instances
+      (project "moonratII"
+        (path "/9ef5effe-cb46-4a9a-bbbe-a65ab44b9e67"
+          (reference "U1") (unit 1)
+        )
+      )
