File: moonratII/moonratII/moonratII.kicad_sch (KiCad schematic)
At the start: 40 parts, among them J1 Barrel_Jack_Switch_SMT, J10 Conn_02x05_Odd_Even, J11 Screw_Terminal_01x02, J2 HS96L03W2C03_0.96_Oled, J5 Conn_02x05_Odd_Even, J6 Screw_Terminal_01x06, J9 Screw_Terminal_01x06, Q1 IRF520N, Q2 BSS138, SW1 6mm 2 Pin Tact NO Breadboard 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, SW2 6mm 2 Pin Tact NO Breadboard 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, SW3 6mm 2 Pin Tact NO Breadboard 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, U1 TMP36GRTZ-REEL7

Commit message: Updated the footprint to the OLED
Parts:
- J2: footprint GeneralPurposeAlarmDevicePCB:HS96L03W2C03_0.96_Oled -> GeneralPurposeAlarmDevicePCB:OLED_HS96L03W2C03_0.96_WithNuts
Changed lines of the file:
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@@
       (effects (font (size 1.27 1.27)))
     )
-    (property "Footprint" "GeneralPurposeAlarmDevicePCB:HS96L03W2C03_0.96_Oled" (at 30.48 101.6 0)
+    (property "Footprint" "GeneralPurposeAlarmDevicePCB:OLED_HS96L03W2C03_0.96_WithNuts" (at 30.48 101.6 0)
       (effects (font (size 1.27 1.27)) hide)
     )

Commit message: Updated JLCPCB BOM and CPL files for PCB order
Parts:
- removed MF102 (x2): CAP TACTILE ROUND IVORY, symbol GPAD_SCH_LIB:ENCLOSURE_GPAD_VER1
- added MF102 (x4): SMD_round_nut_M2*4*5+1.5, See JLCPCB assembly notes for footprint, symbol GPAD_SCH_LIB:ENCLOSURE_GPAD_VER1
- added MF102 (x2): CAP TACTILE ROUND IVORY, See JLCPCB assembly notes for footprint, symbol GPAD_SCH_LIB:ENCLOSURE_GPAD_VER1
- added MF102 (x4): Steel Pan Head Phillips Screw M2 x 0.4 mm Thread,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, symbol GPAD_SCH_LIB:ENCLOSURE_GPAD_VER1
- added MF102: 250V 3A Straight Square Pins 2.5mm 4P 6mm -40℃~+1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, See JLCPCB assembly notes for footprint, symbol GPAD_SCH_LIB:ENCLOSURE_GPAD_VER1
- BZ1: Distributor 1 JCLPCB -> JLCPCB
- MF102: footprint (none) -> See JLCPCB assembly notes for footprint; Cost 1000000 -> 0.3475; Distributor 1 JCLPCB -> JLCPCB
- U1: Cost (none) -> 1.2837; Distributor 1 (none) -> JLCPCB; Distributor 1 PN (none) -> C129489

Commit message: Updated all related files and ordered PCB and Assemblies through JLCPBC.
Parts:
- MF102: footprint See JLCPCB assembly notes for footprint -> TH162050CTJ
- MF102: footprint See JLCPCB assembly notes for footprint -> B32-1600
- MF102: footprint See JLCPCB assembly notes for footprint -> PZ254V-11-04P
Changed lines of the file:
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@@
       (effects (font (size 1.27 1.27)) (justify left))
     )
-    (property "Footprint" "See JLCPCB assembly notes for footprint" (at -21.59 173.99 0)
+    (property "Footprint" "TH162050CTJ" (at -21.59 173.99 0)
       (effects (font (size 1.27 1.27)) hide)
     )
@@
       (effects (font (size 1.27 1.27)) (justify left))
     )
-    (property "Footprint" "See JLCPCB assembly notes for footprint" (at 105.41 186.69 0)
+    (property "Footprint" "B32-1600" (at 105.41 186.69 0)
       (effects (font (size 1.27 1.27)) hide)
     )
@@
       (effects (font (size 1.27 1.27)) (justify left))
     )
-    (property "Footprint" "See JLCPCB assembly notes for footprint" (at -22.86 203.2 0)
+    (property "Footprint" "TH162050CTJ" (at -22.86 203.2 0)
       (effects (font (size 1.27 1.27)) hide)
     )
@@
       (effects (font (size 1.27 1.27)) (justify left))
     )
-    (property "Footprint" "See JLCPCB assembly notes for footprint" (at -50.8 111.76 0)
+    (property "Footprint" "PZ254V-11-04P" (at -50.8 111.76 0)
       (effects (font (size 1.27 1.27)) hide)
     )
@@
       (effects (font (size 1.27 1.27)) (justify left))
     )
-    (property "Footprint" "See JLCPCB assembly notes for footprint" (at -57.15 203.2 0)
+    (property "Footprint" "TH162050CTJ" (at -57.15 203.2 0)
       (effects (font (size 1.27 1.27)) hide)
     )
@@
       (effects (font (size 1.27 1.27)) (justify left))
     )
-    (property "Footprint" "See JLCPCB assembly notes for footprint" (at -55.88 173.99 0)
+    (property "Footprint" "TH162050CTJ" (at -55.88 173.99 0)
       (effects (font (size 1.27 1.27)) hide)
     )
@@
       (effects (font (size 1.27 1.27)) (justify left))
     )
-    (property "Footprint" "See JLCPCB assembly notes for footprint" (at 139.7 186.69 0)
+    (property "Footprint" "B32-1600" (at 139.7 186.69 0)
       (effects (font (size 1.27 1.27)) hide)
     )
@@
       (effects (font (size 1.27 1.27)) (justify left))
     )
-    (property "Footprint" "See JLCPCB assembly notes for footprint" (at 72.39 186.69 0)
-      (effects (font (size 1.27 1.27)) hide)
-    )
+    (property "Footprint" "B32-1600" (at 72.39 186.69 0)
+      (effects (font (size 1.27 1.27)) hide)
+    )

Commit message: Changed connector part number due to availability
Parts:
- BZ1: Cost .16 -> 0.16
- Cable_MoldedFemale1: Cost 17.99 -> 7.00; Distributor 1 PN https://www.amazon.com/807-Connectors-Extension-Connector-W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 -> Female 1/2 of connector https://www.amazon.com/CARROFIX-Tra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
- Cable_MoldedMale1: Cost 16.99 -> 7.00; Distributor 1 PN https://www.amazon.com/807-Connectors-Extension-Connector-W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 -> Male 1/2 of connector https://www.amazon.com/CARROFIX-Trail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
- Cable_Ribbon1: Cost 3.25 -> 6.75

Commit message: Added the buzzer dimensions to mechanical drawing issue 141
Parts:
- J6: Distributor 1 PN C2915642 -> C474924; MPN DB128V-5.08-6P-GN-S -> KF128-2.54-6P; Manufacturer DIBO -> Cixi Kefa Elec
- J9: Distributor 1 PN C2915642 -> C474924
Changed lines of the file:
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@@
       (effects (font (size 1.27 1.27)) hide)
     )
-    (property "Distributor 1 PN" "C2915642" (at 203.2 128.27 0)
+    (property "Distributor 1 PN" "C474924" (at 203.2 128.27 0)
       (effects (font (size 1.27 1.27)) hide)
     )
@@
       (effects (font (size 1.27 1.27)) hide)
     )
-    (property "Datasheet" "DB128V-5.08-6P-GN-S.pdf" (at 151.13 130.81 0)
+    (property "Datasheet" "https://jlcpcb.com/partdetail/Cixi_KefaElec-KF128_2_546P/C474924" (at 151.13 130.81 0)
       (effects (font (size 1.27 1.27)) hide)
     )
@@
       (effects (font (size 1.27 1.27)) hide)
     )
-    (property "Description" "1x6P 20A -40℃~+105℃ 300V Green 12~30 Straight pin 5.08mm 2.5 1 6 Plugin,P=5.08mm Screw terminal ROHS" (at 151.13 130.81 0)
+    (property "Description" "1x6P -40℃~+105℃ 8A 130V Green 18~26 Straight 2.54mm 1 1 6 Plugin,P=2.54mm Screw terminal ROHS" (at 151.13 130.81 0)
       (effects (font (size 1.27 1.27)) hide)
     )
@@
       (effects (font (size 1.27 1.27)) hide)
     )
-    (property "Distributor 1 PN" "C2915642" (at 151.13 130.81 0)
-      (effects (font (size 1.27 1.27)) hide)
-    )
-    (property "MPN" "DB128V-5.08-6P-GN-S" (at 151.13 130.81 0)
-      (effects (font (size 1.27 1.27)) hide)
-    )
-    (property "Manufacturer" "DIBO" (at 151.13 130.81 0)
-      (effects (font (size 1.27 1.27)) hide)
-    )
+    (property "Distributor 1 PN" "C474924" (at 151.13 130.81 0)
+      (effects (font (size 1.27 1.27)) hide)
+    )
+    (property "MPN" "KF128-2.54-6P" (at 151.13 130.81 0)
+      (effects (font (size 1.27 1.27)) hide)
+    )
+    (property "Manufacturer" "Cixi Kefa Elec" (at 151.13 130.81 0)
+      (effects (font (size 1.27 1.27)) hide)
+    )

Commit message: Add README.md file
Parts:
- J9: MPN DB128V-5.08-6P-GN-S -> KF128-2.54-6P; Manufacturer DIBO -> Cixi Kefa Elec
Changed lines of the file:
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@@
       (effects (font (size 1.27 1.27)) hide)
     )
-    (property "Datasheet" "DB128V-5.08-6P-GN-S.pdf" (at 203.2 128.27 0)
+    (property "Datasheet" "https://jlcpcb.com/partdetail/Cixi_KefaElec-KF128_2_546P/C474924" (at 203.2 128.27 0)
       (effects (font (size 1.27 1.27)) hide)
     )
@@
       (effects (font (size 1.27 1.27)) hide)
     )
-    (property "Description" "1x6P 20A -40℃~+105℃ 300V Green 12~30 Straight pin 5.08mm 2.5 1 6 Plugin,P=5.08mm Screw terminal ROHS" (at 203.2 128.27 0)
+    (property "Description" "1x6P -40℃~+105℃ 8A 130V Green 18~26 Straight 2.54mm 1 1 6 Plugin,P=2.54mm Screw terminal ROHS" (at 203.2 128.27 0)
       (effects (font (size 1.27 1.27)) hide)
     )
@@
       (effects (font (size 1.27 1.27)) hide)
     )
-    (property "MPN" "DB128V-5.08-6P-GN-S" (at 203.2 128.27 0)
+    (property "MPN" "KF128-2.54-6P" (at 203.2 128.27 0)
       (effects (font (size 1.27 1.27)) hide)
     )
-    (property "Manufacturer" "DIBO" (at 203.2 128.27 0)
+    (property "Manufacturer" "Cixi Kefa Elec" (at 203.2 128.27 0)
       (effects (font (size 1.27 1.27)) hide)
     )
