File: moonratII/moonratII/moonratII.kicad_pcb (KiCad board)
At the start: 2 copper layers, 10 parts, among them Q101 IRF540N, SW101 6mm 2 Pin Tact NO, SW102 6mm 2 Pin Tact NO, SW103 6mm 2 Pin Tact NO, U101 TMP36xS

Commit message: Pull in parts to PCB. Make some initial placement.
Parts:
- removed A101: Arduino_UNO_R3, Module:Arduino_UNO_R3
- removed Q101: IRF540N, Package_TO_SOT_THT:TO-220-3_Vertical
- removed R101: 1R, Resistor_SMD:R_0603_1608Metric_Pad0.98x0.95mm_HandSolder
- removed R103, R104, R105: 1K, Resistor_SMD:R_0603_1608Metric_Pad0.98x0.95mm_HandSolder
- removed SW101, SW102, SW103: 6mm 2 Pin Tact NO, Button_Switch_THT:SW_PUSH_6mm
- removed U101: TMP36xS, Package_SO:SOIC-8_3.9x4.9mm_P1.27mm
- added A1: Arduino_UNO_R3, Module:Arduino_UNO_R3, F.Cu at (136.3, 68.2)
- added BZ1: Buzzer_Adafruit_P1536A, GeneralPurposeAlarmDevicePCB:Buzzer_12.2mm_9.7mm_7.62mm, F.Cu at (112.1, 111.8)
- added D2: Schottky 2A, Diode_SMD:D_SMB, F.Cu at (208.0, 67.6)
- added J1: Barrel_Jack_Switch_SMT, GeneralPurposeAlarmDevicePCB:BarrelJack_CLIFF_FC681465S_SMT_Horizontal, F.Cu at (117.2, 73.2)
- added J3: Conn_02x05_Odd_Even, Connector_PinHeader_2.54mm:PinHeader_2x05_P2.54mm_Vertical, F.Cu at (163.1, 72.9)
- added J4: Screw_Terminal_01x06, TerminalBlock_TE-Connectivity:TerminalBlock_TE_282834-6_1x06_P2.54mm_Horizontal, F.Cu at (172.0, 85.2)
- added J5: Screw_Terminal_01x06, TerminalBlock_TE-Connectivity:TerminalBlock_TE_282834-6_1x06_P2.54mm_Horizontal, F.Cu at (190.2, 79.2)
- added J6: Conn_02x05_Odd_Even, Connector_PinHeader_2.54mm:PinHeader_2x05_P2.54mm_Vertical, F.Cu at (197.8, 67.2)
- added J7: Screw_Terminal_01x02, TerminalBlock_4Ucon:TerminalBlock_4Ucon_1x02_P3.50mm_Horizontal, F.Cu at (212.3, 78.0)
- added Q1: IRF520N, Package_TO_SOT_THT:TO-220-3_Vertical, F.Cu at (162.5, 96.9)
- added Q2: BSS138, Package_TO_SOT_SMD:SOT-23, F.Cu at (144.2, 112.4)
- added R1: 1R, Resistor_SMD:R_0603_1608Metric_Pad0.98x0.95mm_HandSolder, F.Cu at (127.6, 67.8)
- added R2: 1R, Resistor_SMD:R_0603_1608Metric_Pad0.98x0.95mm_HandSolder, F.Cu at (159.2, 71.8)
- added R3: 1K, Resistor_SMD:R_0603_1608Metric_Pad0.98x0.95mm_HandSolder, F.Cu at (159.2, 112.6)
- added R4: 1K, Resistor_SMD:R_0603_1608Metric_Pad0.98x0.95mm_HandSolder, F.Cu at (156.6, 112.6)
- added R5: 1K, Resistor_SMD:R_0603_1608Metric_Pad0.98x0.95mm_HandSolder, F.Cu at (154.0, 112.6)
- added R6: 1K, Resistor_SMD:R_0603_1608Metric_Pad0.98x0.95mm_HandSolder, F.Cu at (147.4, 113.0)
- added R7: 1R, Resistor_SMD:R_0603_1608Metric_Pad0.98x0.95mm_HandSolder, F.Cu at (211.6, 90.2)
- added R9: 1K, Resistor_SMD:R_0603_1608Metric_Pad0.98x0.95mm_HandSolder, F.Cu at (150.4, 113.0)
- added SW1: 6mm 2 Pin Tact NO Breadboard Friendly, Button_Switch_THT:SW_PUSH_6mm, F.Cu at (147.4, 107.4)
- added SW2: 6mm 2 Pin Tact NO Breadboard Friendly, Button_Switch_THT:SW_PUSH_6mm, F.Cu at (135.4, 107.6)
- added SW3: 6mm 2 Pin Tact NO Breadboard Friendly, Button_Switch_THT:SW_PUSH_6mm, F.Cu at (125.4, 107.8)
- added TP1: TP_GND, TestPoint:TestPoint_Loop_D2.54mm_Drill1.5mm_Beaded, F.Cu at (174.4, 91.2)
- added U1: TMP36xS, Package_SO:SOIC-8_3.9x4.9mm_P1.27mm, F.Cu at (211.8, 85.2)
Other:
- board outline added: 162.8 x 65.8 mm

Commit message: Add remaning new footprint files, add parts files.
Parts:
- moved R7 35.9 mm to (175.8, 88.2), turned to 90 degrees
- moved J7 28.4 mm to (189.8, 95.3), turned to 0 degrees
- moved D2 26.9 mm to (187.5, 85.0), turned to -90 degrees
- moved U1 15.3 mm to (196.6, 85.0), turned to -90 degrees
- moved J5 13.2 mm to (185.5, 66.8), turned to 0 degrees
- moved J6 7.21 mm to (197.5, 74.4), turned to -90 degrees
- moved TP1 1.80 mm to (174.4, 93.0)
Other:
- board size 162.8 x 65.8 mm -> 97.4 x 65.6 mm

Commit message: Add more PCB 3D models. Place and lock down mounting holes.
Parts:
- removed D2: Schottky 2A, Diode_SMD:D_SMB
- removed R9: 1K, Resistor_SMD:R_0603_1608Metric_Pad0.98x0.95mm_HandSolder
- added D1: Schottky 2A, Diode_SMD:D_SMB, F.Cu at (188.4, 95.0)
- added F1: Polyfuse 6A, GeneralPurposeAlarmDevicePCB:PlaceHolderOpossum, F.Cu at (76.6, 92.8)
- added H1: MountingHole_Pad_3.5mm, GeneralPurposeAlarmDevicePCB:MountingHole_3.5mm_Pad_Via, F.Cu at (104.0, 64.0)
- added H2: MountingHole_Pad_3.5mm, GeneralPurposeAlarmDevicePCB:MountingHole_3.5mm_Pad_Via, F.Cu at (104.0, 121.0)
- added H3: MountingHole_Pad_3.5mm, GeneralPurposeAlarmDevicePCB:MountingHole_3.5mm_Pad_Via, F.Cu at (178.0, 121.0)
- added H4: MountingHole_Pad_3.5mm, GeneralPurposeAlarmDevicePCB:MountingHole_3.5mm_Pad_Via, F.Cu at (178.0, 64.0)
- added H5: MountingHole_Pad_3.5mm, GeneralPurposeAlarmDevicePCB:MountingHole_3.5mm_Pad_Via, F.Cu at (192.0, 64.0)
- added H6: MountingHole_Pad_3.5mm, GeneralPurposeAlarmDevicePCB:MountingHole_3.5mm_Pad_Via, F.Cu at (192.0, 121.0)
- added J10: Conn_02x05_Odd_Even, Connector_PinHeader_2.54mm:PinHeader_2x05_P2.54mm_Vertical, F.Cu at (196.9, 82.1)
- added J11: Screw_Terminal_01x02, TerminalBlock_TE-Connectivity:TerminalBlock_TE_282834-2_1x02_P2.54mm_Horizontal, F.Cu at (192.8, 104.2)
- added J2: SSD1306 OLED, Display:Adafruit_SSD1306, F.Cu at (134.8, 63.4)
- added J2: SSD1306 OLED, Connector_PinHeader_2.54mm:PinHeader_1x08_P2.54mm_Vertical, F.Cu at (139.7, 63.2)
- added J8: PinHeader_1x10_P2.54mm_Vertical, Connector_PinHeader_2.54mm:PinHeader_1x10_P2.54mm_Vertical, B.Cu at (129.0, 68.0)
- added J9: Screw_Terminal_01x06, TerminalBlock_TE-Connectivity:TerminalBlock_TE_282834-6_1x06_P2.54mm_Horizontal, F.Cu at (185.2, 74.6)
- added TP2: TP_GND, TestPoint:TestPoint_Loop_D2.54mm_Drill1.5mm_Beaded, F.Cu at (197.0, 116.0)
- A1: footprint Module:Arduino_UNO_R3 -> GeneralPurposeAlarmDevicePCB:Arduino_UNO_R3_NoMountingHoles3D; moved to B.Cu
- J3: value Conn_02x05_Odd_Even -> PinHeader_1x06_P2.54mm_Vertical; footprint Connector_PinHeader_2.54mm:PinHeader_2x05_P2.54mm_Vertical -> Connector_PinHeader_2.54mm:PinHeader_1x06_P2.54mm_Vertical; moved to B.Cu
- J4: value Screw_Terminal_01x06 -> PinHeader_1x08_P2.54mm_Vertical; footprint TerminalBlock_TE-Connectivity:TerminalBlock_TE_282834-6_1x06_P2.54mm_Horizontal -> Connector_PinHeader_2.54mm:PinHeader_1x08_P2.54mm_Vertical; moved to B.Cu
- J5: value Screw_Terminal_01x06 -> Conn_02x05_Odd_Even; footprint TerminalBlock_TE-Connectivity:TerminalBlock_TE_282834-6_1x06_P2.54mm_Horizontal -> Connector_PinHeader_2.54mm:PinHeader_2x05_P2.54mm_Vertical
- J6: value Conn_02x05_Odd_Even -> Screw_Terminal_01x06; footprint Connector_PinHeader_2.54mm:PinHeader_2x05_P2.54mm_Vertical -> TerminalBlock_TE-Connectivity:TerminalBlock_TE_282834-6_1x06_P2.54mm_Horizontal
- J7: value Screw_Terminal_01x02 -> PinHeader_1x08_P2.54mm_Vertical; footprint TerminalBlock_4Ucon:TerminalBlock_4Ucon_1x02_P3.50mm_Horizontal -> Connector_PinHeader_2.54mm:PinHeader_1x08_P2.54mm_Vertical; moved to B.Cu
- R2: value 1R -> 1K
- moved R1 53.5 mm to (161.0, 109.6), turned to 90 degrees
- moved A1 48.2 mm to (138.2, 116.3)
- moved J4 46.0 mm to (138.2, 116.3), turned to -90 degrees
- moved J3 43.5 mm to (161.0, 116.4), turned to -90 degrees
- moved J7 43.4 mm to (156.0, 68.2), turned to -90 degrees
- moved J5 33.3 mm to (176.5, 98.9)
- moved J6 20.3 mm to (177.2, 72.8)
- moved BZ1 16.8 mm to (107.5, 95.6)
- moved Q1 13.9 mm to (165.9, 110.3), turned to 0 degrees
- moved J1 13.4 mm to (104.7, 77.8)
- moved U1 9.81 mm to (196.2, 94.8)
- moved TP1 3.65 mm to (178.0, 93.6)
Connections:
- J1 pad 1: Net-(J1-Pad1) -> Net-(F1-Pad2)
- J1 pad 4: Net-(J1-Pad1) -> Net-(F1-Pad2)
- J3 pad 1: HeaterDrive -> (no net)
- J3 pad 2: GND -> (no net)
- J3 pad 3: +5V -> (no net)
- J3 pad 4: TempOut -> (no net)
- J3 pad 5: VCC -> (no net)
- J3 pad 6: VCC -> (no net)
- J4 pad 1: GND -> (no net)
- J4 pad 2: VCC -> (no net)
- J4 pad 3: HeaterDrive -> (no net)
- J4 pad 4: +5V -> (no net)
- J4 pad 5: TempOut -> (no net)
- J4 pad 6: GND -> (no net)
- J5 pad 1: GND -> HeaterDrive
- J5 pad 2: VCC -> GND
- J5 pad 3: HeaterDrive -> +5V
- J5 pad 4: +5V -> TempOut
- J5 pad 5: TempOut -> VCC
- J5 pad 6: GND -> VCC
- J6 pad 1: HeaterDrive -> GND
- J6 pad 2: GND -> VCC
- J6 pad 3: +5V -> HeaterDrive
- J6 pad 4: TempOut -> +5V
- J6 pad 5: VCC -> TempOut
- J6 pad 6: VCC -> GND
- J7 pad 1: VCC -> (no net)
- J7 pad 2: Net-(D2-Pad2) -> (no net)
- R1 pad 1: Net-(J1-Pad1) -> TEMP_IN
- R1 pad 2: VCC -> TempOut
- R2 pad 1: TEMP_IN -> HEATER_ON
- R2 pad 2: TempOut -> Net-(A1-Pad23)
- SW1 pad 1: BTN_SELECT -> BTN_DOWN
- SW1 pad 2: BTN_SELECT -> BTN_DOWN
- SW2 pad 1: BTN_UP -> BTN_SELECT
- SW2 pad 2: BTN_UP -> BTN_SELECT
- SW3 pad 1: BTN_DOWN -> BTN_UP
- SW3 pad 2: BTN_DOWN -> BTN_UP
Other:
- board size 97.4 x 65.6 mm -> 100 x 65 mm

Commit message: Add OLED display files.
Parts:
- moved J2 11.2 mm to (135.0, 74.6)
Changed lines of the file:
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@@
       (effects (font (size 1 1) (thickness 0.15)))
     )
-    (fp_text value "MountingHole_Pad_3.5mm" (at 0 4.5) (layer "F.Fab")
+    (fp_text value "MountingHole_Pad_3.5mm" (at 13.4 2.6) (layer "F.Fab")
       (effects (font (size 1 1) (thickness 0.15)))
     )
@@
   )
   (footprint "Display:Adafruit_SSD1306" (layer "F.Cu")
-    (at 134.8 63.4)
+    (at 135 74.6)
     (descr "Adafruit SSD1306 OLED 1.3 inch 128x64 I2C & SPI https://learn.adafruit.com/monochrome-oled-breakouts/downloads")
     (tags "Adafruit SSD1306 OLED 1.3 inch 128x64 I2C & SPI ")
@@
     (pad "8" thru_hole circle (at 17.78 0) (size 1.7 1.7) (drill 1) (layers *.Cu *.Mask)
       (net 6 "GND") (pinfunction "Pin_8") (pintype "passive"))
-    (model "${KICAD6_3DMODEL_DIR}/Display.3dshapes/Adafruit_SSD1306.wrl"
-      (offset (xyz 0 0 2.5))
+    (model "${KIPRJMOD}/parts/SSD1306_OLED_Display(128x64).step"
+      (offset (xyz 9 -12 2.5))
       (scale (xyz 1 1 1))
       (rotate (xyz 0 0 0))
@@
   (gr_line (start 100 60) (end 100 125) (layer "Edge.Cuts") (width 0.1))
   (gr_line (start 200 125) (end 200 60) (layer "Edge.Cuts") (width 0.1))
+  (dimension (type aligned) (layer "Dwgs.User")
+    (pts (xy 200 125) (xy 200 60))
+    (height 52.4)
+    (gr_text "65.0000 mm" (at 251.25 92.5 90) (layer "Dwgs.User")
+      (effects (font (size 1 1) (thickness 0.15)))
+    )
+    (format (units 3) (units_format 1) (precision 4))
+    (style (thickness 0.15) (arrow_length 1.27) (text_position_mode 0) (extension_height 0.58642) (extension_offset 0.5) keep_text_aligned)
+  )
+  (dimension (type aligned) (layer "Dwgs.User")
+    (pts (xy 192 121) (xy 192 125))
+    (height -13.6)
+    (gr_text "4.0000 mm" (at 204.45 123 90) (layer "Dwgs.User")
+      (effects (font (size 1 1) (thickness 0.15)))
+    )
+    (format (units 3) (units_format 1) (precision 4))
+    (style (thickness 0.15) (arrow_length 1.27) (text_position_mode 0) (extension_height 0.58642) (extension_offset 0.5) keep_text_aligned)
+  )
+  (dimension (type aligned) (layer "Dwgs.User")
+    (pts (xy 104 64) (xy 104 125))
+    (height 49)
+    (gr_text "61.0000 mm" (at 53.85 94.5 90) (layer "Dwgs.User")
+      (effects (font (size 1 1) (thickness 0.15)))
+    )
+    (format (units 3) (units_format 1) (precision 4))
+    (style (thickness 0.15) (arrow_length 1.27) (text_position_mode 0) (extension_height 0.58642) (extension_offset 0.5) keep_text_aligned)
+  )
+  (dimension (type aligned) (layer "Dwgs.User")
+    (pts (xy 192 121) (xy 100 121))
+    (height -23.2)
+    (gr_text "92.0000 mm" (at 146 143.05) (layer "Dwgs.User")
+      (effects (font (size 1 1) (thickness 0.15)))
+    )
+    (format (units 3) (units_format 1) (precision 4))
+    (style (thickness 0.15) (arrow_length 1.27) (text_position_mode 0) (extension_height 0.58642) (extension_offset 0.5) keep_text_aligned)
+  )
+  (dimension (type aligned) (layer "Dwgs.User")
+    (pts (xy 104 121) (xy 104 125))
+    (height 7.2)
+    (gr_text "4.0000 mm" (at 95.65 123 90) (layer "Dwgs.User")
+      (effects (font (size 1 1) (thickness 0.15)))
+    )
+    (format (units 3) (units_format 1) (precision 4))
+    (style (thickness 0.15) (arrow_length 1.27) (text_position_mode 0) (extension_height 0.58642) (extension_offset 0.5) keep_text_aligned)
+  )
+  (dimension (type aligned) (layer "Dwgs.User")
+    (pts (xy 192 64) (xy 192 60))
+    (height 13.6)
+    (gr_text "4.0000 mm" (at 204.45 62 90) (layer "Dwgs.User")
+      (effects (font (size 1 1) (thickness 0.15)))
+    )
+    (format (units 3) (units_format 1) (precision 4))
+    (style (thickness 0.15) (arrow_length 1.27) (text_position_mode 0) (extension_height 0.58642) (extension_offset 0.5) keep_text_aligned)
+  )
+  (dimension (type aligned) (layer "Dwgs.User")
+    (pts (xy 100 60) (xy 200 60))
+    (height -26.6)
+    (gr_text "100.0000 mm" (at 150 32.25) (layer "Dwgs.User")
+      (effects (font (size 1 1) (thickness 0.15)))
+    )
+    (format (units 3) (units_format 1) (precision 4))
+    (style (thickness 0.15) (arrow_length 1.27) (text_position_mode 0) (extension_height 0.58642) (extension_offset 0.5) keep_text_aligned)
+  )
+  (dimension (type aligned) (layer "Dwgs.User")
+    (pts (xy 104 121) (xy 100 121))
+    (height -8.6)
+    (gr_text "4.0000 mm" (at 102 128.45) (layer "Dwgs.User")
+      (effects (font (size 1 1) (thickness 0.15)))
+    )
+    (format (units 3) (units_format 1) (precision 4))
+    (style (thickness 0.15) (arrow_length 1.27) (text_position_mode 0) (extension_height 0.58642) (extension_offset 0.5) keep_text_aligned)
+  )
+  (dimension (type aligned) (layer "Dwgs.User")
+    (pts (xy 178 121) (xy 100 121))
+    (height -15)
+    (gr_text "78.0000 mm" (at 139 134.85) (layer "Dwgs.User")
+      (effects (font (size 1 1) (thickness 0.15)))
+    )
+    (format (units 3) (units_format 1) (precision 4))
+    (style (thickness 0.15) (arrow_length 1.27) (text_position_mode 0) (extension_height 0.58642) (extension_offset 0.5) keep_text_aligned)
+  )
 )

Commit message: Created a footprint fuse BSMD1812
Parts:
- F1: footprint GeneralPurposeAlarmDevicePCB:PlaceHolderOpossum -> GeneralPurposeAlarmDevicePCB:Fuse_BSMD_1812
- moved F1 48.4 mm to (116.8, 66.0), turned to 90 degrees

Commit message: Fixed error in SO4B & add new OLED footprint to schematic & PCB
Parts:
- removed the J2 at (135.0, 74.6)
- added G***: LOGO, GeneralPurposeAlarmDevicePCB:Logo_PI_BandW_70percent_10x10, F.Cu at (223.5, 96.5)
- J2: value SSD1306 OLED -> HS96L03W2C03_0.96_Oled; footprint Connector_PinHeader_2.54mm:PinHeader_1x08_P2.54mm_Vertical -> GeneralPurposeAlarmDevicePCB:HS96L03W2C03_0.96_Oled
- moved J2 36.7 mm to (132.1, 99.1), turned to 0 degrees

Commit message: Fixed OLED footprint, BOM maintenance
Parts:
- J10, J5: footprint Connector_PinHeader_2.54mm:PinHeader_2x05_P2.54mm_Vertical -> Connector_IDC:IDC-Header_2x06_P2.54mm_Vertical
- moved SW1 80.4 mm to (67.0, 110.0)
- moved SW3 61.3 mm to (67.0, 126.5)
- moved A1 55.9 mm to (88.2, 141.3)
- moved J1 55.9 mm to (54.6, 102.8)
- moved J4 55.9 mm to (88.2, 141.3)
- moved Q1 55.9 mm to (115.9, 135.3)
- moved D1 55.9 mm to (138.4, 120.0)
- moved F1 55.9 mm to (66.8, 91.0)
- moved G*** 55.9 mm to (173.5, 121.5)
- moved H1 55.9 mm to (54.0, 89.0)
- moved H2 55.9 mm to (54.0, 146.0)
- moved H3 55.9 mm to (128.0, 146.0)
- moved H4 55.9 mm to (128.0, 89.0)
- moved H5 55.9 mm to (142.0, 89.0)
- moved H6 55.9 mm to (142.0, 146.0)
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Other:
- board size 100 x 65 mm -> 108 x 65 mm

Commit message: PCB elements edited and moved
Parts:
- moved R7 24.9 mm to (147.0, 126.2), turned to 0 degrees
- moved TP1 20.3 mm to (112.7, 105.3)
- moved J9 16.1 mm to (151.2, 98.2), turned to 180 degrees
- moved J6 12.6 mm to (127.0, 110.5), turned to 90 degrees
- moved R1 5.49 mm to (105.8, 133.0)
- moved J5 5.43 mm to (125.5, 118.6)
- moved J11 4.46 mm to (139.5, 132.2)
- moved Q1 2.67 mm to (113.2, 135.7)
Connections:
- D1 pad 1: HeaterDrive -> HeaterDrive_IB
- H5 pad 1: GND -> GND1
- H6 pad 1: GND -> GND1
- J10 pad 1: HeaterDrive -> HeaterDrive_IB
- J10 pad 10: HeaterDrive -> HeaterDrive_IB
- J10 pad 2: GND -> GND1
- J10 pad 3: +5V -> +5P
- J10 pad 4: TempOut -> TempOut_IB
- J10 pad 5: VCC -> VCCQ
- J10 pad 6: VCC -> VCCQ
- J10 pad 7: TempOut -> TempOut_IB
- J10 pad 8: +5V -> +5P
- J10 pad 9: GND -> GND1
- J11 pad 1: VCC -> VCCQ
- J9 pad 1: GND -> GND1
- J9 pad 2: VCC -> VCCQ
- J9 pad 3: HeaterDrive -> HeaterDrive_IB
- J9 pad 4: +5V -> +5P
- J9 pad 5: TempOut -> TempOut_IB
- J9 pad 6: GND -> GND1
- R7 pad 2: +5V -> +5P
- TP2 pad 1: GND -> GND1
- U1 pad 1: TempOut -> TempOut_IB
- U1 pad 4: GND -> GND1
- U1 pad 8: +5V -> +5P
Routing:
- net GND: track 0.00 -> 341.3 mm
- net VCC: track 0.00 -> 101.8 mm
- net +5V: track 0.00 -> 80.2 mm
- net BTN_DOWN: track 0.00 -> 74.3 mm
- net GND1: track 0.00 -> 54.9 mm
- net BTN_UP: track 0.00 -> 41.3 mm
- net (no net): track 0.00 -> 39.8 mm
- net BTN_SELECT: track 0.00 -> 34.1 mm
- net +5P: track 0.00 -> 31.6 mm
- net TempOut_IB: track 0.00 -> 28.9 mm
- net TempOut: track 0.00 -> 24.2 mm
- net VCCQ: track 0.00 -> 20.7 mm
- net HeaterDrive_IB: track 0.00 -> 20.3 mm
- net HeaterDrive: track 0.00 -> 17.4 mm
- net TEMP_IN: track 0.00 -> 10.5 mm
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