File: moonratII/moonratII/moonratII.kicad_pcb (KiCad board)
At the start: 2 copper layers, 108 x 65 mm, 37 parts, among them J1 Barrel_Jack_Switch_SMT, J10 Conn_02x05_Odd_Even, J11 Screw_Terminal_01x02, J2 HS96L03W2C03_0.96_Oled, J3 PinHeader_1x06_P2.54mm_Vertic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, J4 PinHeader_1x08_P2.54mm_Vertic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, J5 Conn_02x05_Odd_Even, J6 Screw_Terminal_01x06, J7 PinHeader_1x08_P2.54mm_Vertic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, J8 PinHeader_1x10_P2.54mm_Vertic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, J9 Screw_Terminal_01x06, Q1 IRF520N, Q2 BSS138, SW1 6mm 2 Pin Tact NO Breadboard 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, SW2 6mm 2 Pin Tact NO Breadboard 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, SW3 6mm 2 Pin Tact NO Breadboard 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, U1 TMP36xS

Commit message: moonratII
Parts:
- J10, J5: footprint Connector_IDC:IDC-Header_2x06_P2.54mm_Vertical -> Connector_IDC:IDC-Header_2x05_P2.54mm_Vertical
- moved D1 15.3 mm to (153.6, 121.5)
- moved R7 8.01 mm to (139.7, 129.5)
- moved J11 7.78 mm to (147.3, 132.2), turned to 0 degrees
- moved U1 7.39 mm to (139.1, 121.9)
Routing:
- net GND: track 341.3 -> 0.00 mm
- net VCC: track 101.8 -> 0.00 mm
- net +5V: track 80.2 -> 0.00 mm
- net BTN_DOWN: track 74.3 -> 0.00 mm
- net GND1: track 54.9 -> 0.00 mm
- net VCCQ: track 20.7 -> 63.3 mm, vias 0 -> 4
- net BTN_UP: track 41.3 -> 0.00 mm
- net (no net): track 39.8 -> 0.00 mm
- net BTN_SELECT: track 34.1 -> 0.00 mm
- net HeaterDrive_IB: track 20.3 -> 47.7 mm, vias 0 -> 2
- net TempOut: track 24.2 -> 0.00 mm
- net +5P: track 31.6 -> 51.2 mm, vias 0 -> 3
- net HeaterDrive: track 17.4 -> 0.00 mm
- net TempOut_IB: track 28.9 -> 46.4 mm, vias 0 -> 4
- net TEMP_IN: track 10.5 -> 0.00 mm
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
Commit message: Routed the PCB heater side
Parts:
- moved TP2 7.81 mm to (153.0, 146.0)
- moved J11 5.86 mm to (142.7, 135.9)
- moved H5 2.00 mm to (144.0, 89.0)
- moved H6 2.00 mm to (144.0, 146.0)
Routing:
- net VCCQ: track 63.3 -> 71.1 mm
- net Net-(D1-A): track 12.5 -> 18.6 mm
- net +5P: track 51.2 -> 51.9 mm, vias 3 -> 4
- net TempOut_IB: track 46.4 -> 45.8 mm, vias 4 -> 3
- net Net-(U1-~{SHUTDOWN}): vias 2 -> 1
- net HeaterDrive_IB: vias 2 -> 3
- net GND1: vias 0 -> 7
- added copper zone on B.Cu, net GND1
- added copper zone on F.Cu, net GND1

Commit message: Deleted board to board headers. Placed components before getting to route
Parts:
- removed J3: PinHeader_1x06_P2.54mm_Vertical, Connector_PinHeader_2.54mm:PinHeader_1x06_P2.54mm_Vertical
- removed J4, J7: PinHeader_1x08_P2.54mm_Vertical, Connector_PinHeader_2.54mm:PinHeader_1x08_P2.54mm_Vertical
- removed J8: PinHeader_1x10_P2.54mm_Vertical, Connector_PinHeader_2.54mm:PinHeader_1x10_P2.54mm_Vertical
- added G***: LOGO, GeneralPurposeAlarmDevicePCB:Logo_PI_BandW_70percent_10x10, F.Cu at (63.5, 136.5)
- Q1: footprint Package_TO_SOT_THT:TO-220-3_Vertical -> Package_TO_SOT_THT:TO-220-3_Horizontal_TabDown
- moved G*** 48.4 mm to (137.2, 89.5)
- moved R5 41.3 mm to (69.5, 114.9), turned to 0 degrees
- moved R6 40.2 mm to (97.8, 97.8), turned to 180 degrees
- moved R4 37.5 mm to (69.8, 130.2), turned to 0 degrees
- moved R3 28.0 mm to (112.7, 109.9), turned to 0 degrees
- moved R1 20.0 mm to (125.5, 136.5), turned to 0 degrees
- moved Q2 8.00 mm to (87.3, 133.3)
- moved R2 6.41 mm to (102.9, 97.8), turned to 180 degrees
- moved SW2 5.59 mm to (116.0, 117.2), turned to 180 degrees
- moved Q1 3.08 mm to (113.0, 138.8)

Commit message: Routed the PCB main side
Routing:
- net +5V: track 0.00 -> 141.7 mm
- net VCC: track 0.00 -> 121.4 mm
- net Net-(Q2-G): track 0.00 -> 100.1 mm
- net HEATER_ON: track 0.00 -> 85.1 mm
- net BTN_UP: track 0.00 -> 71.4 mm
- net SCL: track 0.00 -> 68.0 mm
- net SDA: track 0.00 -> 55.5 mm
- net BTN_DOWN: track 0.00 -> 54.5 mm
- net HeaterDrive: track 0.00 -> 36.4 mm, vias 0 -> 1
- net BTN_SELECT: track 0.00 -> 26.7 mm
- net TempOut: track 0.00 -> 23.8 mm, vias 0 -> 1
- net Net-(F1-Pad2): track 0.00 -> 21.7 mm
- net TEMP_IN: track 0.00 -> 17.5 mm
- net Net-(BZ1-+): track 0.00 -> 4.78 mm

Commit message: Fixed footprint for SW 1, 2, 3. Significant update on bottom copper ground
Parts:
- SW1, SW2, SW3: footprint Button_Switch_THT:SW_PUSH_6mm -> GeneralPurposeAlarmDevicePCB:Switch_Tactile_THT_6x6mm
- moved R3 8.26 mm to (112.7, 101.6), turned to 180 degrees
- moved SW2 7.91 mm to (109.5, 112.8), turned to 0 degrees
- moved R5 1.56 mm to (69.2, 113.4), turned to 180 degrees
- moved R4 0.73 mm to (69.4, 129.6), turned to 180 degrees
Routing:
- net +5V: track 141.7 -> 208.5 mm, vias 0 -> 10
- net VCC: track 121.4 -> 168.2 mm, vias 0 -> 2
- net TempOut: track 23.8 -> 56.8 mm, vias 1 -> 7
- net SDA: track 55.5 -> 74.7 mm, vias 0 -> 6
- net HeaterDrive: track 36.4 -> 52.6 mm, vias 1 -> 3
- net Net-(Q2-G): track 100.1 -> 112.4 mm
- net BTN_DOWN: track 54.5 -> 59.8 mm, vias 0 -> 3
- net SCL: track 68.0 -> 62.7 mm, vias 0 -> 3
- net BTN_UP: track 71.4 -> 76.0 mm, vias 0 -> 5
- net BTN_SELECT: track 26.7 -> 29.1 mm, vias 0 -> 2
- net Net-(F1-Pad2): track 21.7 -> 21.0 mm
- net +5P: track 51.9 -> 51.3 mm, vias 4 -> 2
- net VCCQ: track 71.1 -> 70.7 mm, vias 4 -> 6
- net HeaterDrive_IB: vias 3 -> 2
- added copper zone on B.Cu, net GND
- added copper zone on F.Cu, net GND

Commit message: Performing design rule checks. Added ground between SCL & SDA traces to reduce the opportunity for cross talk.
Routing:
- net SDA: track 74.7 -> 56.3 mm
- net Net-(BZ1-+): track 4.78 -> 8.76 mm, vias 0 -> 1
- net SCL: track 62.7 -> 62.1 mm
- net GND: vias 0 -> 9

Commit message: PCB: Solved 2 DNR errors and added teardrops.
Routing:
- net SDA: vias 6 -> 7

Commit message: Solved 2 more PCB DNR errors.
Routing:
- net HeaterDrive: track 52.6 -> 54.3 mm
- net VCC: track 168.2 -> 168.9 mm
- net SCL: track 62.1 -> 62.4 mm, vias 3 -> 4
