File: moonratII/moonratII/moonratII.kicad_pcb (KiCad board)
At the start: 2 copper layers, 108 x 65 mm, 34 parts, among them J1 Barrel_Jack_Switch_SMT, J10 Conn_02x05_Odd_Even, J11 Screw_Terminal_01x02, J2 HS96L03W2C03_0.96_Oled, J5 Conn_02x05_Odd_Even, J6 Screw_Terminal_01x06, J9 Screw_Terminal_01x06, Q1 IRF520N, Q2 BSS138, SW1 6mm 2 Pin Tact NO Breadboard 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, SW2 6mm 2 Pin Tact NO Breadboard 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, SW3 6mm 2 Pin Tact NO Breadboard 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, U1 TMP36xS

Commit message: Cleared all PCB DRC errors and connection items.
Routing:
- net GND: track 0.00 -> 13.9 mm, vias 9 -> 19
- net BUZZER_ON: track 0.00 -> 5.53 mm
- net Net-(A1-D8): track 0.00 -> 4.73 mm
- net TempOut_IB: track 45.8 -> 45.9 mm, vias 3 -> 2
- net +5P: track 51.3 -> 51.2 mm, vias 2 -> 1
- net Net-(U1-~{SHUTDOWN}): vias 1 -> 0

Commit message: Cleared all DRC errors and warnings. Added 3 footprints
Parts:
- A1: footprint GeneralPurposeAlarmDevicePCB:Arduino_UNO_R3_NoMountingHoles3D -> GeneralPurposeAlarmDevicePCB:Arduino_UNO_R3_NoMountingHoles3D_Text_Top_&_Bottom
- J6, J9: footprint TerminalBlock_TE-Connectivity:TerminalBlock_TE_282834-6_1x06_P2.54mm_Horizontal -> GeneralPurposeAlarmDevicePCB:1x6P 20A -40℃~+105℃ 300V Green 12~30 Straight pin 5.08mm 2.5 1 6 Plugin,P=5.08mm Screw ter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
- moved G*** 15.1 mm to (152.3, 89.5)
Routing:
- net TempOut_IB: track 45.9 -> 44.9 mm, vias 2 -> 1
- net HeaterDrive: track 54.3 -> 53.6 mm, vias 3 -> 2
- net SDA: vias 7 -> 6
- net Net-(D1-A): vias 2 -> 1
- net HeaterDrive_IB: vias 2 -> 1
- net GND1: vias 7 -> 9
Other:
- board text added: "locked"

Commit message: Issue 70 completed: Add license info & open hardware & PI logo/symbols and related to schematic and PCB (Kicad)
Routing:
- net +5P: track 51.2 -> 49.7 mm
- net VCCQ: track 70.8 -> 69.8 mm, vias 6 -> 5
Other:
- board text added: "CERN Open Hardware License Version 2 - Strongly Reciprocal"
- board text added: "CERN Open Hardware License Version 2 Strongly Reciprocal"
- board text added: "MoonratII Controller, Public Invention, Rev 1.0 20231112"
- board text added: "MoonratII Heater, Public Invention, Rev 1.0 20231112"

Commit message: Issue 114: Corrected U1 footprint. Changed from SOIC-8 to SOT-23-5.
Parts:
- BZ1: value Buzzer_Adafruit_P1536A -> Buzzer_D12mm_H9.6mm_LS7.6mm
- U1: value TMP36xS -> TMP36GRTZ-REEL7; footprint Package_SO:SOIC-8_3.9x4.9mm_P1.27mm -> Package_TO_SOT_SMD:SOT-23-5
- moved U1 16.6 mm to (146.1, 136.9)
- moved J11 16.1 mm to (152.5, 123.1), turned to 90 degrees
- moved D1 9.22 mm to (144.4, 121.5)
- moved R7 7.87 mm to (142.4, 136.9), turned to 90 degrees
Connections:
- R7 pad 1: Net-(U1-~{SHUTDOWN}) -> Net-(U1-/SHUTDOWN)
- U1 pad 2: (no net) -> +5P
- U1 pad 3: (no net) -> unconnected-(U1-NC-Pad3)
- U1 pad 4: GND1 -> Net-(U1-/SHUTDOWN)
- U1 pad 5: Net-(U1-~{SHUTDOWN}) -> GND1
Routing:
- net TempOut_IB: track 44.9 -> 67.3 mm
- net VCCQ: track 69.8 -> 49.7 mm, vias 5 -> 3
- net +5P: track 49.7 -> 59.2 mm, vias 1 -> 3
- net Net-(D1-A): track 18.9 -> 9.42 mm
- net Net-(U1-/SHUTDOWN): track 0.00 -> 6.02 mm
- net Net-(U1-~{SHUTDOWN}): track 5.91 -> 0.00 mm
- net HeaterDrive_IB: track 47.9 -> 47.0 mm
- net GND1: vias 9 -> 12
Other:
- board text added: "MoonratII Controller, Public Invention, Rev 1.0 20231115"
- board text added: "MoonratII Heater, Public Invention, Rev 1.0 20231115"
- board text removed: "MoonratII Controller, Public Invention, Rev 1.0 20231112"
- board text removed: "MoonratII Heater, Public Invention, Rev 1.0 20231112"
