File: moonratII/pcb_moonratII/moonratII.kicad_sch (KiCad schematic)
At the start: 49 parts, among them J1 Barrel_Jack_Switch_SMT, J10 Conn_02x05_Odd_Even, J11 Screw_Terminal_01x02, J2 HS96L03W2C03_0.96_Oled, J5 Conn_02x05_Odd_Even, J6 Screw_Terminal_01x06, J9 Screw_Terminal_01x06, Q1 IRF520N, Q2 BSS138, SW1 6mm 2 Pin Tact NO Breadboard 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, SW2 6mm 2 Pin Tact NO Breadboard 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, SW3 6mm 2 Pin Tact NO Breadboard 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, U1 TMP36GRTZ-REEL7

Commit message: Fix issues 210, 211, 215, 195, and 216.
Parts:
- added R9: 1K, Resistor_SMD:R_0603_1608Metric_Pad0.98x0.95mm_HandSolder, symbol Device:R_US
- A1: Cost 1000000 -> 5.65; Distributor 1 (none) -> Aliexpress; Distributor 1 PN (none) -> https://www.aliexpress.us/item/3256802931453542.html; Notes (none) -> ORDER WITH CABLE
- MF102: value CAP TACTILE ROUND IVORY -> CAP TACTILE ROUND IVORY 6.00mm Dia; footprint B32-1600 -> B32-2000; Cost 0.3475 -> 0.95; Distributor 1 JLCPCB -> Digikey; Distributor 1 PN C231316 -> Z6127-ND
- MF102: value CAP TACTILE ROUND IVORY -> CAP TACTILE ROUND IVORY 6.00mm Dia; footprint B32-1600 -> B32-2000; Cost 0.3475 -> 0.95; Distributor 1 JLCPCB -> Digikey; Distributor 1 PN C231316 -> Z6127-ND; Notes (none) -> For Black use: SW1139-ND
- R2: value 1K -> DNI; now left out of the parts list
Connections:
- net HEATER_ON: now also R9.1
- net at A1.25 (D10): now also R9.2
- no-connect marks 49 -> 48
Other:
- note added: "MF12 is the header connecting the OLED to the PCB at what looks like J12 on the silk screen"
Changed lines of the file:
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@@
   (junction (at 133.35 95.25) (diameter 0) (color 0 0 0 0)
   )
+  (junction (at 106.68 128.905) (diameter 0) (color 0 0 0 0)
+  )
   (junction (at 109.22 111.76) (diameter 0) (color 0 0 0 0)
   )
@@
   (no_connect (at 73.66 85.09))
   (no_connect (at 99.06 95.25))
-  (no_connect (at 99.06 87.63))
   (no_connect (at 99.06 90.17))
   (no_connect (at 99.06 92.71))
@@
   (no_connect (at 196.85 63.5))
   (no_connect (at 199.39 35.56))
+  (wire (pts (xy 97.155 128.905) (xy 97.155 123.825))
+    (stroke (width 0) (type default))
+  )
   (wire (pts (xy 146.05 138.43) (xy 143.51 138.43))
     (stroke (width 0) (type default))
@@
     (stroke (width 0) (type default))
   )
+  (wire (pts (xy 97.155 110.49) (xy 97.155 116.205))
+    (stroke (width 0) (type default))
+  )
   (wire (pts (xy 185.42 151.13) (xy 196.85 151.13))
     (stroke (width 0) (type default))
@@
     (stroke (width 0) (type default))
   )
+  (wire (pts (xy 106.68 128.905) (xy 97.155 128.905))
+    (stroke (width 0) (type default))
+  )
   (wire (pts (xy 241.3 152.4) (xy 243.84 152.4))
     (stroke (width 0) (type default))
@@
     (stroke (width 0) (type default))
   )
+  (wire (pts (xy 106.68 128.905) (xy 106.68 132.08))
+    (stroke (width 0) (type default))
+  )
   (wire (pts (xy 78.74 151.13) (xy 80.01 151.13))
     (stroke (width 0) (type default))
@@
     (stroke (width 0) (type default))
   )
+  (wire (pts (xy 99.06 87.63) (xy 103.505 87.63))
+    (stroke (width 0) (type default))
+  )
   (wire (pts (xy 222.25 125.73) (xy 222.25 130.81))
     (stroke (width 0) (type default))
@@
     (stroke (width 0) (type default))
   )
+  (wire (pts (xy 103.505 87.63) (xy 103.505 110.49))
+    (stroke (width 0) (type default))
+  )
   (wire (pts (xy 62.23 99.06) (xy 62.23 107.95))
     (stroke (width 0) (type default))
@@
     (stroke (width 0) (type default))
   )
+  (wire (pts (xy 103.505 110.49) (xy 97.155 110.49))
+    (stroke (width 0) (type default))
+  )
   (wire (pts (xy 52.07 49.53) (xy 52.07 96.52))
     (stroke (width 0) (type default))
@@
     (stroke (width 0) (type default))
   )
-  (wire (pts (xy 106.68 124.46) (xy 106.68 132.08))
+  (wire (pts (xy 106.68 124.46) (xy 106.68 128.905))
     (stroke (width 0) (type default))
   )
@@
     (effects (font (size 1.27 1.27)) (justify left bottom))
   )
+  (text "MF12 is the header connecting the OLED to the PCB \nat what looks like J12 on the silk screen"
+    (at -106.045 133.985 0)
+    (effects (font (size 2.54 2.54)) (justify left bottom))
+  )
   (text "OLED Display\n1-GND\n2-+5V\n3-SCL\n4-SDA\n5-MH1\n6-MH2\n7-MH3\n8-MH4"
     (at 13.97 110.49 0)
@@
       (effects (font (size 1.27 1.27)) hide)
     )
-    (property "Cost" "1000000" (at 86.36 77.47 0)
+    (property "Cost" "5.65" (at 86.36 77.47 0)
       (effects (font (size 1.27 1.27)) hide)
     )
-    (property "Notes" "" (at 86.36 77.47 0)
+    (property "Notes" "ORDER WITH CABLE" (at 86.36 77.47 0)
+      (effects (font (size 1.27 1.27)) hide)
+    )
+    (property "Description" "Arduino UNO EXCEPT with micro USB" (at 86.36 77.47 0)
+      (effects (font (size 1.27 1.27)) hide)
+    )
+    (property "Distributor 1" "Aliexpress" (at 86.36 77.47 0)
+      (effects (font (size 1.27 1.27)) hide)
+    )
+    (property "Distributor 1 PN" "https://www.aliexpress.us/item/3256802931453542.html" (at 86.36 77.47 0)
       (effects (font (size 1.27 1.27)) hide)
     )
@@
       (effects (font (size 1.27 1.27)) (justify left))
     )
-    (property "Value" "CAP TACTILE ROUND IVORY" (at 91.44 186.69 0)
+    (property "Value" "CAP TACTILE ROUND IVORY 6.00mm Dia " (at 91.44 186.69 0)
       (effects (font (size 1.27 1.27)) (justify left))
     )
-    (property "Footprint" "B32-1600" (at 105.41 186.69 0)
+    (property "Footprint" "B32-2000" (at 105.41 186.69 0)
       (effects (font (size 1.27 1.27)) hide)
     )
@@
       (effects (font (size 1.27 1.27)) hide)
     )
-    (property "Distributor 1" "JLCPCB" (at 105.41 186.69 0)
+    (property "Distributor 1" "Digikey" (at 105.41 186.69 0)
       (effects (font (size 1.27 1.27)) hide)
     )
-    (property "Distributor 1 PN" "C231316" (at 105.41 186.69 0)
+    (property "Distributor 1 PN" "Z6127-ND" (at 105.41 186.69 0)
       (effects (font (size 1.27 1.27)) hide)
     )
-    (property "Cost" "0.3475 " (at 105.41 186.69 0)
+    (property "Cost" "0.95" (at 105.41 186.69 0)
       (effects (font (size 1.27 1.27)) hide)
     )
@@
       (effects (font (size 1.27 1.27)) hide)
     )
+    (property "Description" "Round Tactile Switch Cap Ivory Slip On, 6.00mm Dia x 5.50mm H" (at 105.41 186.69 0)
+      (effects (font (size 1.27 1.27)) hide)
+    )
     (instances
       (project "GeneralPurposeAlarmDevicePCB"
@@
   )
   (symbol (lib_id "Device:R_US") (at 106.68 120.65 180) (unit 1)
-    (in_bom yes) (on_board yes) (dnp no)
+    (in_bom no) (on_board yes) (dnp no)
     (property "Reference" "R2" (at 104.14 124.46 90)
       (effects (font (size 1.27 1.27)))
     )
-    (property "Value" "1K" (at 104.14 116.84 90)
+    (property "Value" "DNI" (at 104.14 116.84 90)
       (effects (font (size 1.27 1.27)))
     )
@@
       (effects (font (size 1.27 1.27)) (justify left))
     )
-    (property "Value" "CAP TACTILE ROUND IVORY" (at 125.73 186.69 0)
+    (property "Value" "CAP TACTILE ROUND IVORY 6.00mm Dia " (at 125.73 186.69 0)
       (effects (font (size 1.27 1.27)) (justify left))
     )
-    (property "Footprint" "B32-1600" (at 139.7 186.69 0)
+    (property "Footprint" "B32-2000" (at 139.7 186.69 0)
       (effects (font (size 1.27 1.27)) hide)
     )
@@
       (effects (font (size 1.27 1.27)) hide)
     )
-    (property "Distributor 1" "JLCPCB" (at 139.7 186.69 0)
+    (property "Distributor 1" "Digikey" (at 139.7 186.69 0)
       (effects (font (size 1.27 1.27)) hide)
     )
-    (property "Distributor 1 PN" "C231316" (at 139.7 186.69 0)
+    (property "Distributor 1 PN" "Z6127-ND" (at 139.7 186.69 0)
       (effects (font (size 1.27 1.27)) hide)
     )
-    (property "Cost" "0.3475 " (at 139.7 186.69 0)
+    (property "Cost" "0.95" (at 139.7 186.69 0)
       (effects (font (size 1.27 1.27)) hide)
     )
@@
       (effects (font (size 1.27 1.27)) hide)
     )
+    (property "Description" "Round Tactile Switch Cap Ivory Slip On, 6.00mm Dia x 5.50mm H" (at 139.7 186.69 0)
+      (effects (font (size 1.27 1.27)) hide)
+    )
     (instances
       (project "GeneralPurposeAlarmDevicePCB"
@@
       (effects (font (size 1.27 1.27)) (justify left))
     )
-    (property "Value" "CAP TACTILE ROUND IVORY" (at 58.42 186.69 0)
+    (property "Value" "CAP TACTILE ROUND IVORY 6.00mm Dia " (at 58.42 186.69 0)
       (effects (font (size 1.27 1.27)) (justify left))
     )
-    (property "Footprint" "B32-1600" (at 72.39 186.69 0)
+    (property "Footprint" "B32-2000" (at 72.39 186.69 0)
       (effects (font (size 1.27 1.27)) hide)
     )
@@
       (effects (font (size 1.27 1.27)) hide)
     )
-    (property "Distributor 1" "JLCPCB" (at 72.39 186.69 0)
+    (property "Distributor 1" "Digikey" (at 72.39 186.69 0)
       (effects (font (size 1.27 1.27)) hide)
     )
-    (property "Distributor 1 PN" "C231316" (at 72.39 186.69 0)
+    (property "Distributor 1 PN" "Z6127-ND" (at 72.39 186.69 0)
       (effects (font (size 1.27 1.27)) hide)
     )
-    (property "Cost" "0.3475 " (at 72.39 186.69 0)
+    (property "Cost" "0.95" (at 72.39 186.69 0)
       (effects (font (size 1.27 1.27)) hide)
     )
-    (property "Notes" "" (at 72.39 186.69 0)
+    (property "Notes" "For Black use: SW1139-ND" (at 72.39 186.69 0)
+      (effects (font (size 1.27 1.27)) hide)
+    )
+    (property "Description" "Round Tactile Switch Cap Ivory Slip On, 6.00mm Dia x 5.50mm H" (at 72.39 186.69 0)
       (effects (font (size 1.27 1.27)) hide)
     )
@@
         )
       )
+    )
+  )
+  (symbol (lib_id "Device:R_US") (at 97.155 120.015 180) (unit 1)
+    (in_bom yes) (on_board yes) (dnp no)
+    (property "Reference" "R9" (at 94.615 123.825 90)
+      (effects (font (size 1.27 1.27)))
+    )
+    (property "Value" "1K" (at 94.615 116.205 90)
+      (effects (font (size 1.27 1.27)))
+    )
+    (property "Footprint" "Resistor_SMD:R_0603_1608Metric_Pad0.98x0.95mm_HandSolder" (at 96.139 119.761 90)
+      (effects (font (size 1.27 1.27)) hide)
+    )
+    (property "Datasheet" "RMC06031K1%N.pdf" (at 97.155 120.015 0)
+      (effects (font (size 1.27 1.27)) hide)
+    )
+    (property "AssemblyType" "SMT" (at 97.155 120.015 0)
+      (effects (font (size 1.27 1.27)) hide)
+    )
+    (property "Cost" "0.0015" (at 97.155 120.015 0)
+      (effects (font (size 1.27 1.27)) hide)
+    )
+    (property "Description" "0.1W ±1% 1kΩ 0603 Chip Resistor - Surface Mount ROHS" (at 97.155 120.015 0)
+      (effects (font (size 1.27 1.27)) hide)
+    )
+    (property "Distributor 1" "JLCPCB" (at 97.155 120.015 0)
+      (effects (font (size 1.27 1.27)) hide)
+    )
+    (property "Distributor 1 PN" "C269704" (at 97.155 120.015 0)
+      (effects (font (size 1.27 1.27)) hide)
+    )
+    (property "MPN" "RMC06031K1%N" (at 97.155 120.015 0)
+      (effects (font (size 1.27 1.27)) hide)
+    )
+    (property "Manufacturer" "TyoHM" (at 97.155 120.015 0)
+      (effects (font (size 1.27 1.27)) hide)
+    )
+    (property "Notes" "" (at 97.155 120.015 0)
+      (effects (font (size 1.27 1.27)) hide)
+    )
+    (pin "1")
+    (pin "2")
+    (instances
+      (project "moonratII"
+        (path "/9ef5effe-cb46-4a9a-bbbe-a65ab44b9e67"
+          (reference "R9") (unit 1)
+        )
+      )
