File: moonratII/pcb_moonratII/moonratII.kicad_sch (KiCad schematic)
At the start: 50 parts, among them J1 Barrel_Jack_Switch_SMT, J10 Conn_02x05_Odd_Even, J11 Screw_Terminal_01x02, J2 HS96L03W2C03_0.96_Oled, J5 Conn_02x05_Odd_Even, J6 Screw_Terminal_01x06, J9 Screw_Terminal_01x06, Q1 IRF520N, Q2 BSS138, SW1 6mm 2 Pin Tact NO Breadboard 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, SW2 6mm 2 Pin Tact NO Breadboard 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, SW3 6mm 2 Pin Tact NO Breadboard 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, U1 TMP36GRTZ-REEL7

Commit message: Add a capactor on TMP36 power pin.
Parts:
- added C1: 0.1uF, Capacitor_SMD:C_0603_1608Metric_Pad1.08x0.95mm_HandSolder, symbol Device:C
Connections:
- net +5P: now also C1.1
- net GND1: now also C1.2
Changed lines of the file:
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@@
   (junction (at 190.5 113.03) (diameter 0) (color 0 0 0 0)
   )
+  (junction (at 248.92 116.84) (diameter 0) (color 0 0 0 0)
+  )
   (junction (at 20.32 191.77) (diameter 0) (color 0 0 0 0)
   )
@@
     (stroke (width 0) (type default))
   )
+  (wire (pts (xy 250.19 116.84) (xy 248.92 116.84))
+    (stroke (width 0) (type default))
+  )
   (wire (pts (xy 208.28 123.19) (xy 208.28 113.03))
     (stroke (width 0) (type default))
@@
     (stroke (width 0) (type default))
   )
+  (wire (pts (xy 263.525 99.695) (xy 255.27 99.695))
+    (stroke (width 0) (type default))
+  )
   (wire (pts (xy 241.3 148.59) (xy 257.81 148.59))
     (stroke (width 0) (type default))
@@
     (stroke (width 0) (type default))
   )
+  (wire (pts (xy 255.27 98.425) (xy 255.27 99.695))
+    (stroke (width 0) (type default))
+  )
   (wire (pts (xy 241.3 158.75) (xy 241.3 152.4))
     (stroke (width 0) (type default))
@@
     (stroke (width 0) (type default))
   )
+  (wire (pts (xy 255.27 90.805) (xy 250.19 90.805))
+    (stroke (width 0) (type default))
+  )
   (wire (pts (xy 196.85 156.21) (xy 190.5 156.21))
     (stroke (width 0) (type default))
@@
     (stroke (width 0) (type default))
   )
+  (wire (pts (xy 250.19 90.805) (xy 250.19 116.84))
+    (stroke (width 0) (type default))
+  )
   (wire (pts (xy 140.97 158.75) (xy 140.97 161.29))
     (stroke (width 0) (type default))
@@
     )
   )
+  (symbol (lib_id "power:GND1") (at 263.525 99.695 0) (unit 1)
+    (in_bom yes) (on_board yes) (dnp no) (fields_autoplaced)
+    (property "Reference" "#PWR012" (at 263.525 106.045 0)
+      (effects (font (size 1.27 1.27)) hide)
+    )
+    (property "Value" "GND1" (at 263.525 104.775 0)
+      (effects (font (size 1.27 1.27)))
+    )
+    (property "Footprint" "" (at 263.525 99.695 0)
+      (effects (font (size 1.27 1.27)) hide)
+    )
+    (property "Datasheet" "" (at 263.525 99.695 0)
+      (effects (font (size 1.27 1.27)) hide)
+    )
+    (pin "1")
+    (instances
+      (project "moonratII"
+        (path "/9ef5effe-cb46-4a9a-bbbe-a65ab44b9e67"
+          (reference "#PWR012") (unit 1)
+        )
+      )
+    )
+  )
   (symbol (lib_id "GPAD_SCH_LIB:ENCLOSURE_GPAD_VER1") (at -55.88 173.99 0) (unit 1)
     (in_bom yes) (on_board no) (dnp no)
@@
         )
       )
+    )
+  )
+  (symbol (lib_id "Device:C") (at 255.27 94.615 0) (unit 1)
+    (in_bom yes) (on_board yes) (dnp no) (fields_autoplaced)
+    (property "Reference" "C1" (at 259.08 93.345 0)
+      (effects (font (size 1.27 1.27)) (justify left))
+    )
+    (property "Value" "0.1uF" (at 259.08 95.885 0)
+      (effects (font (size 1.27 1.27)) (justify left))
+    )
+    (property "Footprint" "Capacitor_SMD:C_0603_1608Metric_Pad1.08x0.95mm_HandSolder" (at 256.2352 98.425 0)
+      (effects (font (size 1.27 1.27)) hide)
+    )
+    (property "Datasheet" "~" (at 255.27 94.615 0)
+      (effects (font (size 1.27 1.27)) hide)
+    )
+    (property "Cost" "0.0021" (at 255.27 94.615 0)
+      (effects (font (size 1.27 1.27)) hide)
+    )
+    (property "Description" "50V 100nF X7R ±10% 0603 Multilayer Ceramic Capacitors MLCC - SMD/SMT ROHS" (at 255.27 94.615 0)
+      (effects (font (size 1.27 1.27)) hide)
+    )
+    (property "Distributor 1" "JLCPCB" (at 255.27 94.615 0)
+      (effects (font (size 1.27 1.27)) hide)
+    )
+    (property "Distributor 1 PN" "C14663" (at 255.27 94.615 0)
+      (effects (font (size 1.27 1.27)) hide)
+    )
+    (pin "1")
+    (pin "2")
+    (instances
+      (project "moonratII"
+        (path "/9ef5effe-cb46-4a9a-bbbe-a65ab44b9e67"
+          (reference "C1") (unit 1)
+        )
+      )

Commit message: Change Q1 to IRF540NPBF for higher current rating.
Parts:
- Q1: value IRF520N -> IRF540N; Cost 0.6995 -> 0.3480; Distributor 1 PN C2598 -> C2566; MPN IRF520NPBF -> IRF540NPBF
Changed lines of the file:
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@@
       (effects (font (size 1.27 1.27)) (justify left))
     )
-    (property "Value" "IRF520N" (at 121.92 133.3499 0)
+    (property "Value" "IRF540N" (at 121.92 133.3499 0)
       (effects (font (size 1.27 1.27)) (justify left))
     )
@@
       (effects (font (size 1.27 1.27)) hide)
     )
-    (property "Cost" "0.6995" (at 115.57 132.08 0)
+    (property "Cost" "0.3480" (at 115.57 132.08 0)
       (effects (font (size 1.27 1.27)) hide)
     )
-    (property "Description" "100V 9.7A 48W 200mΩ@10V,5.7A N Channel TO-220 MOSFETs ROHS" (at 115.57 132.08 0)
+    (property "Description" "100V 33A 44mΩ@10V,16A 130W N Channel TO-220 MOSFETs ROHS" (at 115.57 132.08 0)
       (effects (font (size 1.27 1.27)) hide)
     )
@@
       (effects (font (size 1.27 1.27)) hide)
     )
-    (property "Distributor 1 PN" "C2598" (at 115.57 132.08 0)
+    (property "Distributor 1 PN" "C2566" (at 115.57 132.08 0)
       (effects (font (size 1.27 1.27)) hide)
     )
-    (property "MPN" "IRF520NPBF" (at 115.57 132.08 0)
+    (property "MPN" "IRF540NPBF" (at 115.57 132.08 0)
       (effects (font (size 1.27 1.27)) hide)
     )

Commit message: Add resistor so buzzer off during reset.
Parts:
- added R10: 10K, Resistor_SMD:R_0603_1608Metric_Pad0.98x0.95mm_HandSolder, symbol Device:R_US
Connections:
- net BUZZER_ON: now also R10.1
- net GND: now also R10.2
Changed lines of the file:
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@@
   (junction (at 190.5 113.03) (diameter 0) (color 0 0 0 0)
   )
+  (junction (at 121.285 111.76) (diameter 0) (color 0 0 0 0)
+  )
   (junction (at 248.92 116.84) (diameter 0) (color 0 0 0 0)
   )
@@
     (stroke (width 0) (type default))
   )
+  (wire (pts (xy 123.825 104.14) (xy 121.285 104.14))
+    (stroke (width 0) (type default))
+  )
   (wire (pts (xy 209.55 151.13) (xy 222.25 151.13))
     (stroke (width 0) (type default))
@@
     (stroke (width 0) (type default))
   )
-  (wire (pts (xy 109.22 111.76) (xy 144.78 111.76))
+  (wire (pts (xy 109.22 111.76) (xy 121.285 111.76))
     (stroke (width 0) (type default))
   )
@@
     (stroke (width 0) (type default))
   )
+  (wire (pts (xy 131.445 104.14) (xy 136.525 104.14))
+    (stroke (width 0) (type default))
+  )
   (wire (pts (xy 263.525 99.695) (xy 255.27 99.695))
     (stroke (width 0) (type default))
@@
     (stroke (width 0) (type default))
   )
+  (wire (pts (xy 121.285 104.14) (xy 121.285 111.76))
+    (stroke (width 0) (type default))
+  )
   (wire (pts (xy 58.42 77.47) (xy 58.42 153.67))
     (stroke (width 0) (type default))
@@
     (stroke (width 0) (type default))
   )
+  (wire (pts (xy 121.285 111.76) (xy 144.78 111.76))
+    (stroke (width 0) (type default))
+  )
   (wire (pts (xy 257.81 128.27) (xy 257.81 148.59))
     (stroke (width 0) (type default))
@@
     )
   )
+  (symbol (lib_id "Device:R_US") (at 127.635 104.14 90) (unit 1)
+    (in_bom yes) (on_board yes) (dnp no)
+    (property "Reference" "R10" (at 123.825 101.6 90)
+      (effects (font (size 1.27 1.27)))
+    )
+    (property "Value" "10K" (at 131.445 101.6 90)
+      (effects (font (size 1.27 1.27)))
+    )
+    (property "Footprint" "Resistor_SMD:R_0603_1608Metric_Pad0.98x0.95mm_HandSolder" (at 127.889 103.124 90)
+      (effects (font (size 1.27 1.27)) hide)
+    )
+    (property "Datasheet" "RMC06031K1%N.pdf" (at 127.635 104.14 0)
+      (effects (font (size 1.27 1.27)) hide)
+    )
+    (property "AssemblyType" "SMT" (at 127.635 104.14 0)
+      (effects (font (size 1.27 1.27)) hide)
+    )
+    (property "Cost" "0.0036" (at 127.635 104.14 0)
+      (effects (font (size 1.27 1.27)) hide)
+    )
+    (property "Description" "100mW ±1% 10kΩ 0603 Chip Resistor - Surface Mount ROHS" (at 127.635 104.14 0)
+      (effects (font (size 1.27 1.27)) hide)
+    )
+    (property "Distributor 1" "JLCPCB" (at 127.635 104.14 0)
+      (effects (font (size 1.27 1.27)) hide)
+    )
+    (property "Distributor 1 PN" "C269701" (at 127.635 104.14 0)
+      (effects (font (size 1.27 1.27)) hide)
+    )
+    (property "MPN" "RMC060310KFN" (at 127.635 104.14 0)
+      (effects (font (size 1.27 1.27)) hide)
+    )
+    (property "Manufacturer" "TyoHM" (at 127.635 104.14 0)
+      (effects (font (size 1.27 1.27)) hide)
+    )
+    (property "Notes" "" (at 127.635 104.14 0)
+      (effects (font (size 1.27 1.27)) hide)
+    )
+    (pin "1")
+    (pin "2")
+    (instances
+      (project "moonratII"
+        (path "/9ef5effe-cb46-4a9a-bbbe-a65ab44b9e67"
+          (reference "R10") (unit 1)
+        )
+      )
+    )
+  )
   (symbol (lib_id "power:+5P") (at 222.25 147.32 0) (unit 1)
     (in_bom yes) (on_board yes) (dnp no) (fields_autoplaced)
@@
         )
       )
+    )
+  )
+  (symbol (lib_id "power:GND") (at 136.525 104.14 0) (unit 1)
+    (in_bom yes) (on_board yes) (dnp no) (fields_autoplaced)
+    (property "Reference" "#PWR013" (at 136.525 110.49 0)
+      (effects (font (size 1.27 1.27)) hide)
+    )
+    (property "Value" "GND" (at 136.525 109.22 0)
+      (effects (font (size 1.27 1.27)))
+    )
+    (property "Footprint" "" (at 136.525 104.14 0)
+      (effects (font (size 1.27 1.27)) hide)
+    )
+    (property "Datasheet" "" (at 136.525 104.14 0)
+      (effects (font (size 1.27 1.27)) hide)
+    )
+    (pin "1")
+    (instances
+      (project "moonratII"
+        (path "/9ef5effe-cb46-4a9a-bbbe-a65ab44b9e67"
+          (reference "#PWR013") (unit 1)
+        )
+      )

Commit message: Add PDF files, sch and pcb. Updateing to Rev 2 gerbers/drill.
Parts:
- MF102: Notes (none) -> For Black use: SW1139-ND
Other:
- note removed: "MF12 is the header connecting the OLED to the PCB at what looks like J12 on the silk screen"
- moved on the sheet: A1, BZ1, C1, Cable_MoldedFemale1, Cable_MoldedMale1, Cable_Ribbon1, D1, F1, H1, H2, H3, H4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

Commit message: Add position file. Change UNO description to mUSB and with cable.
Parts:
- A1: value Arduino_UNO_R3 -> Arduino_UNO_R3 with uUSB and Cable
Changed lines of the file:
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@@
   (symbol (lib_id "MCU_Module:Arduino_UNO_R3") (at 230.505 99.06 0) (mirror y) (unit 1)
     (in_bom yes) (on_board yes) (dnp no) (fields_autoplaced)
-    (property "Reference" "A1" (at 235.8137 71.12 0)
+    (property "Reference" "A1" (at 236.1947 71.12 0)
       (effects (font (size 1.27 1.27)) (justify right))
     )
-    (property "Value" "Arduino_UNO_R3" (at 235.8137 73.66 0)
+    (property "Value" "Arduino_UNO_R3 with uUSB and Cable" (at 236.1947 73.66 0)
       (effects (font (size 1.27 1.27)) (justify right))
     )

Commit message: Change part number on J11 for 2.54mm screw terminal.
Parts:
- J11: Distributor 1 PN C2915639 -> C557685
Changed lines of the file:
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@@
       (effects (font (size 1.27 1.27)) hide)
     )
-    (property "Datasheet" "DB128V-5.08-2P-GN-S.pdf" (at 390.525 179.07 0)
+    (property "Datasheet" "XY308-2.54-2P.pdf" (at 390.525 179.07 0)
       (effects (font (size 1.27 1.27)) hide)
     )
@@
       (effects (font (size 1.27 1.27)) hide)
     )
-    (property "Description" "1x2P 20A -40℃~+105℃ 300V Green 12~30 Straight pin 5.08mm 2.5 1 2 Plugin,P=5.08mm Screw terminal ROHS" (at 390.525 179.07 0)
+    (property "Description" "1x2P 6A 150V Green 18~26 Straight 2.54mm 1 1 2 Plugin,P=2.54mm Screw terminal ROHS" (at 390.525 179.07 0)
       (effects (font (size 1.27 1.27)) hide)
     )
@@
       (effects (font (size 1.27 1.27)) hide)
     )
-    (property "Distributor 1 PN" "C2915639" (at 390.525 179.07 0)
+    (property "Distributor 1 PN" "C557685" (at 390.525 179.07 0)
       (effects (font (size 1.27 1.27)) hide)
     )

Commit message: Modified BOM, schematic, and created assembly in Freecad of PWA and enclosure.
Parts:
- MF102: value CAP TACTILE ROUND IVORY 6.00mm Dia -> CAP TACTILE ROUND IVORY 6.00mm Dia
