File: moonratII/pcb_moonratII/moonratII.kicad_pcb (KiCad board)
At the start: 2 copper layers, 108 x 65 mm, 34 parts, among them J1 Barrel_Jack_Switch_SMT, J10 Conn_02x05_Odd_Even, J11 Screw_Terminal_01x02, J2 HS96L03W2C03_0.96_Oled, J5 Conn_02x05_Odd_Even, J6 Screw_Terminal_01x06, J9 Screw_Terminal_01x06, Q1 IRF520N, Q2 BSS138, SW1 6mm 2 Pin Tact NO Breadboard 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, SW2 6mm 2 Pin Tact NO Breadboard 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, SW3 6mm 2 Pin Tact NO Breadboard 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, U1 TMP36GRTZ-REEL7

Commit message: Revert "Make vcc heavy"
Parts:
- moved R6 7.77 mm to (97.8, 97.8)
- moved R2 7.72 mm to (102.9, 97.8)
- moved Q1 2.52 mm to (113.0, 138.8)
- moved R1 1.47 mm to (125.5, 136.5)
Connections:
- net /VCC_RAW renamed Net-(F1-Pad2)
Routing:
- net VCC: track 136.3 -> 168.9 mm, vias 3 -> 2
- net GND1: track 11.2 -> 0.00 mm, vias 9 -> 12
- net TempOut: track 46.5 -> 57.3 mm, vias 1 -> 7
- net SCL: track 68.5 -> 62.4 mm
- net SDA: track 62.2 -> 56.3 mm, vias 4 -> 6
- net VCCQ: track 44.7 -> 49.7 mm, vias 2 -> 3
- net HeaterDrive_IB: track 42.3 -> 47.0 mm
- net HeaterDrive: track 57.7 -> 53.6 mm, vias 1 -> 2
- net HEATER_ON: track 88.5 -> 85.4 mm
- net GND: track 11.4 -> 13.9 mm, vias 27 -> 21
- net BUZZER_ON: track 3.14 -> 5.37 mm
- net Net-(Q2-G): track 110.5 -> 112.4 mm
- net Net-(A1-D8): track 3.17 -> 4.73 mm
- net +5V: track 210.6 -> 209.1 mm
- net Net-(D1-A): track 10.1 -> 9.42 mm
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Other:
- board text added: "MoonratII Controller, Public Invention, Rev 1.0 20231120"
- board text added: "MoonratII Heater, Public Invention, Rev 1.0 20231120"
- board text removed: "MoonratII Controller, Public Invention, Rev 2.0 20240206"
- board text removed: "MoonratII Heater, Public Invention, Rev 2.0 20240206"

Commit message: Increase size on Heater traces.
Parts:
- moved R6 7.77 mm to (98.2, 90.0)
- moved R2 7.72 mm to (103.3, 90.1)
- moved Q1 2.52 mm to (110.5, 138.3)
Connections:
- net Net-(F1-Pad2) renamed /VCC_RAW
Routing:
- net VCC: track 168.9 -> 136.5 mm, vias 2 -> 3
- net HeaterDrive_IB: track 47.0 -> 22.4 mm
- net TempOut: track 57.3 -> 46.9 mm, vias 7 -> 1
- net SCL: track 62.4 -> 68.5 mm
- net SDA: track 56.3 -> 62.2 mm, vias 6 -> 4
- net VCCQ: track 49.7 -> 44.0 mm, vias 3 -> 2
- net HeaterDrive: track 53.6 -> 58.1 mm, vias 2 -> 1
- net HEATER_ON: track 85.4 -> 89.7 mm
- net TEMP_IN: track 17.5 -> 20.7 mm, vias 0 -> 1
- net GND: track 13.9 -> 11.4 mm
- net Net-(Q2-G): track 112.4 -> 110.5 mm
- net BUZZER_ON: track 5.37 -> 3.42 mm
- net +5V: track 209.1 -> 211.0 mm
- net Net-(A1-D8): track 4.73 -> 3.17 mm
- net Net-(D1-A): track 9.42 -> 10.5 mm
- removed copper zone on F.Cu, net GND1
Other:
- board text added: "MoonratII Controller, Public Invention, Rev 2.0 20240206"
- board text added: "MoonratII Heater, Public Invention, Rev 2.0 20240206"
- board text removed: "MoonratII Controller, Public Invention, Rev 1.0 20231120"
- board text removed: "MoonratII Heater, Public Invention, Rev 1.0 20231120"

Commit message: Clear all DRC errors. Clear most warnings.
Routing:
- net HeaterDrive_IB: track 22.4 -> 42.3 mm
- net GND1: track 0.00 -> 11.2 mm, vias 12 -> 9
- net TEMP_IN: track 20.7 -> 20.0 mm
- net VCCQ: track 44.0 -> 44.7 mm
- net GND: vias 21 -> 23
- added copper zone on F.Cu, net GND1

Commit message: Clean up some via spacing and ground pours.
Parts:
- moved R1 1.47 mm to (124.0, 136.1)
Routing:
- net TEMP_IN: track 20.0 -> 18.0 mm
- net HEATER_ON: track 89.7 -> 88.5 mm
- net GND: vias 23 -> 27
