File: moonratII/pcb_moonratII/moonratII.kicad_pcb (KiCad board)
At the start: 2 copper layers, 108 x 65 mm, 34 parts, among them J1 Barrel_Jack_Switch_SMT, J10 Conn_02x05_Odd_Even, J11 Screw_Terminal_01x02, J2 HS96L03W2C03_0.96_Oled, J5 Conn_02x05_Odd_Even, J6 Screw_Terminal_01x06, J9 Screw_Terminal_01x06, Q1 IRF520N, Q2 BSS138, SW1 6mm 2 Pin Tact NO Breadboard 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, SW2 6mm 2 Pin Tact NO Breadboard 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, SW3 6mm 2 Pin Tact NO Breadboard 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, U1 TMP36GRTZ-REEL7

Commit message: Fix issues 210, 211, 215, 195, and 216.
Parts:
- added R9: 1K, Resistor_SMD:R_0603_1608Metric_Pad0.98x0.95mm_HandSolder, F.Cu at (109.0, 90.1)
- R2: value 1K -> DNI
- moved R6 5.94 mm to (92.3, 89.8)
Connections:
- A1 pad 25: unconnected-(A1-D10-Pad25) -> Net-(A1-D10)
Routing:
- net Net-(A1-D10): track 0.00 -> 14.9 mm, vias 0 -> 1
- net Net-(Q2-G): track 110.5 -> 104.6 mm
- net BUZZER_ON: track 3.14 -> 8.41 mm
- net HEATER_ON: track 88.5 -> 89.5 mm

Commit message: Change date of schematic and PCB for rev 2. Tweek to PCB after changing BoardSetupContratins.
Routing:
- net GND: track 11.4 -> 35.8 mm
Other:
- board text added: "MoonratII Controller, Public Invention, Rev 2.0 20240302"
- board text added: "MoonratII Heater, Public Invention, Rev 2.0 20240302"
- board text removed: "MoonratII Controller, Public Invention, Rev 2.0 20240206"
- board text removed: "MoonratII Heater, Public Invention, Rev 2.0 20240206"

Commit message: Add a capactor on TMP36 power pin.
Parts:
- added C1: 0.1uF, Capacitor_SMD:C_0603_1608Metric_Pad1.08x0.95mm_HandSolder, F.Cu at (149.3, 136.9)
Connections:
- net /VCC_RAW renamed Net-(F1-Pad2)
Routing:
- net +5P: track 59.5 -> 64.0 mm
- net GND1: track 11.2 -> 13.6 mm

Commit message: Add resistor so buzzer off during reset.
Parts:
- added R10: 10K, Resistor_SMD:R_0603_1608Metric_Pad0.98x0.95mm_HandSolder, F.Cu at (75.0, 92.9)
- Q1: value IRF520N -> IRF540N
- moved R6 21.5 mm to (70.8, 90.9)
Routing:
- net BUZZER_ON: track 8.41 -> 32.6 mm
- net Net-(Q2-G): track 104.6 -> 82.6 mm
- net GND: track 35.8 -> 39.3 mm, vias 27 -> 30
Other:
- board text added: "SN:___________"
