File: moonratII/pcb_moonratII/pcb_moonratII.kicad_pcb (KiCad board)
At the start: 2 copper layers, 108 x 65 mm, 37 parts, among them J1 Barrel_Jack_Switch_SMT, J10 Conn_02x05_Odd_Even, J11 Screw_Terminal_01x02, J2 HS96L03W2C03_0.96_Oled, J5 Conn_02x05_Odd_Even, J6 Screw_Terminal_01x06, J9 Screw_Terminal_01x06, Q1 IRF540N, Q2 BSS138, SW1 6mm 2 Pin Tact NO Breadboard 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, SW2 6mm 2 Pin Tact NO Breadboard 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, SW3 6mm 2 Pin Tact NO Breadboard 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, U1 TMP36GRTZ-REEL7

Commit message: pcb_moonratII.kicad_pcb, repaired switch STEP file.
Other:
- board text added: "V-CUT"
- board text removed: "locked"

Commit message: pcb_moonratII.kicad_pcb,updated 3D models for keycaps and buzzer.
Parts:
- A1: value Arduino_UNO_R3 -> Arduino_UNO_R3 with uUSB and Cable
- BZ1: footprint GeneralPurposeAlarmDevicePCB:Buzzer_12.2mm_9.7mm_7.62mm -> PubInv_KiCad_PCB:Buzzer_12.2mm_9.7mm_7.62mm
