File: moonratII/pcb_Heater/Heater_board_Rev2/Heater_board_Rev2.kicad_pcb (KiCad board)
At the start: 2 copper layers, 108 x 65 mm, 37 parts, among them J1 Barrel_Jack_Switch_SMT, J10 Conn_02x05_Odd_Even, J11 Screw_Terminal_01x02, J2 HS96L03W2C03_0.96_Oled, J5 Conn_02x05_Odd_Even, J6 Screw_Terminal_01x06, J9 Screw_Terminal_01x06, Q1 IRF540N, Q2 BSS138, SW1 6mm 2 Pin Tact NO Breadboard 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, SW2 6mm 2 Pin Tact NO Breadboard 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, SW3 6mm 2 Pin Tact NO Breadboard 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, U1 TMP36GRTZ-REEL7

Commit message: Deleted controller from heater board Schematic and PCB files. Deleted proxy from Assy_Enclosure_Rev2_PWA.FCStd file.
Parts:
- removed A1: Arduino_UNO_R3, GeneralPurposeAlarmDevicePCB:Arduino_UNO_R3_NoMountingHoles3D_Text_Top_&_Bottom
- removed BZ1: Buzzer_D12mm_H9.6mm_LS7.6mm, GeneralPurposeAlarmDevicePCB:Buzzer_12.2mm_9.7mm_7.62mm
- removed F1: Polyfuse 6A, GeneralPurposeAlarmDevicePCB:Fuse_BSMD_1812
- removed the G*** at (63.5, 136.5)
- removed H1, H2, H3, H4: MountingHole_Pad_3.5mm, GeneralPurposeAlarmDevicePCB:MountingHole_3.5mm_Pad_Via
- removed J1: Barrel_Jack_Switch_SMT, GeneralPurposeAlarmDevicePCB:BarrelJack_CLIFF_FC681465S_SMT_Horizontal
- removed J2: HS96L03W2C03_0.96_Oled, GeneralPurposeAlarmDevicePCB:OLED_HS96L03W2C03_0.96_WithNuts
- removed J5: Conn_02x05_Odd_Even, Connector_IDC:IDC-Header_2x05_P2.54mm_Vertical
- removed J6: Screw_Terminal_01x06, GeneralPurposeAlarmDevicePCB:1x6P 20A -40℃~+105℃ 300V Green 12~30 Straight pin 5.08mm 2.5 1 6 Plugin,P=5.08mm Screw ter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
- removed Q1: IRF540N, Package_TO_SOT_THT:TO-220-3_Horizontal_TabDown
- removed Q2: BSS138, Package_TO_SOT_SMD:SOT-23
- removed R1: 1R, Resistor_SMD:R_0603_1608Metric_Pad0.98x0.95mm_HandSolder
- removed R10: 10K, Resistor_SMD:R_0603_1608Metric_Pad0.98x0.95mm_HandSolder
- removed R2: DNI, Resistor_SMD:R_0603_1608Metric_Pad0.98x0.95mm_HandSolder
- removed R3, R4, R5, R6, R9: 1K, Resistor_SMD:R_0603_1608Metric_Pad0.98x0.95mm_HandSolder
- removed SW1, SW2, SW3: 6mm 2 Pin Tact NO Breadboard Friendly, GeneralPurposeAlarmDevicePCB:Switch_Tactile_THT_6x6mm
- removed TP1: TP_GND, TestPoint:TestPoint_Loop_D2.54mm_Drill1.5mm_Beaded
Connections:
- J11 pad 2: Net-(D1-A) -> HeaterDrive_IB
- R7 pad 1: Net-(U1-/SHUTDOWN) -> unconnected-(R7-Pad1)
Routing:
- net +5V: track 210.6 -> 0.00 mm, vias 10 -> 0
- net VCC: track 136.3 -> 0.00 mm, vias 3 -> 0
- net HEATER_ON: track 89.4 -> 0.00 mm
- net Net-(Q2-G): track 82.6 -> 0.00 mm
- net BTN_UP: track 77.5 -> 0.00 mm, vias 5 -> 0
- net SCL: track 68.5 -> 0.00 mm, vias 4 -> 0
- net SDA: track 62.2 -> 0.00 mm, vias 4 -> 0
- net BTN_DOWN: track 60.0 -> 0.00 mm, vias 3 -> 0
- net HeaterDrive: track 57.7 -> 0.00 mm, vias 1 -> 0
- net TempOut: track 46.5 -> 0.00 mm, vias 1 -> 0
- net GND: track 39.3 -> 0.00 mm, vias 30 -> 0
- net BUZZER_ON: track 32.6 -> 0.00 mm
- net BTN_SELECT: track 29.1 -> 0.00 mm, vias 2 -> 0
- net Net-(F1-Pad2): track 21.0 -> 0.00 mm
- net TEMP_IN: track 18.0 -> 0.00 mm, vias 1 -> 0
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- removed copper zone on B.Cu, net GND
- removed copper zone on F.Cu, net GND
Other:
- board text added: "MoonratII Heater, Public Invention, Rev 3.0 20241206"
- board text removed: "CERN Open Hardware License Version 2 - Strongly Reciprocal"
- board text removed: "MoonratII Controller, Public Invention, Rev 2.0 20240302"
- board text removed: "MoonratII Heater, Public Invention, Rev 2.0 20240302"
- board text removed: "locked"

Commit message: Updated PCB.
Parts:
- added U1: DS18B20, Package_TO_SOT_THT:TO-92_Inline, F.Cu at (147.5, 129.8)
Connections:
- R7 pad 1: unconnected-(R7-Pad1) -> TempOut_IB
