File: moonratII_2_1/pcb_moonratII/moonratII.kicad_sch (KiCad schematic)
At the start: 52 parts, among them J1 Barrel_Jack_Switch_SMT, J10 Conn_02x05_Odd_Even, J11 Screw_Terminal_01x02, J2 HS96L03W2C03_0.96_Oled, J5 Conn_02x05_Odd_Even, J6 Screw_Terminal_01x06, J9 Screw_Terminal_01x06, Q1 IRF540N, Q2 BSS138, SW1 6mm 2 Pin Tact NO Breadboard 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, SW2 6mm 2 Pin Tact NO Breadboard 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, SW3 6mm 2 Pin Tact NO Breadboard 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, U1 TMP36GRTZ-REEL7

Commit message: Updated heater schematic
Parts:
- removed U1: TMP36GRTZ-REEL7, Package_TO_SOT_SMD:SOT-23-5, symbol GPAD_SCH_LIB:TMP36GRTZ-REEL7
- added U1: TSIC306-TO92, Package_TO_SOT_THT:TO-92_Inline, symbol Sensor_Temperature:TSIC306-TO92
- added U2: TLP175A, Package_SO:MFSOP6-4_4.4x3.6mm_P1.27mm, symbol Relay_SolidState:TLP175A
- A1: value Arduino_UNO_R3 with uUSB and Cable -> Arduino_UNO_R4 with USB-C connector
Connections:
- net HeaterDrive_IB is gone; now on net VCCQ: D1.1 (K), J10.1 (Pin_1), J10.10 (Pin_10), J9.3 (Pin_3)
- net GND1: now also U2.1
- net VCCQ: now also U2.4, U2.6
- net at D1.2 (A), J11.2 (Pin_2), R8.1: now also U2.3
Other:
- moved on the sheet: D1, R7

Commit message: Updated heater board with a power flag.
Connections:
- net +5P: now also R7.1; no longer R7.2
- net GND1: now also U1.3 (GND)
- net TempOut_IB: now also U1.2 (Signal); no longer J10.4 (Pin_4), J10.7 (Pin_7), J9.5 (Pin_5)
- net at U1.1 (V+): now also R7.2
- new net: J10.4 (Pin_4), J10.7 (Pin_7), J9.5 (Pin_5)
- no-connect marks 48 -> 47
Other:
- moved on the sheet: R7, U1
