File: heaterboard_1/heaterboard_1.kicad_sch (KiCad schematic)
At the start: 12 parts, among them J3 Screw_Terminal_01x06, J4 Conn_02x05_Odd_Even, J7 Screw_Terminal_01x02, U2 TLP175A, U3 TSIC206-TO92

Commit message: heaterboard_1/heaterboard_1.kicad_sch Adding DS18B20 digital thermometer and 4.7 resistor to schematic, add datasheet.
Parts:
- removed U3: TSIC206-TO92, Package_TO_SOT_THT:TO-92_Inline, symbol Sensor_Temperature:TSIC206-TO92
- added U1: DS18B20, Package_TO_SOT_THT:TO-92_Inline, symbol Sensor_Temperature:DS18B20
- R11: value 1R -> 4.7R
Connections:
- net GND1: now also U1.1 (GND)
- net TempOut_IB: now also U1.2 (DQ)
- net at R11.2: now also U1.3 (V_{DD})
Other:
- moved on the sheet: R11
Changed lines of the file:
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@@
   (junction (at 52.07 87.63) (diameter 0) (color 0 0 0 0)
   )
-  (junction (at 76.835 48.26) (diameter 0) (color 0 0 0 0)
-  )
   (junction (at 74.295 90.17) (diameter 0) (color 0 0 0 0)
   )
@@
   (junction (at 43.18 54.61) (diameter 0) (color 0 0 0 0)
   )
+  (junction (at 82.55 48.26) (diameter 0) (color 0 0 0 0)
+  )
   (junction (at 46.99 92.71) (diameter 0) (color 0 0 0 0)
   )
@@
   (junction (at 60.96 90.17) (diameter 0) (color 0 0 0 0)
   )
+  (junction (at 76.2 48.26) (diameter 0) (color 0 0 0 0)
+  )
   (junction (at 50.8 72.39) (diameter 0) (color 0 0 0 0)
   )
-  (junction (at 83.82 48.26) (diameter 0) (color 0 0 0 0)
+  (junction (at 76.2 57.15) (diameter 0) (color 0 0 0 0)
   )
   (junction (at 54.61 64.77) (diameter 0) (color 0 0 0 0)
@@
     (stroke (width 0) (type default))
   )
+  (wire (pts (xy 82.55 48.26) (xy 85.09 48.26))
+    (stroke (width 0) (type default))
+  )
   (wire (pts (xy 81.28 83.82) (xy 81.28 91.44))
     (stroke (width 0) (type default))
   )
+  (wire (pts (xy 76.2 48.26) (xy 74.295 48.26))
+    (stroke (width 0) (type default))
+  )
   (wire (pts (xy 81.28 83.82) (xy 97.79 83.82))
     (stroke (width 0) (type default))
@@
     (stroke (width 0) (type default))
   )
-  (wire (pts (xy 79.375 48.26) (xy 83.82 48.26))
+  (wire (pts (xy 79.375 48.26) (xy 82.55 48.26))
     (stroke (width 0) (type default))
   )
@@
     (stroke (width 0) (type default))
   )
-  (wire (pts (xy 90.805 63.5) (xy 90.805 80.01))
+  (wire (pts (xy 90.805 64.77) (xy 90.805 80.01))
+    (stroke (width 0) (type default))
+  )
+  (wire (pts (xy 76.2 55.88) (xy 76.835 55.88))
     (stroke (width 0) (type default))
   )
@@
     (stroke (width 0) (type default))
   )
-  (wire (pts (xy 85.09 48.26) (xy 83.82 48.26))
-    (stroke (width 0) (type default))
-  )
   (wire (pts (xy 50.8 54.61) (xy 50.8 57.15))
     (stroke (width 0) (type default))
@@
     (stroke (width 0) (type default))
   )
-  (wire (pts (xy 83.82 48.26) (xy 83.82 38.1))
+  (wire (pts (xy 82.55 48.26) (xy 82.55 38.1))
     (stroke (width 0) (type default))
   )
@@
     (stroke (width 0) (type default))
   )
-  (wire (pts (xy 76.835 48.26) (xy 74.295 48.26))
-    (stroke (width 0) (type default))
-  )
   (wire (pts (xy 44.45 87.63) (xy 52.07 87.63))
     (stroke (width 0) (type default))
@@
     (stroke (width 0) (type default))
   )
-  (wire (pts (xy 90.805 63.5) (xy 86.995 63.5))
+  (wire (pts (xy 90.805 64.77) (xy 83.82 64.77))
     (stroke (width 0) (type default))
   )
@@
     (stroke (width 0) (type default))
   )
-  (wire (pts (xy 76.835 48.26) (xy 76.835 49.53))
-    (stroke (width 0) (type default))
-  )
-  (wire (pts (xy 76.835 55.88) (xy 76.835 57.15))
+  (wire (pts (xy 76.2 48.26) (xy 76.2 49.53))
+    (stroke (width 0) (type default))
+  )
+  (wire (pts (xy 76.2 55.88) (xy 76.2 57.15))
     (stroke (width 0) (type default))
   )
@@
     (stroke (width 0) (type default))
   )
-  (wire (pts (xy 81.915 73.66) (xy 76.835 73.66))
+  (wire (pts (xy 81.915 72.39) (xy 76.2 72.39))
     (stroke (width 0) (type default))
   )
@@
     (stroke (width 0) (type default))
   )
-  (wire (pts (xy 76.835 48.26) (xy 79.375 48.26))
-    (stroke (width 0) (type default))
-  )
-  (wire (pts (xy 81.915 73.66) (xy 81.915 76.2))
+  (wire (pts (xy 76.2 48.26) (xy 79.375 48.26))
+    (stroke (width 0) (type default))
+  )
+  (wire (pts (xy 81.915 72.39) (xy 81.915 76.2))
     (stroke (width 0) (type default))
   )
@@
   )
   (wire (pts (xy 76.2 83.82) (xy 78.74 83.82))
-    (stroke (width 0) (type default))
-  )
-  (wire (pts (xy 76.835 73.66) (xy 76.835 71.12))
     (stroke (width 0) (type default))
   )
@@
     )
   )
-  (symbol (lib_id "Device:R_US") (at 76.835 53.34 0) (unit 1)
+  (symbol (lib_id "Device:R_US") (at 76.2 53.34 0) (unit 1)
     (in_bom yes) (on_board yes) (dnp no)
-    (property "Reference" "R11" (at 79.375 49.53 90)
-      (effects (font (size 1.27 1.27)))
-    )
-    (property "Value" "1R" (at 79.375 57.15 90)
-      (effects (font (size 1.27 1.27)))
-    )
-    (property "Footprint" "Resistor_SMD:R_0603_1608Metric_Pad0.98x0.95mm_HandSolder" (at 77.851 53.594 90)
-      (effects (font (size 1.27 1.27)) hide)
-    )
-    (property "Datasheet" "https://www.amazon.com/Momentary-Tactile-Through-Breadboard-Friendly/dp/B07WF76VHT/" (at 76.835 53.34 0)
-      (effects (font (size 1.27 1.27)) hide)
-    )
-    (property "AssemblyType" "SMT" (at 76.835 53.34 0)
-      (effects (font (size 1.27 1.27)) hide)
-    )
-    (property "Cost" "0.0015" (at 76.835 53.34 0)
-      (effects (font (size 1.27 1.27)) hide)
-    )
-    (property "Description" "0.1W ±5% 1Ω 0603 Chip Resistor - Surface Mount ROHS" (at 76.835 53.34 0)
-      (effects (font (size 1.27 1.27)) hide)
-    )
-    (property "Distributor 1" "JLCPCB" (at 76.835 53.34 0)
-      (effects (font (size 1.27 1.27)) hide)
-    )
-    (property "Distributor 1 PN" "C269434" (at 76.835 53.34 0)
-      (effects (font (size 1.27 1.27)) hide)
-    )
-    (property "MPN" "RMC060315%N" (at 76.835 53.34 0)
-      (effects (font (size 1.27 1.27)) hide)
-    )
-    (property "Manufacturer" "TyoHM" (at 76.835 53.34 0)
-      (effects (font (size 1.27 1.27)) hide)
-    )
-    (property "Notes" "" (at 76.835 53.34 0)
+    (property "Reference" "R11" (at 78.74 52.07 90)
+      (effects (font (size 1.27 1.27)))
+    )
+    (property "Value" "4.7R" (at 72.39 53.34 0)
+      (effects (font (size 1.27 1.27)))
+    )
+    (property "Footprint" "Resistor_SMD:R_0603_1608Metric_Pad0.98x0.95mm_HandSolder" (at 77.216 53.594 90)
+      (effects (font (size 1.27 1.27)) hide)
+    )
+    (property "Datasheet" "https://www.amazon.com/Momentary-Tactile-Through-Breadboard-Friendly/dp/B07WF76VHT/" (at 76.2 53.34 0)
+      (effects (font (size 1.27 1.27)) hide)
+    )
+    (property "AssemblyType" "SMT" (at 76.2 53.34 0)
+      (effects (font (size 1.27 1.27)) hide)
+    )
+    (property "Cost" "0.0015" (at 76.2 53.34 0)
+      (effects (font (size 1.27 1.27)) hide)
+    )
+    (property "Description" "0.1W ±5% 1Ω 0603 Chip Resistor - Surface Mount ROHS" (at 76.2 53.34 0)
+      (effects (font (size 1.27 1.27)) hide)
+    )
+    (property "Distributor 1" "JLCPCB" (at 76.2 53.34 0)
+      (effects (font (size 1.27 1.27)) hide)
+    )
+    (property "Distributor 1 PN" "C269434" (at 76.2 53.34 0)
+      (effects (font (size 1.27 1.27)) hide)
+    )
+    (property "MPN" "RMC060315%N" (at 76.2 53.34 0)
+      (effects (font (size 1.27 1.27)) hide)
+    )
+    (property "Manufacturer" "TyoHM" (at 76.2 53.34 0)
+      (effects (font (size 1.27 1.27)) hide)
+    )
+    (property "Notes" "" (at 76.2 53.34 0)
       (effects (font (size 1.27 1.27)) hide)
     )
@@
     )
   )
-  (symbol (lib_id "power:PWR_FLAG") (at 83.82 38.1 0) (unit 1)
+  (symbol (lib_id "power:PWR_FLAG") (at 82.55 38.1 0) (unit 1)
     (in_bom yes) (on_board yes) (dnp no)
-    (property "Reference" "#FLG010" (at 83.82 36.195 0)
-      (effects (font (size 1.27 1.27)) hide)
-    )
-    (property "Value" "PWR_FLAG" (at 90.17 37.465 0)
-      (effects (font (size 1.27 1.27)))
-    )
-    (property "Footprint" "" (at 83.82 38.1 0)
-      (effects (font (size 1.27 1.27)) hide)
-    )
-    (property "Datasheet" "~" (at 83.82 38.1 0)
+    (property "Reference" "#FLG010" (at 82.55 36.195 0)
+      (effects (font (size 1.27 1.27)) hide)
+    )
+    (property "Value" "PWR_FLAG" (at 88.9 37.465 0)
+      (effects (font (size 1.27 1.27)))
+    )
+    (property "Footprint" "" (at 82.55 38.1 0)
+      (effects (font (size 1.27 1.27)) hide)
+    )
+    (property "Datasheet" "~" (at 82.55 38.1 0)
       (effects (font (size 1.27 1.27)) hide)
     )
@@
     )
   )
+  (symbol (lib_id "Sensor_Temperature:DS18B20") (at 76.2 64.77 0) (unit 1)
+    (in_bom yes) (on_board yes) (dnp no)
+    (property "Reference" "U1" (at 69.85 63.5 0)
+      (effects (font (size 1.27 1.27)) (justify right))
+    )
+    (property "Value" "DS18B20" (at 72.39 58.42 0)
+      (effects (font (size 1.27 1.27)) (justify right))
+    )
+    (property "Footprint" "Package_TO_SOT_THT:TO-92_Inline" (at 50.8 71.12 0)
+      (effects (font (size 1.27 1.27)) hide)
+    )
+    (property "Datasheet" "https://cdn-shop.adafruit.com/datasheets/DS18B20.pdf" (at 72.39 58.42 0)
+      (effects (font (size 1.27 1.27)) hide)
+    )
+    (pin "1")
+    (pin "2")
+    (pin "3")
+    (instances
+      (project "heaterboard_1"
+        (path "/9ef5effe-cb46-4a9a-bbbe-a65ab44b9e67"
+          (reference "U1") (unit 1)
+        )
+      )
+    )
+  )
   (symbol (lib_id "power:PWR_FLAG") (at 20.32 40.64 0) (unit 1)
     (in_bom yes) (on_board yes) (dnp no)
@@
         )
       )
-    )
-  )
-  (symbol (lib_id "Sensor_Temperature:TSIC206-TO92") (at 76.835 63.5 0) (unit 1)
-    (in_bom yes) (on_board yes) (dnp no)
-    (property "Reference" "U3" (at 67.945 62.23 0)
-      (effects (font (size 1.27 1.27)) (justify right))
-    )
-    (property "Value" "TSIC206-TO92" (at 74.295 55.88 0)
-      (effects (font (size 1.27 1.27)) (justify right))
-    )
-    (property "Footprint" "Package_TO_SOT_THT:TO-92_Inline" (at 67.945 59.69 0)
-      (effects (font (size 1.27 1.27)) (justify left) hide)
-    )
-    (property "Datasheet" "https://shop.bb-sensors.com/out/media/Datasheet_Digital_Semiconductor_temperatur_sensor_TSIC.pdf" (at 76.835 63.5 0)
-      (effects (font (size 1.27 1.27)) hide)
-    )
-    (property "Description" "Digital temperature sensor, range -50 ... +150 °C, 0.3 K accuracy, TO-92" (at 76.835 63.5 0)
-      (effects (font (size 1.27 1.27)) hide)
-    )
-    (pin "1")
-    (pin "2")
-    (pin "3")
-    (instances
-      (project "heaterboard_1"
-        (path "/9ef5effe-cb46-4a9a-bbbe-a65ab44b9e67"
-          (reference "U3") (unit 1)
-        )
-      )

Commit message: heaterboard_1.kicad_sch Adding connectors for the Dalla One wire and 4K7 pullup.
Parts:
- removed C2: 0.1uF, Capacitor_SMD:C_0603_1608Metric_Pad1.08x0.95mm_HandSolder, symbol Device:C
- removed D2: Schottky 2A, Diode_SMD:D_SMB, symbol Device:D_Schottky
- removed H7, H8: MountingHole_Pad_3.5mm, GeneralPurposeAlarmDevicePCB:MountingHole_3.5mm_Pad_Via, symbol GPAD_SCH_LIB:MountingHole_Pad_3.5mm
- removed J3: Screw_Terminal_01x06, GeneralPurposeAlarmDevicePCB:1x6P 20A -40℃~+105℃ 300V Green 12~30 Straight pin 5.08mm 2.5 1 6 Plugin,P=5.08mm Screw ter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, symbol Connector:Screw_Terminal_01x06
- removed J4: Conn_02x05_Odd_Even, Connector_IDC:IDC-Header_2x05_P2.54mm_Vertical, symbol Connector_Generic:Conn_02x05_Odd_Even
- removed J7: Screw_Terminal_01x02, TerminalBlock_TE-Connectivity:TerminalBlock_TE_282834-2_1x02_P2.54mm_Horizontal, symbol Connector:Screw_Terminal_01x02
- removed R11: 4.7R, Resistor_SMD:R_0603_1608Metric_Pad0.98x0.95mm_HandSolder, symbol Device:R_US
- removed R12: Heater, symbol Device:Heater
- removed U1: DS18B20, Package_TO_SOT_THT:TO-92_Inline, symbol Sensor_Temperature:DS18B20
- removed U2: TLP175A, Package_SO:MFSOP6-4_4.4x3.6mm_P1.27mm, symbol Relay_SolidState:TLP175A
- added C1: 0.1uF, Capacitor_SMD:C_0603_1608Metric_Pad1.08x0.95mm_HandSolder, symbol Device:C
- added H1, H2: MountingHole_Pad_3.5mm, GeneralPurposeAlarmDevicePCB:MountingHole_3.5mm_Pad_Via, symbol GPAD_SCH_LIB:MountingHole_Pad_3.5mm
- added J1: Screw_Terminal_01x06, GeneralPurposeAlarmDevicePCB:1x6P 20A -40℃~+105℃ 300V Green 12~30 Straight pin 5.08mm 2.5 1 6 Plugin,P=5.08mm Screw ter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, symbol Connector:Screw_Terminal_01x06
- added J2: Conn_02x05_Odd_Even, Connector_IDC:IDC-Header_2x05_P2.54mm_Vertical, symbol Connector_Generic:Conn_02x05_Odd_Even
- added J5, J8: Screw_Terminal_01x02, TerminalBlock_TE-Connectivity:TerminalBlock_TE_282834-2_1x02_P2.54mm_Horizontal, symbol Connector:Screw_Terminal_01x02
- added J7: Screw_Terminal_01x03, symbol Connector:Screw_Terminal_01x03
- added R1: 4K7, Resistor_SMD:R_0603_1608Metric_Pad0.98x0.95mm_HandSolder, symbol Device:R_US
- added R2, R5: Heater, symbol Device:Heater
- added TP1: TP_GND, TestPoint:TestPoint_Loop_D2.54mm_Drill1.5mm_Beaded, symbol Connector:TestPoint
Connections:
- net +5P: now also C1.1, J1.4 (Pin_4), J2.3 (Pin_3), J2.8 (Pin_8), J7.3 (Pin_3), R1.2
- net GND1: now also C1.2, H1.1, H2.1, J1.1 (Pin_1), J1.6 (Pin_6), J2.2 (Pin_2), J2.9 (Pin_9), J7.1 (Pin_1), TP1.1
- net HeaterDrive_IB: now also J1.3 (Pin_3), J2.1 (Pin_1), J2.10 (Pin_10), J5.2 (Pin_2), J8.2 (Pin_2), R2.1, R5.1
- net TempOut_IB: now also J1.5 (Pin_5), J2.4 (Pin_4), J2.7 (Pin_7), J7.2 (Pin_2), R1.1
- net VCCQ: now also J1.2 (Pin_2), J2.5 (Pin_5), J2.6 (Pin_6), J5.1 (Pin_1), J8.1 (Pin_1), R2.2, R5.2
Other:
- note added: "Connect to Dallas B8120 Color Code Pin 1-> Black(Blue): Ground Pin 2-> Yellow: Data Pin 3-> Red: +V"

Commit message: heaterboard_1.kicad_sch Using bulk editor, all part numbers and vaules correct.
Parts:
- C1: Cost 0.0021 -> 0.0024; MPN (none) -> CC0603KRX7R9BB104; Manufacturer (none) -> YAGEO
- H1, H2: MPN (none) -> NA; Manufacturer (none) -> NA
- J5, J8: MPN (none) -> XY308-2.54-2P; Manufacturer (none) -> Ningbo Xinlaiya Elec.
- J7: footprint (none) -> TerminalBlock_TE-Connectivity:TerminalBlock_TE_282834-3_1x03_P2.54mm_Horizontal; Cost (none) -> 0.35; Distributor 1 (none) -> JLCPCB; Distributor 1 PN (none) -> C557686; MPN (none) -> XY308-2.54-3P; Manufacturer (none) -> Ningbo Xinlaiya Elec.
- R2, R5: value Heater -> Heating Pad - 5x10cm; Cost 4.50 -> 4.75; MPN (none) -> NA; Manufacturer (none) -> NA
- SM1: Cost (none) -> 0; Distributor 1 (none) -> Public Invention; Distributor 1 PN (none) -> NA; MPN (none) -> NA; Manufacturer (none) -> NA
Changed lines of the file:
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@@
+      (effects (font (size 1.27 1.27)) hide)
+    )
+    (property "MPN" "NA" (at 110.49 66.04 0)
+      (effects (font (size 1.27 1.27)) hide)
+    )
+    (property "Manufacturer" "NA" (at 110.49 66.04 0)
       (effects (font (size 1.27 1.27)) hide)
     )
@@
       (effects (font (size 1.27 1.27)))
     )
-    (property "Footprint" "" (at 162.56 95.25 0)
+    (property "Footprint" "TerminalBlock_TE-Connectivity:TerminalBlock_TE_282834-3_1x03_P2.54mm_Horizontal" (at 162.56 95.25 0)
       (effects (font (size 1.27 1.27)) hide)
     )
     (property "Datasheet" "~" (at 162.56 95.25 0)
+      (effects (font (size 1.27 1.27)) hide)
+    )
+    (property "Distributor 1" "JLCPCB" (at 162.56 95.25 0)
+      (effects (font (size 1.27 1.27)) hide)
+    )
+    (property "Distributor 1 PN" "C557686" (at 162.56 95.25 0)
+      (effects (font (size 1.27 1.27)) hide)
+    )
+    (property "MPN" "XY308-2.54-3P" (at 162.56 95.25 0)
+      (effects (font (size 1.27 1.27)) hide)
+    )
+    (property "Manufacturer" "Ningbo Xinlaiya Elec." (at 162.56 95.25 0)
+      (effects (font (size 1.27 1.27)) hide)
+    )
+    (property "Cost" "0.35" (at 162.56 95.25 0)
       (effects (font (size 1.27 1.27)) hide)
     )
@@
       (effects (font (size 1.27 1.27)) (justify right))
     )
-    (property "Value" "Heater" (at 161.29 127 0)
+    (property "Value" "Heating Pad - 5x10cm" (at 161.29 127 0)
       (effects (font (size 1.27 1.27)) (justify right))
     )
@@
       (effects (font (size 1.27 1.27)) hide)
     )
-    (property "Cost" "4.50" (at 170.18 125.73 0)
+    (property "Cost" "4.75" (at 170.18 125.73 0)
       (effects (font (size 1.27 1.27)) hide)
     )
@@
     )
     (property "Notes" "" (at 170.18 125.73 0)
+      (effects (font (size 1.27 1.27)) hide)
+    )
+    (property "MPN" "NA" (at 170.18 125.73 0)
+      (effects (font (size 1.27 1.27)) hide)
+    )
+    (property "Manufacturer" "NA" (at 170.18 125.73 0)
       (effects (font (size 1.27 1.27)) hide)
     )
@@
       (effects (font (size 1.27 1.27)) hide)
     )
+    (property "Cost" "0" (at 236.22 180.34 0)
+      (effects (font (size 1.27 1.27)) hide)
+    )
+    (property "Distributor 1" "Public Invention" (at 236.22 180.34 0)
+      (effects (font (size 1.27 1.27)) hide)
+    )
+    (property "Distributor 1 PN" "NA" (at 236.22 180.34 0)
+      (effects (font (size 1.27 1.27)) hide)
+    )
+    (property "MPN" "NA" (at 236.22 180.34 0)
+      (effects (font (size 1.27 1.27)) hide)
+    )
+    (property "Manufacturer" "NA" (at 236.22 180.34 0)
+      (effects (font (size 1.27 1.27)) hide)
+    )
     (instances
       (project "heaterboard_1"
@@
       (effects (font (size 1.27 1.27)) hide)
     )
+    (property "MPN" "XY308-2.54-2P" (at 143.51 120.65 0)
+      (effects (font (size 1.27 1.27)) hide)
+    )
+    (property "Manufacturer" "Ningbo Xinlaiya Elec." (at 143.51 120.65 0)
+      (effects (font (size 1.27 1.27)) hide)
+    )
     (pin "1")
     (pin "2")
@@
       (effects (font (size 1.27 1.27)) hide)
     )
-    (property "Cost" "0.0021" (at 167.64 58.42 0)
+    (property "Cost" "0.0024" (at 167.64 58.42 0)
       (effects (font (size 1.27 1.27)) hide)
     )
@@
     )
     (property "Distributor 1 PN" "C14663" (at 167.64 58.42 0)
+      (effects (font (size 1.27 1.27)) hide)
+    )
+    (property "MPN" "CC0603KRX7R9BB104" (at 167.64 58.42 0)
+      (effects (font (size 1.27 1.27)) hide)
+    )
+    (property "Manufacturer" "YAGEO" (at 167.64 58.42 0)
       (effects (font (size 1.27 1.27)) hide)
     )
@@
       (effects (font (size 1.27 1.27)))
     )
-    (property "Value" "Heater" (at 142.24 127 90)
+    (property "Value" "Heating Pad - 5x10cm" (at 142.24 127 90)
       (effects (font (size 1.27 1.27)))
     )
@@
       (effects (font (size 1.27 1.27)) hide)
     )
-    (property "Cost" "4.50" (at 142.24 130.81 0)
+    (property "Cost" "4.75" (at 142.24 130.81 0)
       (effects (font (size 1.27 1.27)) hide)
     )
@@
     )
     (property "Notes" "" (at 142.24 130.81 0)
+      (effects (font (size 1.27 1.27)) hide)
+    )
+    (property "MPN" "NA" (at 142.24 130.81 0)
+      (effects (font (size 1.27 1.27)) hide)
+    )
+    (property "Manufacturer" "NA" (at 142.24 130.81 0)
       (effects (font (size 1.27 1.27)) hide)
     )
@@
       (effects (font (size 1.27 1.27)) hide)
     )
+    (property "MPN" "NA" (at 110.49 73.66 0)
+      (effects (font (size 1.27 1.27)) hide)
+    )
+    (property "Manufacturer" "NA" (at 110.49 73.66 0)
+      (effects (font (size 1.27 1.27)) hide)
+    )
     (pin "1")
     (instances
@@
       (effects (font (size 1.27 1.27)) hide)
     )
+    (property "MPN" "XY308-2.54-2P" (at 158.75 116.84 0)
+      (effects (font (size 1.27 1.27)) hide)
+    )
+    (property "Manufacturer" "Ningbo Xinlaiya Elec." (at 158.75 116.84 0)
+      (effects (font (size 1.27 1.27)) hide)
+    )

Commit message: heaterboard_1/heaterboard_1.kicad_sch Adding test points to all nets.
Parts:
- removed TP1: TP_GND, TestPoint:TestPoint_Loop_D2.54mm_Drill1.5mm_Beaded, symbol Connector:TestPoint
- added TP101: HeaterDrive_IB, TestPoint:TestPoint_Loop_D2.54mm_Drill1.5mm_Beaded, symbol Connector:TestPoint
- added TP101: TempOut_IB, TestPoint:TestPoint_Loop_D2.54mm_Drill1.5mm_Beaded, symbol Connector:TestPoint
- added TP101: VCCQ, TestPoint:TestPoint_Loop_D2.54mm_Drill1.5mm_Beaded, symbol Connector:TestPoint
- added TP101: +5P, TestPoint:TestPoint_Loop_D2.54mm_Drill1.5mm_Beaded, symbol Connector:TestPoint
- added TP101: TP_GND, TestPoint:TestPoint_Loop_D2.54mm_Drill1.5mm_Beaded, symbol Connector:TestPoint
Connections:
- net +5P: now also TP101.1
- net GND1: now also TP101.1
- net HeaterDrive_IB: now also TP101.1
- net TempOut_IB: now also TP101.1
- net VCCQ: now also TP101.1
Other:
- note added: "VCCQ 12V"
