File: heaterboard_1/heaterboard_1.kicad_sch (KiCad schematic)
At the start: 17 parts, among them J1 Screw_Terminal_01x06, J2 Conn_02x05_Odd_Even, J5 Screw_Terminal_01x02, J7 Screw_Terminal_01x03, J8 Screw_Terminal_01x02

Commit message: heaterboard_1/heaterboard_1.kicad_sch Addingnet names and added external components boundary box.
Other:
- note added: "Make traces heavy: - VCCQ 12V - HeaterDrive_IB"
- note added: "R5 & R2 are NOT on the PCB"
- moved on the sheet: R2
Changed lines of the file:
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@@
     (stroke (width 0) (type default))
   )
-  (wire (pts (xy 158.75 111.76) (xy 158.75 121.92))
+  (wire (pts (xy 158.75 111.76) (xy 158.75 127))
     (stroke (width 0) (type default))
   )
@@
     (stroke (width 0) (type default))
   )
-  (wire (pts (xy 156.21 111.76) (xy 156.21 129.54))
+  (wire (pts (xy 156.21 111.76) (xy 156.21 134.62))
     (stroke (width 0) (type default))
   )
@@
     (stroke (width 0) (type default))
   )
-  (wire (pts (xy 158.75 121.92) (xy 170.18 121.92))
+  (wire (pts (xy 158.75 127) (xy 170.18 127))
     (stroke (width 0) (type default))
   )
@@
     (stroke (width 0) (type default))
   )
-  (wire (pts (xy 156.21 129.54) (xy 170.18 129.54))
+  (wire (pts (xy 156.21 134.62) (xy 170.18 134.62))
     (stroke (width 0) (type default))
   )
@@
   (wire (pts (xy 102.87 107.95) (xy 102.87 104.14))
     (stroke (width 0) (type default))
+  )
+  (rectangle (start 135.89 123.19) (end 201.93 144.78)
+    (stroke (width 0.5) (type dash))
+    (fill (type none))
   )
   (image (at 254 180.34) (scale 0.75)
@@
     (effects (font (size 2.54 2.54)) (justify left bottom))
   )
+  (text "Make traces heavy:\n- VCCQ 12V\n- HeaterDrive_IB \n" (at 179.07 110.49 0)
+    (effects (font (size 1.27 1.27)) (justify left bottom))
+  )
+  (text "R5 & R2 are NOT on the PCB" (at 170.18 142.24 0)
+    (effects (font (size 1.27 1.27)) (justify left bottom))
+  )
   (text "Connect to Dallas B8120\n\nColor Code\nPin 1-> Black(Blue): Ground\nPin 2-> Yellow: Data\nPin 3-> Red: +V\n"
     (at 179.07 99.06 0)
@@
     )
   )
-  (symbol (lib_id "Device:Heater") (at 170.18 125.73 180) (unit 1)
+  (symbol (lib_id "Device:Heater") (at 170.18 130.81 180) (unit 1)
     (in_bom yes) (on_board no) (dnp no)
-    (property "Reference" "R2" (at 177.8 124.46 0)
+    (property "Reference" "R2" (at 177.8 129.54 0)
       (effects (font (size 1.27 1.27)) (justify right))
     )
-    (property "Value" "Heating Pad - 5x10cm" (at 176.53 127 0)
+    (property "Value" "Heating Pad - 5x10cm" (at 176.53 132.08 0)
       (effects (font (size 1.27 1.27)) (justify right))
     )
-    (property "Footprint" "" (at 171.958 125.73 90)
-      (effects (font (size 1.27 1.27)) hide)
-    )
-    (property "Datasheet" "https://www.sparkfun.com/products/11288" (at 170.18 125.73 0)
-      (effects (font (size 1.27 1.27)) hide)
-    )
-    (property "AssemblyType" "OTHER" (at 170.18 125.73 0)
-      (effects (font (size 1.27 1.27)) hide)
-    )
-    (property "Cost" "4.75" (at 170.18 125.73 0)
-      (effects (font (size 1.27 1.27)) hide)
-    )
-    (property "Description" "Heating Pad - 5x10cm" (at 170.18 125.73 0)
-      (effects (font (size 1.27 1.27)) hide)
-    )
-    (property "Distributor 1" "Sparkfun" (at 170.18 125.73 0)
-      (effects (font (size 1.27 1.27)) hide)
-    )
-    (property "Distributor 1 PN" "COM-11288" (at 170.18 125.73 0)
-      (effects (font (size 1.27 1.27)) hide)
-    )
-    (property "Notes" "" (at 170.18 125.73 0)
-      (effects (font (size 1.27 1.27)) hide)
-    )
-    (property "MPN" "NA" (at 170.18 125.73 0)
-      (effects (font (size 1.27 1.27)) hide)
-    )
-    (property "Manufacturer" "NA" (at 170.18 125.73 0)
+    (property "Footprint" "" (at 171.958 130.81 90)
+      (effects (font (size 1.27 1.27)) hide)
+    )
+    (property "Datasheet" "https://www.sparkfun.com/products/11288" (at 170.18 130.81 0)
+      (effects (font (size 1.27 1.27)) hide)
+    )
+    (property "AssemblyType" "OTHER" (at 170.18 130.81 0)
+      (effects (font (size 1.27 1.27)) hide)
+    )
+    (property "Cost" "4.75" (at 170.18 130.81 0)
+      (effects (font (size 1.27 1.27)) hide)
+    )
+    (property "Description" "Heating Pad - 5x10cm" (at 170.18 130.81 0)
+      (effects (font (size 1.27 1.27)) hide)
+    )
+    (property "Distributor 1" "Sparkfun" (at 170.18 130.81 0)
+      (effects (font (size 1.27 1.27)) hide)
+    )
+    (property "Distributor 1 PN" "COM-11288" (at 170.18 130.81 0)
+      (effects (font (size 1.27 1.27)) hide)
+    )
+    (property "Notes" "" (at 170.18 130.81 0)
+      (effects (font (size 1.27 1.27)) hide)
+    )
+    (property "MPN" "NA" (at 170.18 130.81 0)
+      (effects (font (size 1.27 1.27)) hide)
+    )
+    (property "Manufacturer" "NA" (at 170.18 130.81 0)
       (effects (font (size 1.27 1.27)) hide)
     )
@@
   (symbol (lib_id "Connector:Screw_Terminal_01x02") (at 158.75 116.84 270) (unit 1)
     (in_bom yes) (on_board yes) (dnp no)
-    (property "Reference" "J5" (at 170.815 127.635 0)
-      (effects (font (size 1.27 1.27)) (justify left))
-    )
+    (property "Reference" "J5" (at 171.45 125.73 0)
+      (effects (font (size 1.27 1.27)) (justify left))
+    )

Commit message: heaterboard_1/heaterboard_1.kicad_sch Correcting changed reference designators.
Parts:
- renumbered H1 to H5, H2 to H6, J2 to J10, J8 to J11, J5 to J12, J1 to J9, R1 to R7
Changed lines of the file:
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@@
   (symbol (lib_id "GPAD_SCH_LIB:MountingHole_Pad_3.5mm") (at 110.49 66.04 0) (unit 1)
     (in_bom yes) (on_board yes) (dnp no)
-    (property "Reference" "H1" (at 113.03 62.4586 0)
+    (property "Reference" "H5" (at 113.03 62.4586 0)
       (effects (font (size 1.27 1.27)) (justify left))
     )
@@
       (project "heaterboard_1"
         (path "/9ef5effe-cb46-4a9a-bbbe-a65ab44b9e67"
-          (reference "H1") (unit 1)
+          (reference "H5") (unit 1)
         )
       )
@@
   (symbol (lib_id "Device:R_US") (at 146.05 82.55 90) (unit 1)
     (in_bom yes) (on_board yes) (dnp no)
-    (property "Reference" "R1" (at 142.24 80.01 90)
+    (property "Reference" "R7" (at 142.24 80.01 90)
       (effects (font (size 1.27 1.27)))
     )
@@
       (project "heaterboard_1"
         (path "/9ef5effe-cb46-4a9a-bbbe-a65ab44b9e67"
-          (reference "R1") (unit 1)
+          (reference "R7") (unit 1)
         )
       )
@@
   (symbol (lib_id "Connector:Screw_Terminal_01x02") (at 143.51 120.65 270) (unit 1)
     (in_bom yes) (on_board yes) (dnp no)
-    (property "Reference" "J8" (at 146.685 121.285 90)
+    (property "Reference" "J11" (at 147.32 115.57 90)
       (effects (font (size 1.27 1.27)) (justify left))
     )
@@
       (project "heaterboard_1"
         (path "/9ef5effe-cb46-4a9a-bbbe-a65ab44b9e67"
-          (reference "J8") (unit 1)
+          (reference "J11") (unit 1)
         )
       )
@@
   (symbol (lib_id "Connector:Screw_Terminal_01x06") (at 115.57 91.44 0) (mirror y) (unit 1)
     (in_bom yes) (on_board yes) (dnp no)
-    (property "Reference" "J1" (at 113.03 91.4399 0)
+    (property "Reference" "J9" (at 113.03 91.4399 0)
       (effects (font (size 1.27 1.27)) (justify left))
     )
@@
       (project "heaterboard_1"
         (path "/9ef5effe-cb46-4a9a-bbbe-a65ab44b9e67"
-          (reference "J1") (unit 1)
+          (reference "J9") (unit 1)
         )
       )
@@
       (project "heaterboard_1"
         (path "/9ef5effe-cb46-4a9a-bbbe-a65ab44b9e67"
-          (reference "TP2") (unit 1)
+          (reference "TP1") (unit 1)
         )
       )
@@
       (project "heaterboard_1"
         (path "/9ef5effe-cb46-4a9a-bbbe-a65ab44b9e67"
-          (reference "TP1") (unit 1)
+          (reference "TP2") (unit 1)
         )
       )
@@
   (symbol (lib_id "Device:Heater") (at 142.24 130.81 90) (unit 1)
     (in_bom yes) (on_board no) (dnp no)
-    (property "Reference" "R5" (at 142.24 124.46 90)
+    (property "Reference" "R5" (at 143.51 128.27 90)
       (effects (font (size 1.27 1.27)))
     )
@@
   (symbol (lib_id "GPAD_SCH_LIB:MountingHole_Pad_3.5mm") (at 110.49 73.66 0) (unit 1)
     (in_bom yes) (on_board yes) (dnp no)
-    (property "Reference" "H2" (at 113.03 69.85 0)
+    (property "Reference" "H6" (at 113.03 69.85 0)
       (effects (font (size 1.27 1.27)) (justify left))
     )
@@
       (project "heaterboard_1"
         (path "/9ef5effe-cb46-4a9a-bbbe-a65ab44b9e67"
-          (reference "H2") (unit 1)
+          (reference "H6") (unit 1)
         )
       )
@@
   (symbol (lib_id "Connector:Screw_Terminal_01x02") (at 158.75 116.84 270) (unit 1)
     (in_bom yes) (on_board yes) (dnp no)
-    (property "Reference" "J5" (at 171.45 125.73 0)
+    (property "Reference" "J12" (at 162.56 113.03 90)
       (effects (font (size 1.27 1.27)) (justify left))
     )
@@
       (project "heaterboard_1"
         (path "/9ef5effe-cb46-4a9a-bbbe-a65ab44b9e67"
-          (reference "J5") (unit 1)
+          (reference "J12") (unit 1)
         )
       )
@@
   (symbol (lib_id "Connector_Generic:Conn_02x05_Odd_Even") (at 116.84 116.84 0) (mirror y) (unit 1)
     (in_bom yes) (on_board yes) (dnp no) (fields_autoplaced)
-    (property "Reference" "J2" (at 115.57 105.41 0)
+    (property "Reference" "J10" (at 115.57 105.41 0)
       (effects (font (size 1.27 1.27)))
     )
@@
       (project "heaterboard_1"
         (path "/9ef5effe-cb46-4a9a-bbbe-a65ab44b9e67"
-          (reference "J2") (unit 1)
-        )
-      )
+          (reference "J10") (unit 1)
+        )
+      )

Commit message: heaterboard_1.kicad_pcb Added open source symbol to the PCB silkscreen layer and unified title block for board silkscreen and schematic.
Parts:
- SM1: footprint GeneralPurposeAlarmDevicePCB:Logo_PI_BandW_70percent_10x10 -> Symbol:OSHW-Logo2_7.3x6mm_SilkScreen
Other:
- title: MoonratII Heaterboard -> MoonratII Heater Board
Changed lines of the file:
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@@
   (paper "A")
   (title_block
-    (title "MoonratII Heaterboard")
+    (title "MoonratII Heater Board")
     (date "2025-04-28")
     (rev "3.0")
@@
   (symbol (lib_id "Device:Heater") (at 170.18 130.81 180) (unit 1)
     (in_bom yes) (on_board no) (dnp no)
-    (property "Reference" "R2" (at 177.8 129.54 0)
+    (property "Reference" "R2" (at 166.37 130.81 0)
       (effects (font (size 1.27 1.27)) (justify right))
     )
-    (property "Value" "Heating Pad - 5x10cm" (at 176.53 132.08 0)
+    (property "Value" "Heating Pad - 5x10cm" (at 168.91 137.16 0)
       (effects (font (size 1.27 1.27)) (justify right))
     )
@@
   )
   (symbol (lib_id "Graphic:Logo_Open_Hardware_Small") (at 236.22 180.34 0) (unit 1)
-    (in_bom no) (on_board no) (dnp no) (fields_autoplaced)
+    (in_bom no) (on_board yes) (dnp no) (fields_autoplaced)
     (property "Reference" "SM1" (at 236.22 173.355 0)
       (effects (font (size 1.27 1.27)) hide)
@@
       (effects (font (size 1.27 1.27)) hide)
     )
-    (property "Footprint" "GeneralPurposeAlarmDevicePCB:Logo_PI_BandW_70percent_10x10" (at 236.22 180.34 0)
+    (property "Footprint" "Symbol:OSHW-Logo2_7.3x6mm_SilkScreen" (at 236.22 180.34 0)
       (effects (font (size 1.27 1.27)) hide)
     )
@@
   (symbol (lib_id "Connector:Screw_Terminal_01x02") (at 143.51 120.65 270) (unit 1)
     (in_bom yes) (on_board yes) (dnp no)
-    (property "Reference" "J11" (at 147.32 115.57 90)
+    (property "Reference" "J11" (at 142.24 114.3 90)
       (effects (font (size 1.27 1.27)) (justify left))
     )
@@
   (symbol (lib_id "Connector:Screw_Terminal_01x02") (at 158.75 116.84 270) (unit 1)
     (in_bom yes) (on_board yes) (dnp no)
-    (property "Reference" "J12" (at 162.56 113.03 90)
-      (effects (font (size 1.27 1.27)) (justify left))
-    )
+    (property "Reference" "J12" (at 160.02 114.3 90)
+      (effects (font (size 1.27 1.27)) (justify left))
+    )

Commit message: heaterboard_1.kicad_pcb and _sch files Cleared all design errors and warnings.
Parts:
- J11, J12: footprint TerminalBlock_TE-Connectivity:TerminalBlock_TE_282834-2_1x02_P2.54mm_Horizontal -> GeneralPurposeAlarmDevicePCB:GeneralPurposeAlarmDevicePCB_282834-2_1x02_P2.54mm_Horizontal
- J7: footprint TerminalBlock_TE-Connectivity:TerminalBlock_TE_282834-3_1x03_P2.54mm_Horizontal -> GeneralPurposeAlarmDevicePCB:GeneralPurposeAlarmDevicePCB_282834-3_1x03_P2.54mm_Horizontal
- J9: footprint GeneralPurposeAlarmDevicePCB:1x6P 20A -40℃~+105℃ 300V Green 12~30 Straight pin 5.08mm 2.5 1 6 Plugin,P=5.08mm Screw ter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 -> GeneralPurposeAlarmDevicePCB:GeneralPurposeAlarmDevicePCB_282834-6_1x02_p254mm_Horizontal
Changed lines of the file:
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@@
       (effects (font (size 1.27 1.27)))
     )
-    (property "Footprint" "TerminalBlock_TE-Connectivity:TerminalBlock_TE_282834-3_1x03_P2.54mm_Horizontal" (at 162.56 95.25 0)
+    (property "Footprint" "GeneralPurposeAlarmDevicePCB:GeneralPurposeAlarmDevicePCB_282834-3_1x03_P2.54mm_Horizontal" (at 162.56 95.25 0)
       (effects (font (size 1.27 1.27)) hide)
     )
@@
       (effects (font (size 1.27 1.27)) (justify left))
     )
-    (property "Footprint" "TerminalBlock_TE-Connectivity:TerminalBlock_TE_282834-2_1x02_P2.54mm_Horizontal" (at 143.51 120.65 0)
+    (property "Footprint" "GeneralPurposeAlarmDevicePCB:GeneralPurposeAlarmDevicePCB_282834-2_1x02_P2.54mm_Horizontal" (at 143.51 120.65 0)
       (effects (font (size 1.27 1.27)) hide)
     )
@@
       (effects (font (size 1.27 1.27)) (justify left))
     )
-    (property "Footprint" "GeneralPurposeAlarmDevicePCB:1x6P 20A -40℃~+105℃ 300V Green 12~30 Straight pin 5.08mm 2.5 1 6 Plugin,P=5.08mm Screw terminal ROHS" (at 115.57 91.44 0)
+    (property "Footprint" "GeneralPurposeAlarmDevicePCB:GeneralPurposeAlarmDevicePCB_282834-6_1x02_p254mm_Horizontal" (at 115.57 91.44 0)
       (effects (font (size 1.27 1.27)) hide)
     )
@@
       (effects (font (size 1.27 1.27)) (justify left))
     )
-    (property "Footprint" "TerminalBlock_TE-Connectivity:TerminalBlock_TE_282834-2_1x02_P2.54mm_Horizontal" (at 158.75 116.84 0)
-      (effects (font (size 1.27 1.27)) hide)
-    )
+    (property "Footprint" "GeneralPurposeAlarmDevicePCB:GeneralPurposeAlarmDevicePCB_282834-2_1x02_P2.54mm_Horizontal" (at 158.75 116.84 0)
+      (effects (font (size 1.27 1.27)) hide)
+    )
