File: heaterboard_1/heaterboard_1.kicad_sch (KiCad schematic)
At the start: 17 parts, among them J10 Conn_02x05_Odd_Even, J11 Screw_Terminal_01x02, J12 Screw_Terminal_01x02, J7 Screw_Terminal_01x03, J9 Screw_Terminal_01x06

Commit message: heaterboard_1.kicad_sch, change H5 and H6 to exclude from BOM. Generate CSV BOM file. Modify .gitignore so as to put CSV under version control.
Parts:
- H5, H6: now left out of the parts list
Changed lines of the file:
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@@
   )
   (symbol (lib_id "GPAD_SCH_LIB:MountingHole_Pad_3.5mm") (at 110.49 66.04 0) (unit 1)
-    (in_bom yes) (on_board yes) (dnp no)
+    (in_bom no) (on_board yes) (dnp no)
     (property "Reference" "H5" (at 113.03 62.4586 0)
       (effects (font (size 1.27 1.27)) (justify left))
@@
   )
   (symbol (lib_id "GPAD_SCH_LIB:MountingHole_Pad_3.5mm") (at 110.49 73.66 0) (unit 1)
-    (in_bom yes) (on_board yes) (dnp no)
+    (in_bom no) (on_board yes) (dnp no)
     (property "Reference" "H6" (at 113.03 69.85 0)
       (effects (font (size 1.27 1.27)) (justify left))
