File: heaterboard_1/heaterboard_1.kicad_pcb (KiCad board)
At the start: 2 copper layers, 108 x 65 mm, 37 parts, among them J1 Barrel_Jack_Switch_SMT, J10 Conn_02x05_Odd_Even, J11 Screw_Terminal_01x02, J2 HS96L03W2C03_0.96_Oled, J5 Conn_02x05_Odd_Even, J6 Screw_Terminal_01x06, J9 Screw_Terminal_01x06, Q1 IRF540N, Q2 BSS138, SW1 6mm 2 Pin Tact NO Breadboard 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, SW2 6mm 2 Pin Tact NO Breadboard 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, SW3 6mm 2 Pin Tact NO Breadboard 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, U1 TMP36GRTZ-REEL7

Commit message: heaterboard_1/heaterboard_1.kicad_pcb Removed deleted components from the PCB.
Parts:
- removed A1: Arduino_UNO_R3, GeneralPurposeAlarmDevicePCB:Arduino_UNO_R3_NoMountingHoles3D_Text_Top_&_Bottom
- removed BZ1: Buzzer_D12mm_H9.6mm_LS7.6mm, GeneralPurposeAlarmDevicePCB:Buzzer_12.2mm_9.7mm_7.62mm
- removed D1: Schottky 2A, Diode_SMD:D_SMB
- removed F1: Polyfuse 6A, GeneralPurposeAlarmDevicePCB:Fuse_BSMD_1812
- removed the G*** at (63.5, 136.5)
- removed H1, H2, H3, H4: MountingHole_Pad_3.5mm, GeneralPurposeAlarmDevicePCB:MountingHole_3.5mm_Pad_Via
- removed J1: Barrel_Jack_Switch_SMT, GeneralPurposeAlarmDevicePCB:BarrelJack_CLIFF_FC681465S_SMT_Horizontal
- removed J2: HS96L03W2C03_0.96_Oled, GeneralPurposeAlarmDevicePCB:OLED_HS96L03W2C03_0.96_WithNuts
- removed J5: Conn_02x05_Odd_Even, Connector_IDC:IDC-Header_2x05_P2.54mm_Vertical
- removed J6: Screw_Terminal_01x06, GeneralPurposeAlarmDevicePCB:1x6P 20A -40℃~+105℃ 300V Green 12~30 Straight pin 5.08mm 2.5 1 6 Plugin,P=5.08mm Screw ter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
- removed Q1: IRF540N, Package_TO_SOT_THT:TO-220-3_Horizontal_TabDown
- removed Q2: BSS138, Package_TO_SOT_SMD:SOT-23
- removed R1: 1R, Resistor_SMD:R_0603_1608Metric_Pad0.98x0.95mm_HandSolder
- removed R10: 10K, Resistor_SMD:R_0603_1608Metric_Pad0.98x0.95mm_HandSolder
- removed R2: DNI, Resistor_SMD:R_0603_1608Metric_Pad0.98x0.95mm_HandSolder
- removed R3, R4, R5, R6, R9: 1K, Resistor_SMD:R_0603_1608Metric_Pad0.98x0.95mm_HandSolder
- removed SW1, SW2, SW3: 6mm 2 Pin Tact NO Breadboard Friendly, GeneralPurposeAlarmDevicePCB:Switch_Tactile_THT_6x6mm
- removed U1: TMP36GRTZ-REEL7, Package_TO_SOT_SMD:SOT-23-5
- added J12: Screw_Terminal_01x02, TerminalBlock_TE-Connectivity:TerminalBlock_TE_282834-2_1x02_P2.54mm_Horizontal, F.Cu at (170.9, 128.6)
- added J7: Screw_Terminal_01x03, TerminalBlock_TE-Connectivity:TerminalBlock_TE_282834-3_1x03_P2.54mm_Horizontal, F.Cu at (170.9, 120.0)
- added TP3: TempOut_IB, TestPoint:TestPoint_Loop_D2.54mm_Drill1.5mm_Beaded, F.Cu at (165.8, 118.3)
- added TP4: HeaterDrive_IB, TestPoint:TestPoint_Loop_D2.54mm_Drill1.5mm_Beaded, F.Cu at (165.8, 123.3)
- added TP5: VCCQ, TestPoint:TestPoint_Loop_D2.54mm_Drill1.5mm_Beaded, F.Cu at (165.8, 128.4)
- R7: value 1R -> 4K7
- TP1: value TP_GND -> +5P
- moved TP1 57.3 mm to (153.0, 146.0)
- moved TP2 6.18 mm to (152.7, 139.8)
Connections:
- J10 pad 1: HeaterDrive_IB -> /HeaterDrive_IB
- J10 pad 10: HeaterDrive_IB -> /HeaterDrive_IB
- J10 pad 4: TempOut_IB -> /TempOut_IB
- J10 pad 7: TempOut_IB -> /TempOut_IB
- J11 pad 2: Net-(D1-A) -> /HeaterDrive_IB
- J9 pad 3: HeaterDrive_IB -> /HeaterDrive_IB
- J9 pad 5: TempOut_IB -> /TempOut_IB
- R7 pad 1: Net-(U1-/SHUTDOWN) -> /TempOut_IB
- TP1 pad 1: GND -> +5P
Routing:
- net (no net): track 0.00 -> 193.1 mm
- net HEATER_ON: track 89.4 -> 0.00 mm
- net Net-(Q2-G): track 82.6 -> 0.00 mm
- net /TempOut_IB: track 0.00 -> 73.2 mm, vias 0 -> 1
- net TempOut_IB: track 67.2 -> 0.00 mm, vias 1 -> 0
- net /HeaterDrive_IB: track 0.00 -> 52.5 mm, vias 0 -> 2
- net HeaterDrive_IB: track 42.3 -> 0.00 mm, vias 1 -> 0
- net +5P: track 64.0 -> 103.3 mm
- net GND: track 39.3 -> 0.00 mm, vias 30 -> 0
- net Net-(F1-Pad2): track 21.0 -> 0.00 mm
- net Net-(D1-A): track 10.1 -> 0.00 mm, vias 1 -> 0
- net Net-(U1-/SHUTDOWN): track 6.02 -> 0.00 mm
- net VCC: vias 3 -> 0
- net TempOut: vias 1 -> 0
- net TEMP_IN: vias 1 -> 0
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- added copper zone on B.Cu, net +5P
- added copper zone on F.Cu, net +5P
- removed copper zone on B.Cu, net GND
- removed copper zone on F.Cu, net GND
Other:
- board text removed: "CERN Open Hardware License Version 2 - Strongly Reciprocal"
- board text removed: "MoonratII Controller, Public Invention, Rev 2.0 20240302"

Commit message: heaterboard_1/heaterboard_1.kicad_pcb Adding new test points and parts from schematic to the PCB.
Parts:
- moved TP1 59.6 mm to (136.4, 88.7)
- moved TP3 26.7 mm to (144.1, 133.7)
- moved J7 24.8 mm to (152.8, 137.0), turned to 90 degrees
- moved TP5 24.5 mm to (143.9, 117.3)
- moved TP4 21.9 mm to (143.9, 124.4)
- moved J12 18.2 mm to (152.8, 126.9), turned to 90 degrees
- moved R7 9.14 mm to (138.6, 128.6)
- moved TP2 6.50 mm to (151.1, 146.1)
- moved C1 4.46 mm to (150.8, 141.1), turned to 180 degrees
- moved J11 4.43 mm to (152.5, 118.7)
Routing:
- net (no net): track 193.1 -> 1018.9 mm
- net +5V: track 210.6 -> 0.00 mm
- net VCC: track 136.3 -> 0.00 mm
- net BTN_UP: track 77.5 -> 0.00 mm
- net SCL: track 68.5 -> 0.00 mm
- net SDA: track 62.2 -> 0.00 mm
- net BTN_DOWN: track 60.0 -> 0.00 mm
- net HeaterDrive: track 57.7 -> 0.00 mm
- net TempOut: track 46.5 -> 0.00 mm
- net BUZZER_ON: track 32.6 -> 0.00 mm
- net BTN_SELECT: track 29.1 -> 0.00 mm
- net TEMP_IN: track 18.0 -> 0.00 mm
- net Net-(A1-D10): track 14.9 -> 0.00 mm
- net Net-(BZ1-+): track 8.76 -> 0.00 mm
- net Net-(A1-D8): track 3.17 -> 0.00 mm

Commit message: heaterboard_1/heaterboard_1.kicad_pcb Deleting all traces associated with the Control Board. Heater Board: placing connectors and testpoints.
Parts:
- moved R7 11.1 mm to (148.1, 134.3)
- moved TP4 7.16 mm to (143.1, 117.3)
- moved TP5 7.06 mm to (143.1, 124.3)
- moved TP3 1.89 mm to (143.1, 135.3)
- moved J11 1.42 mm to (153.0, 120.0)
- moved J7 1.02 mm to (153.0, 138.0)
- moved J12 0.28 mm to (153.0, 127.0)
Routing:
- net (no net): track 1018.9 -> 0.00 mm
- net +5P: track 103.3 -> 46.6 mm, vias 3 -> 0
- net /TempOut_IB: track 73.2 -> 90.6 mm
- net /HeaterDrive_IB: track 52.5 -> 42.2 mm, vias 2 -> 0
- net VCCQ: track 44.7 -> 54.8 mm
- net GND1: vias 9 -> 5

Commit message: heaterboard_1/heaterboard_1.kicad_pcb Setting the Heater Board edge cut.
Routing:
- net /TempOut_IB: track 90.6 -> 72.5 mm
- net GND1: track 13.6 -> 11.2 mm
Other:
- board size 108 x 65 mm -> 25.2 x 65 mm
Changed lines of the file:
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@@
     )
   )
-  (gr_line locked (start 50 150) (end 158 150)
-    (stroke (width 0.1) (type solid)) (layer "Edge.Cuts"))
-  (gr_line locked (start 158 85) (end 50 85)
-    (stroke (width 0.1) (type solid)) (layer "Edge.Cuts"))
-  (gr_line locked (start 50 85) (end 50 150)
+  (gr_line locked (start 132.8 150) (end 158 150)
+    (stroke (width 0.1) (type solid)) (layer "Edge.Cuts"))
+  (gr_line locked (start 158 85) (end 132.8 85)
+    (stroke (width 0.1) (type solid)) (layer "Edge.Cuts"))
+  (gr_line locked (start 132.8 85) (end 132.8 150)
     (stroke (width 0.1) (type solid)) (layer "Edge.Cuts"))
   (gr_line locked (start 158 150) (end 158 85)
@@
     (style (thickness 0.15) (arrow_length 1.27) (text_position_mode 0) (extension_height 0.58642) (extension_offset 0.5) keep_text_aligned)
   )
-  (segment (start 148.485 136.845214) (end 146.2775 136.845214) (width 0.381) (layer "F.Cu") (net 1))
-  (segment (start 146.1 135.792214) (end 146.1 133.829714) (width 0.508) (layer "F.Cu") (net 1))
-  (segment (start 142.4 139.329714) (end 142.4 137.842214) (width 0.508) (layer "F.Cu") (net 1))
   (segment (start 137.16 102.1588) (end 136.5 102.8188) (width 0.762) (layer "F.Cu") (net 1))
   (segment (start 143.9 133.475214) (end 143.9 133.456714) (width 0.762) (layer "F.Cu") (net 1))
   (segment (start 136.5 129.029714) (end 136.5 115.129714) (width 0.508) (layer "F.Cu") (net 1))
   (segment (start 140.092 132.621714) (end 136.5 129.029714) (width 0.508) (layer "F.Cu") (net 1))
-  (segment (start 145.15 138.067214) (end 145.15 139.079714) (width 0.508) (layer "F.Cu") (net 1))
-  (segment (start 149.273 136.057214) (end 148.485 136.845214) (width 0.381) (layer "F.Cu") (net 1))
   (segment (start 145.893263 132.621714) (end 140.092 132.621714) (width 0.508) (layer "F.Cu") (net 1))
-  (segment (start 143.2 140.129714) (end 142.4 139.329714) (width 0.508) (layer "F.Cu") (net 1))
   (segment (start 147.05 135.792214) (end 147.05 133.778451) (width 0.508) (layer "F.Cu") (net 1))
-  (segment (start 143.9 133.329714) (end 142.4 134.829714) (width 0.508) (layer "F.Cu") (net 1))
-  (segment (start 145.15 139.079714) (end 144.1 140.129714) (width 0.508) (layer "F.Cu") (net 1))
-  (segment (start 145.6 133.329714) (end 143.9 133.329714) (width 0.508) (layer "F.Cu") (net 1))
-  (segment (start 144.1 140.129714) (end 143.2 140.129714) (width 0.508) (layer "F.Cu") (net 1))
-  (segment (start 146.1 133.829714) (end 145.6 133.329714) (width 0.508) (layer "F.Cu") (net 1))
   (segment (start 136.5 102.8188) (end 136.5 115.129714) (width 0.762) (layer "F.Cu") (net 1))
-  (segment (start 142.4 134.829714) (end 142.4 136.017214) (width 0.508) (layer "F.Cu") (net 1))
-  (segment (start 146.2775 136.845214) (end 146.1 136.667714) (width 0.381) (layer "F.Cu") (net 1))
   (segment (start 147.05 133.778451) (end 145.893263 132.621714) (width 0.508) (layer "F.Cu") (net 1))
-  (segment (start 146.1 136.667714) (end 146.1 135.792214) (width 0.381) (layer "F.Cu") (net 1))
   (via (at 137.16 102.1588) (size 0.8) (drill 0.4) (layers "F.Cu" "B.Cu") (net 1))
   (segment (start 143.63 102.99) (end 141.09 100.45) (width 0.762) (layer "B.Cu") (net 1))
@@
   (segment (start 146.17 98.25) (end 146.17 100.45) (width 1.27) (layer "B.Cu") (net 2))
   (segment (start 142.294714 108.329714) (end 141.09 107.125) (width 0.254) (layer "F.Cu") (net 3))
-  (segment (start 148.988 138.067214) (end 149.273 137.782214) (width 0.381) (layer "F.Cu") (net 3))
   (segment (start 149.914714 108.329714) (end 142.294714 108.329714) (width 0.254) (layer "F.Cu") (net 3))
   (segment (start 151.25 109.665) (end 149.914714 108.329714) (width 0.254) (layer "F.Cu") (net 3))
-  (segment (start 147.05 138.067214) (end 148.988 138.067214) (width 0.381) (layer "F.Cu") (net 3))
   (via (at 139.8 102.579714) (size 0.8) (drill 0.4) (layers "F.Cu" "B.Cu") (free) (net 3))
   (via (at 138.43 109.22) (size 0.8) (drill 0.4) (layers "F.Cu" "B.Cu") (free) (net 3))

Commit message: heaterboard_1/heaterboard_1.kicad_pcb Corrected the silkscreen date and version for the Heater Board.
Other:
- board text added: "MoonratII Heater Board, Public Invention, Rev 3.0 20250428"
- board text removed: "MoonratII Heater, Public Invention, Rev 2.0 20240302"
- board text removed: "locked"
Changed lines of the file:
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@@
   (title_block
     (title "MoonratII")
-    (date "2023-11-20")
-    (rev "1.0")
+    (date "2025-04-28")
+    (rev "3.0")
     (company "PublicInvention")
     (comment 1 "GNU Affero General Public License v3.0")
@@
   (gr_line locked (start 158 150) (end 158 85)
     (stroke (width 0.1) (type solid)) (layer "Edge.Cuts"))
-  (gr_line locked (start 132.8 149.9) (end 132.8 85.1)
-    (stroke (width 0.25) (type solid)) (layer "User.1"))
-  (gr_text "MoonratII Heater, Public Invention, Rev 2.0 20240302" (at 135.1 139.029714 90) (layer "F.SilkS")
+  (gr_text "MoonratII Heater Board, Public Invention, Rev 3.0 20250428" (at 135.05 148.329714 90) (layer "F.SilkS")
     (effects (font (size 1.143 1.143) (thickness 0.1524)) (justify left bottom))
   )
@@
     (effects (font (size 2 2) (thickness 0.3)) (justify left bottom))
   )
-  (gr_text "CERN Open Hardware \nLicense Version 2 \nStrongly Reciprocal\n" (at 139.3 148.529714 90) (layer "F.SilkS")
+  (gr_text "CERN Open Hardware \nLicense Version 2 \nStrongly Reciprocal\n" (at 139.3 148.329714 90) (layer "F.SilkS")
     (effects (font (size 0.889 0.889) (thickness 0.15)) (justify left bottom))
   )
-  (gr_text locked "V-CUT" (at 130.3 156.9) (layer "User.1")
-    (effects (font (size 1 1) (thickness 0.15)) (justify left bottom))
-  )
   (dimension (type aligned) (layer "Dwgs.User")

Commit message: heaterboard_1.kicad_pcb Added open source symbol to the PCB silkscreen layer and unified title block for board silkscreen and schematic.
Parts:
- added SM1: Logo_Open_Hardware_Small, Symbol:OSHW-Logo2_7.3x6mm_SilkScreen, F.Cu at (155.1, 143.3)
- moved G*** 0.96 mm to (153.2, 89.3)
Routing:
- net +5P: track 46.6 -> 86.6 mm, vias 0 -> 2
- net /TempOut_IB: track 72.5 -> 82.0 mm
- net VCCQ: track 54.8 -> 62.7 mm
- net /HeaterDrive_IB: track 42.2 -> 41.2 mm
- removed copper zone on B.Cu, net +5P
- removed copper zone on F.Cu, net +5P
- removed copper zone on B.Cu, net GND1
- removed copper zone on F.Cu, net GND1
Other:
- board text added: "Public Invention, MoonratII Heater Board, Rev 3.0 20250428"
- board text removed: "MoonratII Heater Board, Public Invention, Rev 3.0 20250428"
