File: heaterboard_1/heaterboard_1.kicad_pcb (KiCad board)
At the start: 2 copper layers, 25.2 x 65 mm, 16 parts, among them J10 Conn_02x05_Odd_Even, J11 Screw_Terminal_01x02, J12 Screw_Terminal_01x02, J7 Screw_Terminal_01x03, J9 Screw_Terminal_01x06

Commit message: heaterboard_1/heaterboard_1.kicad_pcb Adding a copper fill.
Routing:
- net /HeaterDrive_IB: track 41.2 -> 56.9 mm
- net GND1: vias 5 -> 7
- added copper zone on B.Cu, net GND1
- added copper zone on F.Cu, net GND1
Changed lines of the file:
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@@
     (pad "6" thru_hole circle (at 12.7 0 180) (size 2.1 2.1) (drill 1.1) (layers "*.Cu" "*.Mask")
       (net 3 "GND1") (pinfunction "Pin_6") (pintype "passive"))
+    (model "${KICAD6_3DMODEL_DIR}/TerminalBlock_TE-Connectivity.3dshapes/TerminalBlock_TE_282834-6_1x06_P2.54mm_Horizontal.wrl"
+      (offset (xyz 0 0 0))
+      (scale (xyz 1 1 1))
+      (rotate (xyz 0 0 0))
+    )
     (model "${KIPRJMOD}/parts/KF128-2.54-6P.step"
       (offset (xyz 6.3 0.2 0))
@@
       (rotate (xyz 0 0 0))
     )
-    (model "${KIPRJMOD}/parts/KF128-2.54-3P.step"
-      (offset (xyz 0 0 0))
-      (scale (xyz 1 1 1))
-      (rotate (xyz 0 0 0))
-    )
   )
   (footprint "TerminalBlock_TE-Connectivity:TerminalBlock_TE_282834-2_1x02_P2.54mm_Horizontal" locked (layer "F.Cu")
@@
     (pad "2" thru_hole circle (at 2.54 0 90) (size 2.1 2.1) (drill 1.1) (layers "*.Cu" "*.Mask")
       (net 2 "/HeaterDrive_IB") (pinfunction "Pin_2") (pintype "passive"))
-    (model "${KIPRJMOD}/parts/KF128-2.54-2P.step"
+    (model "${KICAD6_3DMODEL_DIR}/TerminalBlock_TE-Connectivity.3dshapes/TerminalBlock_TE_282834-2_1x02_P2.54mm_Horizontal.wrl"
       (offset (xyz 0 0 0))
       (scale (xyz 1 1 1))
@@
     (pts (xy 144 89) (xy 144 146))
     (height -22.3)
-    (gr_text "2244.0945 mils" (at 166.4 117.129714 90) (layer "Dwgs.User")
+    (gr_text "57.0000 mm" (at 166.4 117.129714 90) (layer "Dwgs.User")
       (effects (font (size 1 1) (thickness 0.15)))
     )
@@
     (pts (xy 144 146) (xy 144 150))
     (height -16.6)
-    (gr_text "157.4803 mils" (at 162.4 152.229714 90) (layer "Dwgs.User")
+    (gr_text "4.0000 mm" (at 162.4 152.229714 90) (layer "Dwgs.User")
       (effects (font (size 1 1) (thickness 0.15)))
     )
@@
     (pts (xy 144 89) (xy 144 85))
     (height 16.1)
-    (gr_text "157.4803 mils" (at 161.7 82.629714 90) (layer "Dwgs.User")
+    (gr_text "4.0000 mm" (at 161.7 82.629714 90) (layer "Dwgs.User")
       (effects (font (size 1 1) (thickness 0.15)))
     )
@@
     (pts (xy 144 89) (xy 132.8 89.029714))
     (height 8.509649)
-    (gr_text "440.9464 mils" (at 138.374373 79.355242 0.1520073927) (layer "Dwgs.User")
+    (gr_text "11.2000 mm" (at 138.374373 79.355242 0.1520073927) (layer "Dwgs.User")
       (effects (font (size 1 1) (thickness 0.15)))
     )
@@
     (pts (xy 132.8 85.1) (xy 158 85))
     (height -20.273767)
-    (gr_text "992.1338 mils" (at 145.314986 63.626402 0.227363011) (layer "Dwgs.User")
+    (gr_text "25.2002 mm" (at 145.314986 63.626402 0.227363011) (layer "Dwgs.User")
       (effects (font (size 1 1) (thickness 0.15)))
     )
@@
   (segment (start 153 135.46) (end 148.05 135.46) (width 1) (layer "B.Cu") (net 1))
   (segment (start 144.807 111.733) (end 145.074 112) (width 0.254) (layer "B.Cu") (net 1))
+  (segment (start 143.05 117.329714) (end 143.55 116.829714) (width 2.7) (layer "F.Cu") (net 2))
   (segment (start 152.845286 107.125) (end 153.55 107.829714) (width 0.762) (layer "F.Cu") (net 2))
-  (segment (start 143.55 116.829714) (end 152.05 116.829714) (width 2.7) (layer "F.Cu") (net 2))
   (segment (start 153.55 107.829714) (end 153.55 111.829714) (width 2.5) (layer "F.Cu") (net 2))
-  (segment (start 152.05 116.829714) (end 153.55 115.329714) (width 2.7) (layer "F.Cu") (net 2))
-  (segment (start 143.05 117.329714) (end 143.55 116.829714) (width 2.7) (layer "F.Cu") (net 2))
-  (segment (start 153.55 115.329714) (end 153.55 111.829714) (width 2.7) (layer "F.Cu") (net 2))
+  (segment (start 153.3 117.16) (end 153.55 116.91) (width 2.7) (layer "F.Cu") (net 2))
+  (segment (start 143.55 116.829714) (end 152.369714 116.829714) (width 2.7) (layer "F.Cu") (net 2))
+  (segment (start 152.7 117.16) (end 153.3 117.16) (width 2.7) (layer "F.Cu") (net 2))
   (segment (start 151.25 107.125) (end 152.845286 107.125) (width 0.762) (layer "F.Cu") (net 2))
+  (segment (start 153.55 116.91) (end 153.55 111.829714) (width 2.7) (layer "F.Cu") (net 2))
+  (segment (start 152.369714 116.829714) (end 152.7 117.16) (width 2.7) (layer "F.Cu") (net 2))
   (segment (start 143.05 117.329714) (end 141.09 115.369714) (width 2.7) (layer "B.Cu") (net 2))
   (segment (start 146.17 100.45) (end 151.25 105.53) (width 2.7) (layer "B.Cu") (net 2))
+  (segment (start 149.005286 124.46) (end 148.765 124.219714) (width 2.7) (layer "B.Cu") (net 2))
   (segment (start 146.304 98.552) (end 146.304 98.384) (width 0.508) (layer "B.Cu") (net 2))
+  (segment (start 153 124.46) (end 149.005286 124.46) (width 2.5) (layer "B.Cu") (net 2))
+  (segment (start 148.765 119.035) (end 150.4 117.4) (width 2.7) (layer "B.Cu") (net 2))
+  (segment (start 148.765 124.219714) (end 148.765 119.035) (width 2.7) (layer "B.Cu") (net 2))
   (segment (start 151.25 105.53) (end 151.25 107.125) (width 0.762) (layer "B.Cu") (net 2))
   (segment (start 146.304 98.384) (end 146.17 98.25) (width 0.508) (layer "B.Cu") (net 2))
+  (segment (start 150.4 117.4) (end 153 117.4) (width 2.5) (layer "B.Cu") (net 2))
   (segment (start 141.09 115.369714) (end 141.09 109.665) (width 2.7) (layer "B.Cu") (net 2))
   (segment (start 146.17 98.25) (end 146.17 100.45) (width 1.27) (layer "B.Cu") (net 2))
@@
   (via (at 139.8 102.579714) (size 0.8) (drill 0.4) (layers "F.Cu" "B.Cu") (free) (net 3))
   (via (at 138.43 109.22) (size 0.8) (drill 0.4) (layers "F.Cu" "B.Cu") (free) (net 3))
+  (via (at 145.59 121.044714) (size 0.8) (drill 0.4) (layers "F.Cu" "B.Cu") (free) (net 3))
   (via (at 148.59 112.395) (size 0.8) (drill 0.4) (layers "F.Cu" "B.Cu") (free) (net 3))
   (via (at 141.951122 105.005524) (size 0.8) (drill 0.4) (layers "F.Cu" "B.Cu") (free) (net 3))
+  (via (at 153.845 105.169714) (size 0.8) (drill 0.4) (layers "F.Cu" "B.Cu") (free) (net 3))
   (via (at 139.065 106.045) (size 0.8) (drill 0.4) (layers "F.Cu" "B.Cu") (free) (net 3))
   (segment (start 146.115 127.394714) (end 143.05 124.329714) (width 2.7) (layer "F.Cu") (net 4))
@@
       )
     )
+  )
+  (zone (net 3) (net_name "GND1") (layers "F&B.Cu") (hatch edge 0.5)
+    (connect_pads (clearance 0.508))
+    (min_thickness 0.25) (filled_areas_thickness no)
+    (fill yes (thermal_gap 0.5) (thermal_bridge_width 0.5))
+    (polygon
+      (pts
+        (xy 160.195 82.944714)
+        (xy 160.195 151.524714)
+        (xy 129.08 151.524714)
+        (xy 129.08 82.944714)
+      )
+    )

Commit message: heaterboard_1.kicad_pcb and _sch files Cleared all design errors and warnings.
Parts:
- J11, J12: footprint TerminalBlock_TE-Connectivity:TerminalBlock_TE_282834-2_1x02_P2.54mm_Horizontal -> GeneralPurposeAlarmDevicePCB:GeneralPurposeAlarmDevicePCB_282834-2_1x02_P2.54mm_Horizontal
- J7: footprint TerminalBlock_TE-Connectivity:TerminalBlock_TE_282834-3_1x03_P2.54mm_Horizontal -> GeneralPurposeAlarmDevicePCB:GeneralPurposeAlarmDevicePCB_282834-3_1x03_P2.54mm_Horizontal
- J9: footprint GeneralPurposeAlarmDevicePCB:1x6P 20A -40℃~+105℃ 300V Green 12~30 Straight pin 5.08mm 2.5 1 6 Plugin,P=5.08mm Screw ter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 -> GeneralPurposeAlarmDevicePCB:GeneralPurposeAlarmDevicePCB_282834-6_1x02_p254mm_Horizontal
Changed lines of the file:
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@@
     )
     (pad_to_mask_clearance 0)
-    (grid_origin 143.05 115.329714)
+    (grid_origin 150.75 135.46)
     (pcbplotparams
       (layerselection 0x00410ff_ffffffff)
@@
     )
   )
-  (footprint "GeneralPurposeAlarmDevicePCB:1x6P 20A -40℃~+105℃ 300V Green 12~30 Straight pin 5.08mm 2.5 1 6 Plugin,P=5.08mm Screw terminal ROHS" (layer "F.Cu")
+  (footprint "GeneralPurposeAlarmDevicePCB:GeneralPurposeAlarmDevicePCB_282834-6_1x02_p254mm_Horizontal" (layer "F.Cu")
     (at 151.25 98.25 180)
     (descr "Terminal Block TE 282834-6, 6 pins, pitch 2.54mm, size 15.7x6.5mm^2, drill diamater 1.1mm, pad diameter 2.1mm, see http://www.te.com/commerce/DocumentDelivery/DDEController?Action=showdoc&DocId=Customer+Drawing%7F282834%7FC1%7Fpdf%7FEnglish%7FENG_CD_282834_C1.pdf, script-generated using https://github.com/pointhi/kicad-footprint-generator/scripts/TerminalBlock_TE-Connectivity")
@@
     (pad "6" thru_hole circle (at 12.7 0 180) (size 2.1 2.1) (drill 1.1) (layers "*.Cu" "*.Mask")
       (net 3 "GND1") (pinfunction "Pin_6") (pintype "passive"))
-    (model "${KICAD6_3DMODEL_DIR}/TerminalBlock_TE-Connectivity.3dshapes/TerminalBlock_TE_282834-6_1x06_P2.54mm_Horizontal.wrl"
-      (offset (xyz 0 0 0))
-      (scale (xyz 1 1 1))
-      (rotate (xyz 0 0 0))
-    )
-    (model "${KIPRJMOD}/parts/KF128-2.54-6P.step"
+    (model "${KIPRJMOD}/parts/KF128 2.54mm/KF128-2.54-6P.step"
       (offset (xyz 6.3 0.2 0))
       (scale (xyz 1 1 1))
@@
     )
   )
-  (footprint "TerminalBlock_TE-Connectivity:TerminalBlock_TE_282834-3_1x03_P2.54mm_Horizontal" (layer "F.Cu")
+  (footprint "GeneralPurposeAlarmDevicePCB:GeneralPurposeAlarmDevicePCB_282834-3_1x03_P2.54mm_Horizontal" (layer "F.Cu")
     (at 153 138 90)
     (descr "Terminal Block TE 282834-3, 3 pins, pitch 2.54mm, size 8.08x6.5mm^2, drill diamater 1.1mm, pad diameter 2.1mm, see http://www.te.com/commerce/DocumentDelivery/DDEController?Action=showdoc&DocId=Customer+Drawing%7F282834%7FC1%7Fpdf%7FEnglish%7FENG_CD_282834_C1.pdf, script-generated using https://github.com/pointhi/kicad-footprint-generator/scripts/TerminalBlock_TE-Connectivity")
@@
     (pad "3" thru_hole circle (at 5.08 0 90) (size 2.1 2.1) (drill 1.1) (layers "*.Cu" "*.Mask")
       (net 5 "+5P") (pinfunction "Pin_3") (pintype "passive"))
-    (model "${KICAD6_3DMODEL_DIR}/TerminalBlock_TE-Connectivity.3dshapes/TerminalBlock_TE_282834-3_1x03_P2.54mm_Horizontal.wrl"
-      (offset (xyz 0 0 0))
+    (model "${KIPRJMOD}/parts/KF128 2.54mm/KF128-2.54-3P.step"
+      (offset (xyz 2.54 0 0))
       (scale (xyz 1 1 1))
       (rotate (xyz 0 0 0))
     )
   )
-  (footprint "TerminalBlock_TE-Connectivity:TerminalBlock_TE_282834-2_1x02_P2.54mm_Horizontal" locked (layer "F.Cu")
+  (footprint "GeneralPurposeAlarmDevicePCB:GeneralPurposeAlarmDevicePCB_282834-2_1x02_P2.54mm_Horizontal" locked (layer "F.Cu")
     (at 153 120 90)
     (descr "Terminal Block TE 282834-2, 2 pins, pitch 2.54mm, size 5.54x6.5mm^2, drill diamater 1.1mm, pad diameter 2.1mm, see http://www.te.com/commerce/DocumentDelivery/DDEController?Action=showdoc&DocId=Customer+Drawing%7F282834%7FC1%7Fpdf%7FEnglish%7FENG_CD_282834_C1.pdf, script-generated using https://github.com/pointhi/kicad-footprint-generator/scripts/TerminalBlock_TE-Connectivity")
@@
     (pad "2" thru_hole circle locked (at 2.54 0 90) (size 2.1 2.1) (drill 1.1) (layers "*.Cu" "*.Mask")
       (net 2 "/HeaterDrive_IB") (pinfunction "Pin_2") (pintype "passive"))
-    (model "${KIPRJMOD}/parts/KF128-2.54-2P.step"
+    (model "${KIPRJMOD}/parts/KF128 2.54mm/KF128-2.54-2P.step"
       (offset (xyz 1.27 0 0))
       (scale (xyz 1 1 1))
@@
     )
   )
-  (footprint "TerminalBlock_TE-Connectivity:TerminalBlock_TE_282834-2_1x02_P2.54mm_Horizontal" (layer "F.Cu")
+  (footprint "GeneralPurposeAlarmDevicePCB:GeneralPurposeAlarmDevicePCB_282834-2_1x02_P2.54mm_Horizontal" (layer "F.Cu")
     (at 153 127 90)
     (descr "Terminal Block TE 282834-2, 2 pins, pitch 2.54mm, size 5.54x6.5mm^2, drill diamater 1.1mm, pad diameter 2.1mm, see http://www.te.com/commerce/DocumentDelivery/DDEController?Action=showdoc&DocId=Customer+Drawing%7F282834%7FC1%7Fpdf%7FEnglish%7FENG_CD_282834_C1.pdf, script-generated using https://github.com/pointhi/kicad-footprint-generator/scripts/TerminalBlock_TE-Connectivity")
@@
     (property "ki_keywords" "screw terminal")
     (attr through_hole)
-    (fp_text reference "J12" (at 0.04 -4.75 90) (layer "F.SilkS")
+    (fp_text reference "J12" (at 0.04 -4.75 270) (layer "F.SilkS")
         (effects (font (size 1 1) (thickness 0.15)))
     )
@@
     (pad "2" thru_hole circle (at 2.54 0 90) (size 2.1 2.1) (drill 1.1) (layers "*.Cu" "*.Mask")
       (net 2 "/HeaterDrive_IB") (pinfunction "Pin_2") (pintype "passive"))
-    (model "${KICAD6_3DMODEL_DIR}/TerminalBlock_TE-Connectivity.3dshapes/TerminalBlock_TE_282834-2_1x02_P2.54mm_Horizontal.wrl"
-      (offset (xyz 0 0 0))
+    (model "${KIPRJMOD}/parts/KF128 2.54mm/KF128-2.54-2P.step"
+      (offset (xyz 1.27 0 0))
       (scale (xyz 1 1 1))
       (rotate (xyz 0 0 0))
